File: signal_driver.sch (KiCad schematic (older format))
At the start: 29 parts, among them U2 74VHC541

Commit message: Modified to use matrix LEDs; Components layout has almost done, tracks and traces not yet.
Parts:
- removed R126, R127, R128: 10k, Resistors_SMD:R_0603_HandSoldering, symbol R
- added R17: 10R, Resistors_SMD:R_0603_HandSoldering, symbol R
- added W5: TEST_1P, Measurement_Points:Measurement_Point_Round-SMD-Pad_Small, symbol TEST_1P
- W1, W11, W2, W3, W4, W7, W9: footprint Pin_Headers:Pin_Header_Straight_1x01 -> Measurement_Points:Measurement_Point_Round-SMD-Pad_Small
Connections:
- net labels added: LED1642VDD, P_PWCLK_N, P_PWCLK_P, P_ROW_CLK, P_ROW_DAT, P_ROW_LAT
- net labels removed: B_RXD, E_HC595LATCH, E_PWCLK, LEDLOGICVDD, RXD
- wire segments 57 -> 52
- no-connect marks 0 -> 1
Changed lines of the file:
@@
 $Descr A4 11693 8268
 encoding utf-8
-Sheet 11 11
+Sheet 10 10
 Title ""
 Date ""
@@
 F 0 "W1" V 6850 4050 50  0000 C CNN
 F 1 "TEST_1P" V 6904 4074 50  0001 C CNN
-F 2 "Pin_Headers:Pin_Header_Straight_1x01" H 7000 4000 50  0001 C CNN
+F 2 "Measurement_Points:Measurement_Point_Round-SMD-Pad_Small" H 7000 4000 50  0001 C CNN
 F 3 "" H 7000 4000 50  0000 C CNN
 	1    6800 4000
@@
 F 0 "W2" V 6850 2700 50  0000 C CNN
 F 1 "TEST_1P" V 6904 2724 50  0001 C CNN
-F 2 "Pin_Headers:Pin_Header_Straight_1x01" H 7000 2650 50  0001 C CNN
+F 2 "Measurement_Points:Measurement_Point_Round-SMD-Pad_Small" H 7000 2650 50  0001 C CNN
 F 3 "" H 7000 2650 50  0000 C CNN
 	1    6800 2650
@@
 F 0 "W3" V 6850 2800 50  0000 C CNN
 F 1 "TEST_1P" V 6904 2824 50  0001 C CNN
-F 2 "Pin_Headers:Pin_Header_Straight_1x01" H 7000 2750 50  0001 C CNN
+F 2 "Measurement_Points:Measurement_Point_Round-SMD-Pad_Small" H 7000 2750 50  0001 C CNN
 F 3 "" H 7000 2750 50  0000 C CNN
 	1    6800 2750
@@
 F 0 "W7" V 6850 3500 50  0000 C CNN
 F 1 "TEST_1P" V 6904 3524 50  0001 C CNN
-F 2 "Pin_Headers:Pin_Header_Straight_1x01" H 7000 3450 50  0001 C CNN
+F 2 "Measurement_Points:Measurement_Point_Round-SMD-Pad_Small" H 7000 3450 50  0001 C CNN
 F 3 "" H 7000 3450 50  0000 C CNN
 	1    6800 3450
@@
 F 0 "W9" V 6850 3700 50  0000 C CNN
 F 1 "TEST_1P" V 6904 3724 50  0001 C CNN
-F 2 "Pin_Headers:Pin_Header_Straight_1x01" H 7000 3650 50  0001 C CNN
+F 2 "Measurement_Points:Measurement_Point_Round-SMD-Pad_Small" H 7000 3650 50  0001 C CNN
 F 3 "" H 7000 3650 50  0000 C CNN
 	1    6800 3650
@@
 $EndComp
 $Comp
-L GND #PWR31
+L GND #PWR0145
 U 1 1 5809183D
 P 5000 3900
-F 0 "#PWR31" H 5000 3650 50  0001 C CNN
+F 0 "#PWR0145" H 5000 3650 50  0001 C CNN
 F 1 "GND" H 5005 3727 50  0000 C CNN
 F 2 "" H 5000 3900 50  0000 C CNN
@@
 $EndComp
 $Comp
-L GND #PWR25
+L GND #PWR0144
 U 1 1 580918BF
 P 4250 3750
-F 0 "#PWR25" H 4250 3500 50  0001 C CNN
+F 0 "#PWR0144" H 4250 3500 50  0001 C CNN
 F 1 "GND" H 4255 3577 50  0000 C CNN
 F 2 "" H 4250 3750 50  0000 C CNN
@@
 $EndComp
 Text GLabel 3850 2950 0    60   Input ~ 0
-E_PWCLK
+P_PWCLK_N
 Text GLabel 3750 2750 0    60   Input ~ 0
 E_COLLATCH
@@
 E_COLSER
 Text GLabel 3750 3250 0    60   Input ~ 0
-E_HC595LATCH
+P_ROW_LAT
 Text GLabel 6550 3850 0    60   Input ~ 0
 E_BUTTONSENSE
@@
 Text GLabel 7800 2750 2    60   Input ~ 0
 COLLATCH
-Text GLabel 7800 2850 2    60   Input ~ 0
+Text GLabel 7800 3550 2    60   Input ~ 0
 COLSEROUT
 Text GLabel 7800 2950 2    60   Input ~ 0
@@
 Text GLabel 7800 3450 2    60   Input ~ 0
 HC595LATCH
-Text GLabel 7800 3550 2    60   Input ~ 0
+Text GLabel 6050 4500 2    60   Input ~ 0
 HC595SEROUT
 Text GLabel 7800 3650 2    60   Input ~ 0
 BUTTONSENSE
 $Comp
-L GND #PWR29
+L GND #PWR0143
 U 1 1 58199147
 P 4750 2350
-F 0 "#PWR29" H 4750 2100 50  0001 C CNN
+F 0 "#PWR0143" H 4750 2100 50  0001 C CNN
 F 1 "GND" H 4750 2200 50  0000 C CNN
 F 2 "" H 4750 2350 50  0000 C CNN
@@
 F 0 "W11" V 6850 3200 50  0000 C CNN
 F 1 "TEST_1P" V 6904 3224 50  0001 C CNN
-F 2 "Pin_Headers:Pin_Header_Straight_1x01" H 7000 3150 50  0001 C CNN
+F 2 "Measurement_Points:Measurement_Point_Round-SMD-Pad_Small" H 7000 3150 50  0001 C CNN
 F 3 "" H 7000 3150 50  0000 C CNN
 	1    6800 3150
@@
 $EndComp
 $Comp
-L GND #PWR27
+L GND #PWR0142
 U 1 1 582DB35E
 P 4400 2350
-F 0 "#PWR27" H 4400 2100 50  0001 C CNN
+F 0 "#PWR0142" H 4400 2100 50  0001 C CNN
 F 1 "GND" H 4405 2177 50  0000 C CNN
 F 2 "" H 4400 2350 50  0000 C CNN
@@
 F 0 "W4" V 6850 3600 50  0000 C CNN
 F 1 "TEST_1P" V 6904 3624 50  0001 C CNN
-F 2 "Pin_Headers:Pin_Header_Straight_1x01" H 7000 3550 50  0001 C CNN
+F 2 "Measurement_Points:Measurement_Point_Round-SMD-Pad_Small" H 7000 3550 50  0001 C CNN
 F 3 "" H 7000 3550 50  0000 C CNN
 	1    6800 3550
@@
 $EndComp
 $Comp
-L GND #PWR23
+L GND #PWR0141
 U 1 1 583D6553
 P 3650 2300
-F 0 "#PWR23" H 3650 2050 50  0001 C CNN
+F 0 "#PWR0141" H 3650 2050 50  0001 C CNN
 F 1 "GND" H 3655 2127 50  0000 C CNN
 F 2 "" H 3650 2300 50  0000 C CNN
@@
 	1    0    0    -1
 $EndComp
-$Comp
-L R R126
-U 1 1 5850CCB7
-P 6450 3550
-F 0 "R126" V 6450 3450 50  0000 L CNN
-F 1 "10k" V 6550 3400 50  0000 L CNN
-F 2 "Resistors_SMD:R_0603_HandSoldering" V 6380 3550 50  0001 C CNN
-F 3 "" H 6450 3550 50  0000 C CNN
-	1    6450 3550
-	0    -1   1    0
-$EndComp
 Text GLabel 5600 3600 3    60   Input ~ 0
 E_COLSER
@@
 L R R121
 U 1 1 585189D4
-P 6100 3700
-F 0 "R121" V 6100 3600 50  0000 L CNN
-F 1 "22k" V 6150 3800 50  0000 L CNN
-F 2 "Resistors_SMD:R_0603_HandSoldering" V 6030 3700 50  0001 C CNN
-F 3 "" H 6100 3700 50  0000 C CNN
-	1    6100 3700
-	0    1    1    0
-$EndComp
-$Comp
-L GND #PWR35
-U 1 1 5851C0D6
-P 5950 3700
-F 0 "#PWR35" H 5950 3450 50  0001 C CNN
-F 1 "GND" H 5955 3527 50  0000 C CNN
-F 2 "" H 5950 3700 50  0000 C CNN
-F 3 "" H 5950 3700 50  0000 C CNN
-	1    5950 3700
-	0    1    1    0
-$EndComp
-$Comp
-L R R127
-U 1 1 5850C306
 P 6050 3550
-F 0 "R127" V 6050 3450 50  0000 L CNN
-F 1 "10k" V 6000 3300 50  0000 L CNN
+F 0 "R121" V 6050 3450 50  0000 L CNN
+F 1 "22k" V 6100 3650 50  0000 L CNN
 F 2 "Resistors_SMD:R_0603_HandSoldering" V 5980 3550 50  0001 C CNN
 F 3 "" H 6050 3550 50  0000 C CNN
 	1    6050 3550
-	0    -1   1    0
-$EndComp
-Text GLabel 3250 2000 0    60   Input ~ 0
-LEDLOGICVDD
-Text GLabel 3850 2850 0    60   Input ~ 0
-RXD
-$Comp
-L R R128
-U 1 1 58A63E4D
-P 4150 2450
-F 0 "R128" V 4150 2350 50  0000 L CNN
-F 1 "10k" V 4050 2450 50  0000 L CNN
-F 2 "Resistors_SMD:R_0603_HandSoldering" V 4080 2450 50  0001 C CNN
-F 3 "" H 4150 2450 50  0000 C CNN
-	1    4150 2450
-	1    0    0    1
-$EndComp
-Text GLabel 6250 2850 2    60   Input ~ 0
-B_RXD
+	0    1    1    0
+$EndComp
 $Comp
 L R R131
@@
 $EndComp
 $Comp
-L GND #PWR40
+L GND #PWR0146
 U 1 1 58D16B99
 P 7100 4350
-F 0 "#PWR40" H 7100 4100 50  0001 C CNN
+F 0 "#PWR0146" H 7100 4100 50  0001 C CNN
 F 1 "GND" V 7100 4150 50  0000 C CNN
 F 2 "" H 7100 4350 50  0000 C CNN
@@
 $EndComp
 $Comp
-L GND #PWR42
+L GND #PWR0147
 U 1 1 58D18823
 P 7200 4350
-F 0 "#PWR42" H 7200 4100 50  0001 C CNN
+F 0 "#PWR0147" H 7200 4100 50  0001 C CNN
 F 1 "GND" V 7200 4150 50  0000 C CNN
 F 2 "" H 7200 4350 50  0000 C CNN
@@
 $EndComp
 $Comp
-L GND #PWR43
+L GND #PWR0148
 U 1 1 58D188C1
 P 7300 4350
-F 0 "#PWR43" H 7300 4100 50  0001 C CNN
+F 0 "#PWR0148" H 7300 4100 50  0001 C CNN
 F 1 "GND" V 7300 4150 50  0000 C CNN
 F 2 "" H 7300 4350 50  0000 C CNN
@@
 $EndComp
 $Comp
-L GND #PWR45
+L GND #PWR0149
 U 1 1 58D188CD
 P 7400 4350
-F 0 "#PWR45" H 7400 4100 50  0001 C CNN
+F 0 "#PWR0149" H 7400 4100 50  0001 C CNN
 F 1 "GND" V 7400 4150 50  0000 C CNN
 F 2 "" H 7400 4350 50  0000 C CNN
@@
 $EndComp
 $Comp
-L GND #PWR46
+L GND #PWR0150
 U 1 1 58D1A73B
 P 7500 4350
-F 0 "#PWR46" H 7500 4100 50  0001 C CNN
+F 0 "#PWR0150" H 7500 4100 50  0001 C CNN
 F 1 "GND" V 7500 4150 50  0000 C CNN
 F 2 "" H 7500 4350 50  0000 C CNN
@@
 Wire Wire Line
 	6850 3250 7800 3250
-Wire Wire Line
-	6900 2850 6900 3150
 Connection ~ 6800 4000
 Connection ~ 6800 2750
@@
 	5800 3450 5850 3450
 Wire Wire Line
-	4300 3050 4250 3050
-Wire Wire Line
-	4250 3050 4250 2950
-Connection ~ 4250 2950
+	3850 3050 4300 3050
 Wire Wire Line
 	6150 3150 6850 3150
@@
 	5850 3150 5700 3150
 Wire Wire Line
-	4300 3150 4050 3150
-Wire Wire Line
-	4050 3150 4050 2650
-Connection ~ 4050 2650
+	3750 3150 4300 3150
 Wire Wire Line
 	5700 4000 5700 3350
-Wire Wire Line
-	6900 2850 7800 2850
 Wire Wire Line
 	4400 2300 4400 2350
 Connection ~ 4750 2000
 Wire Wire Line
-	6600 3550 7800 3550
+	6200 3550 7800 3550
 Connection ~ 4400 2000
 Wire Wire Line
@@
 Connection ~ 6800 3550
 Wire Wire Line
-	6200 3550 6300 3550
-Wire Wire Line
-	6250 3700 6250 3550
-Connection ~ 6250 3550
-Wire Wire Line
 	5900 3550 5600 3550
-Wire Wire Line
-	5700 2850 6250 2850
-Wire Wire Line
-	4150 2300 4150 2000
-Connection ~ 4150 2000
-Wire Wire Line
-	4150 2600 4150 2850
-Connection ~ 4150 2850
 Wire Wire Line
 	5600 3550 5600 3600
@@
 $EndComp
 $Comp
-L GND #PWR48
+L GND #PWR0151
 U 1 1 58D1C151
 P 7600 4350
-F 0 "#PWR48" H 7600 4100 50  0001 C CNN
+F 0 "#PWR0151" H 7600 4100 50  0001 C CNN
 F 1 "GND" V 7600 4150 50  0000 C CNN
 F 2 "" H 7600 4350 50  0000 C CNN
@@
 Text Notes 7750 5450 1    60   ~ 0
 Terminators for long line end
+Text GLabel 3850 3050 0    60   Input ~ 0
+P_PWCLK_P
+Text GLabel 3750 3150 0    60   Input ~ 0
+P_ROW_CLK
+$Comp
+L TEST_1P W5
+U 1 1 59AD03CB
+P 6800 2850
+F 0 "W5" V 6850 2900 50  0000 C CNN
+F 1 "TEST_1P" V 6904 2924 50  0001 C CNN
+F 2 "Measurement_Points:Measurement_Point_Round-SMD-Pad_Small" H 7000 2850 50  0001 C CNN
+F 3 "" H 7000 2850 50  0000 C CNN
+	1    6800 2850
+	0    -1   -1   0
+$EndComp
+Wire Wire Line
+	6900 2850 6900 3150
+Connection ~ 6800 2850
+Text GLabel 3850 2850 0    60   Input ~ 0
+P_ROW_DAT
+Wire Wire Line
+	6050 4500 5600 4500
+NoConn ~ 5600 4500
+Text GLabel 3250 2000 0    60   Input ~ 0
+LED1642VDD
+$Comp
+L R R17
+U 1 1 59B20363
+P 6000 2850
+F 0 "R17" V 6000 2750 50  0000 L CNN
+F 1 "10R" V 6050 2550 50  0000 L CNN
+F 2 "Resistors_SMD:R_0603_HandSoldering" V 5930 2850 50  0001 C CNN
+F 3 "" H 6000 2850 50  0000 C CNN
+	1    6000 2850
+	0    -1   -1   0
+$EndComp
+Wire Wire Line
+	5700 2850 5850 2850
+Wire Wire Line
+	6150 2850 6900 2850
 $EndSCHEMATC

Commit message: Removed termination resisters (was never used in 3.0 series); Pattern improvements; DRC clear
Parts:
- removed R131, R132, R133, R134, R135, R136: 120R DNI, Resistors_SMD:R_0603_HandSoldering, symbol R
Connections:
- wire segments 52 -> 46
Other:
- note removed: "Terminators for long line end"
Changed lines of the file:
@@
-EESchema Schematic File Version 2
+EESchema Schematic File Version 3
 LIBS:power
 LIBS:device
@@
 	0    1    1    0
 $EndComp
-$Comp
-L R R131
-U 1 1 58D14E13
-P 7100 4200
-F 0 "R131" V 7100 4100 50  0000 L CNN
-F 1 "120R DNI" V 7100 3350 50  0000 L CNN
-F 2 "Resistors_SMD:R_0603_HandSoldering" V 7030 4200 50  0001 C CNN
-F 3 "" H 7100 4200 50  0000 C CNN
-	1    7100 4200
-	1    0    0    -1
-$EndComp
-$Comp
-L GND #PWR144
-U 1 1 58D16B99
-P 7100 4350
-F 0 "#PWR144" H 7100 4100 50  0001 C CNN
-F 1 "GND" V 7100 4150 50  0000 C CNN
-F 2 "" H 7100 4350 50  0000 C CNN
-F 3 "" H 7100 4350 50  0000 C CNN
-	1    7100 4350
-	1    0    0    -1
-$EndComp
-$Comp
-L R R132
-U 1 1 58D1881D
-P 7200 4200
-F 0 "R132" V 7200 4100 50  0000 L CNN
-F 1 "120R DNI" V 7200 3350 50  0000 L CNN
-F 2 "Resistors_SMD:R_0603_HandSoldering" V 7130 4200 50  0001 C CNN
-F 3 "" H 7200 4200 50  0000 C CNN
-	1    7200 4200
-	1    0    0    -1
-$EndComp
-$Comp
-L GND #PWR145
-U 1 1 58D18823
-P 7200 4350
-F 0 "#PWR145" H 7200 4100 50  0001 C CNN
-F 1 "GND" V 7200 4150 50  0000 C CNN
-F 2 "" H 7200 4350 50  0000 C CNN
-F 3 "" H 7200 4350 50  0000 C CNN
-	1    7200 4350
-	1    0    0    -1
-$EndComp
-$Comp
-L R R133
-U 1 1 58D188BB
-P 7300 4200
-F 0 "R133" V 7300 4100 50  0000 L CNN
-F 1 "120R DNI" V 7300 3350 50  0000 L CNN
-F 2 "Resistors_SMD:R_0603_HandSoldering" V 7230 4200 50  0001 C CNN
-F 3 "" H 7300 4200 50  0000 C CNN
-	1    7300 4200
-	1    0    0    -1
-$EndComp
-$Comp
-L GND #PWR146
-U 1 1 58D188C1
-P 7300 4350
-F 0 "#PWR146" H 7300 4100 50  0001 C CNN
-F 1 "GND" V 7300 4150 50  0000 C CNN
-F 2 "" H 7300 4350 50  0000 C CNN
-F 3 "" H 7300 4350 50  0000 C CNN
-	1    7300 4350
-	1    0    0    -1
-$EndComp
-$Comp
-L R R134
-U 1 1 58D188C7
-P 7400 4200
-F 0 "R134" V 7400 4100 50  0000 L CNN
-F 1 "120R DNI" V 7400 3350 50  0000 L CNN
-F 2 "Resistors_SMD:R_0603_HandSoldering" V 7330 4200 50  0001 C CNN
-F 3 "" H 7400 4200 50  0000 C CNN
-	1    7400 4200
-	1    0    0    -1
-$EndComp
-$Comp
-L GND #PWR147
-U 1 1 58D188CD
-P 7400 4350
-F 0 "#PWR147" H 7400 4100 50  0001 C CNN
-F 1 "GND" V 7400 4150 50  0000 C CNN
-F 2 "" H 7400 4350 50  0000 C CNN
-F 3 "" H 7400 4350 50  0000 C CNN
-	1    7400 4350
-	1    0    0    -1
-$EndComp
-$Comp
-L R R135
-U 1 1 58D1A735
-P 7500 4200
-F 0 "R135" V 7500 4100 50  0000 L CNN
-F 1 "120R DNI" V 7500 3350 50  0000 L CNN
-F 2 "Resistors_SMD:R_0603_HandSoldering" V 7430 4200 50  0001 C CNN
-F 3 "" H 7500 4200 50  0000 C CNN
-	1    7500 4200
-	1    0    0    -1
-$EndComp
-$Comp
-L GND #PWR148
-U 1 1 58D1A73B
-P 7500 4350
-F 0 "#PWR148" H 7500 4100 50  0001 C CNN
-F 1 "GND" V 7500 4150 50  0000 C CNN
-F 2 "" H 7500 4350 50  0000 C CNN
-F 3 "" H 7500 4350 50  0000 C CNN
-	1    7500 4350
-	1    0    0    -1
-$EndComp
 Wire Wire Line
 	6900 3150 7800 3150
@@
 Wire Wire Line
 	5600 3550 5600 3600
-Wire Wire Line
-	7100 4050 7100 2650
-Wire Wire Line
-	7200 4050 7200 2750
-Wire Wire Line
-	7300 2950 7300 4050
-Wire Wire Line
-	7400 3050 7400 4050
-Wire Wire Line
-	7500 3250 7500 4050
-$Comp
-L R R136
-U 1 1 58D1C14B
-P 7600 4200
-F 0 "R136" V 7600 4100 50  0000 L CNN
-F 1 "120R DNI" V 7600 3350 50  0000 L CNN
-F 2 "Resistors_SMD:R_0603_HandSoldering" V 7530 4200 50  0001 C CNN
-F 3 "" H 7600 4200 50  0000 C CNN
-	1    7600 4200
-	1    0    0    -1
-$EndComp
-$Comp
-L GND #PWR149
-U 1 1 58D1C151
-P 7600 4350
-F 0 "#PWR149" H 7600 4100 50  0001 C CNN
-F 1 "GND" V 7600 4150 50  0000 C CNN
-F 2 "" H 7600 4350 50  0000 C CNN
-F 3 "" H 7600 4350 50  0000 C CNN
-	1    7600 4350
-	1    0    0    -1
-$EndComp
-Wire Wire Line
-	7600 4050 7600 3450
-Connection ~ 7600 3450
-Connection ~ 7500 3250
-Connection ~ 7400 3050
-Connection ~ 7300 2950
-Connection ~ 7200 2750
-Connection ~ 7100 2650
-Text Notes 7750 5450 1    60   ~ 0
-Terminators for long line end
 Text GLabel 3850 3050 0    60   Input ~ 0
 P_PWCLK_P

Commit message: This is the MazoClock hw 4.0 series; Uses ESP32 processor instead of ESP8266 used in prior MazoClock hw 3.0 series.
Parts:
- removed R121: 22k, Resistors_SMD:R_0603_HandSoldering, symbol R
- removed W4, W5, W9: TEST_1P, Measurement_Points:Measurement_Point_Round-SMD-Pad_Small, symbol TEST_1P
- added J6: Conn_01x10_Female, Pin_Headers:Pin_Header_Straight_1x10_Pitch2.54mm, symbol Conn_01x10_Female
- added R15, R16, R26, R27, R34: 22k, Resistors_SMD:R_0603_HandSoldering, symbol R
- R17: value 10R -> 22k
Connections:
- net labels added: D_COLCLK, D_COLLATCH, D_COLSER, D_LED1642_RST, D_PWCLK_N, D_PWCLK_P, D_ROW_CLK, D_ROW_LAT
- net labels removed: E_BUTTONSENSE, E_COLCLK, E_COLLATCH, E_COLSER, P_PWCLK_N, P_PWCLK_P, P_ROW_CLK, P_ROW_DAT, P_ROW_LAT
- wire segments 46 -> 60

Commit message: Added quick-and-dirty class-D amplifier circuit for just testing
Parts:
- added C73, C74, C75, C76, C77, C78, C79, C95: 0.1u, Capacitors_ThroughHole:C_Disc_D3.8mm_W2.6mm_P2.50mm, symbol C
- added C96, C97, C98: 1u, Capacitors_SMD:C_0603_HandSoldering, symbol C
- added J14, J15: Audio-Jack-3, components:MJ-8435, symbol Audio-Jack-3
- added L10, L11, L8, L9: L, Choke_Axial_ThroughHole:Choke_Horizontal_RM10mm, symbol L
- added R51, R52, R54, R55, R57, R74: 22k, Resistors_SMD:R_0603_HandSoldering, symbol R
- added R53, R56: 22k, Resistors_ThroughHole:R_Axial_DIN0204_L3.6mm_D1.6mm_P7.62mm_Horizontal, symbol R
- added U23: LMV393, Housings_SSOP:MSOP-8_3x3mm_Pitch0.65mm, symbol LMV393
- added U24, U25: 74VHC541, components:SOIC-20-0.65mm-w8.0mm, symbol 74HCT541_PWR
Connections:
- net labels added: VCC
- wire segments 60 -> 138

Commit message: Updated to kicad 6.0.0 rc; removed outdated gerber files; Schematic is not complete
Parts:
- removed C73, C74, C75, C76, C77, C78, C79, C95: 0.1u, Capacitors_ThroughHole:C_Disc_D3.8mm_W2.6mm_P2.50mm, symbol C
- removed C96, C97, C98: 1u, Capacitors_SMD:C_0603_HandSoldering, symbol C
- removed J14, J15: Audio-Jack-3, components:MJ-8435, symbol Audio-Jack-3
- removed L10, L11, L8, L9: L, Choke_Axial_ThroughHole:Choke_Horizontal_RM10mm, symbol L
- removed R51, R52, R54, R55, R57, R74: 22k, Resistors_SMD:R_0603_HandSoldering, symbol R
- removed R53, R56: 22k, Resistors_ThroughHole:R_Axial_DIN0204_L3.6mm_D1.6mm_P7.62mm_Horizontal, symbol R
- removed U23: LMV393, Housings_SSOP:MSOP-8_3x3mm_Pitch0.65mm, symbol LMV393
- removed U24, U25: 74VHC541, components:SOIC-20-0.65mm-w8.0mm, symbol 74HCT541_PWR
- C55, C62, C70: symbol C -> device:C
- J6: symbol Conn_01x10_Female -> Connector:Conn_01x10_Female
- L3: symbol Ferrite_Bead_Small -> device:Ferrite_Bead_Small
- R114, R115, R116, R117, R118, R119, R120, R15, R16, R17, R26, R27, R34: symbol R -> device:R
- U2: symbol 74HCT541_PWR -> Logic_74xx:74LS541
- W1, W11, W2, W3, W7: symbol TEST_1P -> Connector:Test_Point
Connections:
- net labels removed: VCC
- wire segments 138 -> 76
