File: dotmatrix_64x48.sch (KiCad schematic (older format))
At the start: 40 parts, among them P3 CONN_01X06, Q2 Q_NPN_BEC, Q4 Q_NPN_BEC, SW1 SW_PUSH_SMALL_H, SW2 SW_PUSH_SMALL_H, U1 WROOM-02

Commit message: Modified to use matrix LEDs; Components layout has almost done, tracks and traces not yet.
Parts:
- removed R17: 120R, Resistors_SMD:R_0603_HandSoldering, symbol R
- added C88, C90, C91: 0.1u, Capacitors_SMD:C_0603_HandSoldering, symbol C
- added C89: 1u, Capacitors_SMD:C_0603_HandSoldering, symbol C
- added C92: 10u, Capacitors_SMD:C_0805_HandSoldering, symbol C
- added C93, C94: 22p, Capacitors_SMD:C_0603_HandSoldering, symbol C
- added CONN4: USB_OTG, components:USB-MICRO-B-RECEPT-UNIVERSAL, symbol USB_OTG
- added J1: CONN_01X04, Pin_Headers:Pin_Header_Straight_1x04_Pitch2.54mm, symbol CONN_01X04
- added J2: CONN_01X05, Pin_Headers:Pin_Header_Straight_1x05_Pitch2.54mm, symbol CONN_01X05
- added JP1, JP2, JP3, JP4, JP5: Jumper_NC_Small, components:SolderJumper, symbol Jumper_NC_Small
- added L5: BLM18RK102SN1 1k @ 100MHz, Resistors_SMD:R_0603_HandSoldering, symbol Ferrite_Bead_Small
- added R126, R127, R137, R138, R139, R140, R141: 120R, Resistors_SMD:R_0603_HandSoldering, symbol R
- added R130: 10R, Resistors_SMD:R_0603_HandSoldering, symbol R
- added R142, R143, R144, R145: 22k, Resistors_SMD:R_0603_HandSoldering, symbol R
- added U19: PIC32MX220F032B-I/ML, components:QFN-28-1EP_6x6mm_Pitch0.65mm_Handsoldering, symbol PIC32MX220F032B-I/ML
- added Y1: 8MHz, components:Crystal_SMD_HC49-SD_and_MA506_HandSoldering_mod, symbol Crystal_Small
- R13: value 120R -> 4.7k
- R16: value 1k -> 10k
Connections:
- net labels added: E_MCLR, E_PGEC, E_PGED, PIC_VDD, P_ESP_GPIO0, P_ESP_RST, P_LED1642_RST, P_MCLR, P_PGEC, P_PGED, P_PWCLK_N, P_PWCLK_P, P_ROW_CLK, P_ROW_DAT, P_ROW_LAT, P_RX, P_SYNC, P_TX, USB_D_N, USB_D_P, USB_VBUS, VCAP
- net labels removed: B_RXD, E_HC595LATCH, E_PWCLK, GPIO0_BTN, RST, RXD, TXD
- wire segments 88 -> 151
- no-connect marks 1 -> 5
Other:
- note added: "HW revision strip"

Commit message: Added serial pull-ups; DRC clear; Silks should be clear.
Parts:
- added R38, R39: 22k, Resistors_SMD:R_0603_HandSoldering, symbol R
Connections:
- wire segments 151 -> 158
Changed lines of the file:
@@
 $EndComp
 $Comp
-L GND #PWR011
+L GND #PWR11
 U 1 1 57A04933
 P 2500 2300
-F 0 "#PWR011" H 2500 2050 50  0001 C CNN
+F 0 "#PWR11" H 2500 2050 50  0001 C CNN
 F 1 "GND" H 2505 2127 50  0000 C CNN
 F 2 "" H 2500 2300 50  0000 C CNN
@@
 $EndComp
 $Comp
-L GND #PWR09
+L GND #PWR9
 U 1 1 57A049CA
 P 5100 1900
-F 0 "#PWR09" H 5100 1650 50  0001 C CNN
+F 0 "#PWR9" H 5100 1650 50  0001 C CNN
 F 1 "GND" H 5105 1727 50  0000 C CNN
 F 2 "" H 5100 1900 50  0000 C CNN
@@
 $EndComp
 $Comp
-L GND #PWR014
+L GND #PWR14
 U 1 1 57A08E43
 P 3050 3200
-F 0 "#PWR014" H 3050 2950 50  0001 C CNN
+F 0 "#PWR14" H 3050 2950 50  0001 C CNN
 F 1 "GND" H 3055 3027 50  0000 C CNN
 F 2 "" H 3050 3200 50  0000 C CNN
@@
 $EndComp
 $Comp
-L GND #PWR08
+L GND #PWR8
 U 1 1 57A0D69E
 P 5950 1700
-F 0 "#PWR08" H 5950 1450 50  0001 C CNN
+F 0 "#PWR8" H 5950 1450 50  0001 C CNN
 F 1 "GND" H 6050 1600 50  0000 C CNN
 F 2 "" H 5950 1700 50  0000 C CNN
@@
 $EndComp
 $Comp
-L GND #PWR02
+L GND #PWR2
 U 1 1 57BEEBBA
 P 1500 1100
-F 0 "#PWR02" H 1500 850 50  0001 C CNN
+F 0 "#PWR2" H 1500 850 50  0001 C CNN
 F 1 "GND" H 1505 927 50  0000 C CNN
 F 2 "" H 1500 1100 50  0000 C CNN
@@
 E_AIN
 $Comp
-L GND #PWR06
+L GND #PWR6
 U 1 1 5807ECB9
 P 5100 1400
-F 0 "#PWR06" H 5100 1150 50  0001 C CNN
+F 0 "#PWR6" H 5100 1150 50  0001 C CNN
 F 1 "GND" H 5105 1227 50  0000 C CNN
 F 2 "" H 5100 1400 50  0000 C CNN
@@
 $EndComp
 $Comp
-L GND #PWR013
+L GND #PWR13
 U 1 1 58084DAB
 P 3200 2700
-F 0 "#PWR013" H 3200 2450 50  0001 C CNN
+F 0 "#PWR13" H 3200 2450 50  0001 C CNN
 F 1 "GND" H 3205 2527 50  0000 C CNN
 F 2 "" H 3200 2700 50  0000 C CNN
@@
 $EndComp
 $Comp
-L GND #PWR012
+L GND #PWR12
 U 1 1 580E1127
 P 1600 2650
-F 0 "#PWR012" H 1600 2400 50  0001 C CNN
+F 0 "#PWR12" H 1600 2400 50  0001 C CNN
 F 1 "GND" H 1605 2477 50  0000 C CNN
 F 2 "" H 1600 2650 50  0000 C CNN
@@
 $EndComp
 $Comp
-L GND #PWR03
+L GND #PWR3
 U 1 1 582D864D
 P 1900 1100
-F 0 "#PWR03" H 1900 850 50  0001 C CNN
+F 0 "#PWR3" H 1900 850 50  0001 C CNN
 F 1 "GND" H 1905 927 50  0000 C CNN
 F 2 "" H 1900 1100 50  0000 C CNN
@@
 $EndComp
 $Comp
-L GND #PWR05
+L GND #PWR5
 U 1 1 5833CED3
 P 2100 1200
-F 0 "#PWR05" H 2100 950 50  0001 C CNN
+F 0 "#PWR5" H 2100 950 50  0001 C CNN
 F 1 "GND" H 2105 1027 50  0000 C CNN
 F 2 "" H 2100 1200 50  0000 C CNN
@@
 $EndComp
 $Comp
-L GND #PWR01
+L GND #PWR1
 U 1 1 583D4F7D
 P 1100 1100
-F 0 "#PWR01" H 1100 850 50  0001 C CNN
+F 0 "#PWR1" H 1100 850 50  0001 C CNN
 F 1 "GND" H 1105 927 50  0000 C CNN
 F 2 "" H 1100 1100 50  0000 C CNN
@@
 $EndComp
 $Comp
-L GND #PWR026
+L GND #PWR26
 U 1 1 585A447B
 P 4750 7550
-F 0 "#PWR026" H 4750 7300 50  0001 C CNN
+F 0 "#PWR26" H 4750 7300 50  0001 C CNN
 F 1 "GND" H 4755 7377 50  0000 C CNN
 F 2 "" H 4750 7550 50  0000 C CNN
@@
 $EndComp
 $Comp
-L GND #PWR023
+L GND #PWR23
 U 1 1 59AAE886
 P 2850 6000
-F 0 "#PWR023" H 2850 5750 50  0001 C CNN
+F 0 "#PWR23" H 2850 5750 50  0001 C CNN
 F 1 "GND" H 2855 5827 50  0000 C CNN
 F 2 "" H 2850 6000 50  0000 C CNN
@@
 $EndComp
 $Comp
-L GND #PWR015
+L GND #PWR15
 U 1 1 59AB0C0F
 P 2800 3650
-F 0 "#PWR015" H 2800 3400 50  0001 C CNN
+F 0 "#PWR15" H 2800 3400 50  0001 C CNN
 F 1 "GND" H 2805 3477 50  0000 C CNN
 F 2 "" H 2800 3650 50  0000 C CNN
@@
 $EndComp
 $Comp
-L GND #PWR019
+L GND #PWR19
 U 1 1 59AB1D31
 P 1450 4550
-F 0 "#PWR019" H 1450 4300 50  0001 C CNN
+F 0 "#PWR19" H 1450 4300 50  0001 C CNN
 F 1 "GND" H 1455 4377 50  0000 C CNN
 F 2 "" H 1450 4550 50  0000 C CNN
@@
 $EndComp
 $Comp
-L GND #PWR017
+L GND #PWR17
 U 1 1 59AB2186
 P 1050 4550
-F 0 "#PWR017" H 1050 4300 50  0001 C CNN
+F 0 "#PWR17" H 1050 4300 50  0001 C CNN
 F 1 "GND" H 1055 4377 50  0000 C CNN
 F 2 "" H 1050 4550 50  0000 C CNN
@@
 $EndComp
 $Comp
-L GND #PWR020
+L GND #PWR20
 U 1 1 59AB2D04
 P 2250 4900
-F 0 "#PWR020" H 2250 4650 50  0001 C CNN
+F 0 "#PWR20" H 2250 4650 50  0001 C CNN
 F 1 "GND" H 2255 4727 50  0000 C CNN
 F 2 "" H 2250 4900 50  0000 C CNN
@@
 USB_D_N
 $Comp
-L GND #PWR025
+L GND #PWR25
 U 1 1 59AB84CF
 P 3400 7400
-F 0 "#PWR025" H 3400 7150 50  0001 C CNN
+F 0 "#PWR25" H 3400 7150 50  0001 C CNN
 F 1 "GND" H 3405 7227 50  0000 C CNN
 F 2 "" H 3400 7400 50  0000 C CNN
@@
 $EndComp
 $Comp
-L GND #PWR022
+L GND #PWR22
 U 1 1 59ABE251
 P 5400 4950
-F 0 "#PWR022" H 5400 4700 50  0001 C CNN
+F 0 "#PWR22" H 5400 4700 50  0001 C CNN
 F 1 "GND" H 5405 4777 50  0000 C CNN
 F 2 "" H 5400 4950 50  0000 C CNN
@@
 $EndComp
 $Comp
-L GND #PWR021
+L GND #PWR21
 U 1 1 59ABE2A6
 P 5050 4950
-F 0 "#PWR021" H 5050 4700 50  0001 C CNN
+F 0 "#PWR21" H 5050 4700 50  0001 C CNN
 F 1 "GND" H 5055 4777 50  0000 C CNN
 F 2 "" H 5050 4950 50  0000 C CNN
@@
 $EndComp
 $Comp
-L GND #PWR018
+L GND #PWR18
 U 1 1 59AC172F
 P 1250 4550
-F 0 "#PWR018" H 1250 4300 50  0001 C CNN
+F 0 "#PWR18" H 1250 4300 50  0001 C CNN
 F 1 "GND" H 1255 4377 50  0000 C CNN
 F 2 "" H 1250 4550 50  0000 C CNN
@@
 U 1 1 59AC7B73
 P 7350 1950
-F 0 "JP1" H 7350 2200 50  0000 C CNN
+F 0 "JP1" H 7450 1750 50  0000 C CNN
 F 1 "Jumper_NC_Small" H 7360 1890 50  0001 C CNN
 F 2 "components:SolderJumper" H 7350 1950 50  0001 C CNN
@@
 U 1 1 59AC7C3C
 P 7450 1950
-F 0 "JP2" H 7450 2200 50  0000 C CNN
+F 0 "JP2" H 7550 1750 50  0000 C CNN
 F 1 "Jumper_NC_Small" H 7460 1890 50  0001 C CNN
 F 2 "components:SolderJumper" H 7450 1950 50  0001 C CNN
@@
 NoConn ~ 7900 1950
 $Comp
-L GND #PWR010
+L GND #PWR10
 U 1 1 59ACA265
 P 7900 2050
-F 0 "#PWR010" H 7900 1800 50  0001 C CNN
+F 0 "#PWR10" H 7900 1800 50  0001 C CNN
 F 1 "GND" H 7850 1900 50  0000 C CNN
 F 2 "" H 7900 2050 50  0000 C CNN
@@
 DTR
 $Comp
-L GND #PWR04
+L GND #PWR4
 U 1 1 59A7D4FF
 P 7900 1150
-F 0 "#PWR04" H 7900 900 50  0001 C CNN
+F 0 "#PWR4" H 7900 900 50  0001 C CNN
 F 1 "GND" H 7850 1000 50  0000 C CNN
 F 2 "" H 7900 1150 50  0000 C CNN
@@
 $EndComp
 $Comp
-L GND #PWR024
+L GND #PWR24
 U 1 1 59AED967
 P 6000 6700
-F 0 "#PWR024" H 6000 6450 50  0001 C CNN
+F 0 "#PWR24" H 6000 6450 50  0001 C CNN
 F 1 "GND" H 6005 6527 50  0000 C CNN
 F 2 "" H 6000 6700 50  0000 C CNN
@@
 $EndComp
 $Comp
-L GND #PWR07
+L GND #PWR7
 U 1 1 59AF4986
 P 5200 1500
-F 0 "#PWR07" H 5200 1250 50  0001 C CNN
+F 0 "#PWR7" H 5200 1250 50  0001 C CNN
 F 1 "GND" H 5205 1327 50  0000 C CNN
 F 2 "" H 5200 1500 50  0000 C CNN
@@
 Connection ~ 7000 5150
 $Comp
-L GND #PWR016
+L GND #PWR16
 U 1 1 59B0C5EA
 P 7150 4450
-F 0 "#PWR016" H 7150 4200 50  0001 C CNN
+F 0 "#PWR16" H 7150 4200 50  0001 C CNN
 F 1 "GND" H 7155 4277 50  0000 C CNN
 F 2 "" H 7150 4450 50  0000 C CNN
@@
 Text Label 2500 4500 0    60   ~ 0
 VCAP
+$Comp
+L R R38
+U 1 1 59BE21D4
+P 7050 1100
+F 0 "R38" V 7050 1050 50  0000 L CNN
+F 1 "22k" V 7000 1200 50  0000 L CNN
+F 2 "Resistors_SMD:R_0603_HandSoldering" V 6980 1100 50  0001 C CNN
+F 3 "" H 7050 1100 50  0000 C CNN
+	1    7050 1100
+	-1   0    0    1
+$EndComp
+$Comp
+L R R39
+U 1 1 59BE310E
+P 7050 1700
+F 0 "R39" V 7050 1650 50  0000 L CNN
+F 1 "22k" V 7000 1800 50  0000 L CNN
+F 2 "Resistors_SMD:R_0603_HandSoldering" V 6980 1700 50  0001 C CNN
+F 3 "" H 7050 1700 50  0000 C CNN
+	1    7050 1700
+	-1   0    0    1
+$EndComp
+Text GLabel 6950 900  1    60   Input ~ 0
+ESPVDD
+Wire Wire Line
+	6950 900  6950 1550
+Wire Wire Line
+	6950 950  7050 950
+Wire Wire Line
+	7050 1250 7050 1450
+Wire Wire Line
+	7050 1450 7450 1450
+Connection ~ 7450 1450
+Wire Wire Line
+	7350 2100 7050 2100
+Wire Wire Line
+	7050 2100 7050 1850
+Connection ~ 7350 2100
+Wire Wire Line
+	6950 1550 7050 1550
+Connection ~ 6950 950
 $EndSCHEMATC

Commit message: Layout improvements; DRC clear
Connections:
- net labels removed: LEDLOGICVDD
Changed lines of the file:
@@
 	1    0    0    -1
 $EndComp
-Text GLabel 4750 6900 0    60   Input ~ 0
-LEDLOGICVDD
 Text GLabel 2050 2100 0    60   Input ~ 0
 E_SDA
@@
 	6950 1550 7050 1550
 Connection ~ 6950 950
+Text GLabel 4750 6900 0    60   Input ~ 0
+ESPVDD
 $EndSCHEMATC

Commit message: This is the MazoClock hw 4.0 series; Uses ESP32 processor instead of ESP8266 used in prior MazoClock hw 3.0 series.
Parts:
- removed C35, C69: 1u, Capacitors_SMD:C_0603_HandSoldering, symbol C
- removed C61: 0.1u, Capacitors_SMD:C_0603_HandSoldering, symbol C
- removed D10, D8: Led_Small, components:LED1608_Handsoldering, symbol LED_Small
- removed J1: CONN_01X04, Pin_Headers:Pin_Header_Straight_1x04_Pitch2.54mm, symbol CONN_01X04
- removed L4, L7: BLM18RK102SN1 1k @ 100MHz, Resistors_SMD:R_0603_HandSoldering, symbol Ferrite_Bead_Small
- removed P3: CONN_01X06, Pin_Headers:Pin_Header_Straight_1x08_Pitch2.54mm, symbol CONN_01X08
- removed R122, R27: 4.7k, Resistors_SMD:R_0603_HandSoldering, symbol R
- removed R126, R127, R15, R26, R46, R52: 120R, Resistors_SMD:R_0603_HandSoldering, symbol R
- removed R142, R143, R144, R145, R38, R39: 22k, Resistors_SMD:R_0603_HandSoldering, symbol R
- removed R16, R34, R54, R55: 10k, Resistors_SMD:R_0603_HandSoldering, symbol R
- removed R48: 1k, Resistors_SMD:R_0603_HandSoldering, symbol R
- removed SW1, SW2: SW_PUSH_SMALL_H, components:TACT-SW-4P, symbol SW_Push
- removed U1: WROOM-02, components:WROOM-02, symbol WROOM-02
- added J1, J3: Conn_01x19_Female, Pin_Headers:Pin_Header_Straight_1x19_Pitch2.54mm, symbol Conn_01x19_Female
- added J4: Conn_01x14_Female, Pin_Headers:Pin_Header_Straight_1x14_Pitch2.54mm, symbol Conn_01x14_Female
- added J5: Conn_01x10_Female, Pin_Headers:Pin_Header_Straight_1x10_Pitch2.54mm, symbol Conn_01x10_Female
- added J7: Conn_01x03_Female, Pin_Headers:Pin_Header_Straight_1x03_Pitch2.54mm, symbol Conn_01x03_Female
- added J8: Conn_01x08_Female, Pin_Headers:Pin_Header_Straight_1x08_Pitch2.54mm, symbol Conn_01x08_Female
- added JP10, JP11, JP12, JP6, JP7, JP8, JP9: Jumper_NC_Small, components:SolderJumper, symbol Jumper_NC_Small
- added U1: ESP32-DEVKIT-C, components:ESP32-DEVKIT-C, symbol ESP32-DEVKIT-C
- added U16: ESP32-WROOM, components:ESP32-WROOM-AND-SIDE-PINS, symbol ESP32-WROOM
- R1: value 120R -> 22k
- R10, R9: value 22k -> 4.7k
- R14, R7: value 120R -> 10k
- R5: value 10k -> 120R
- R8: value 4.7k -> 22k
Connections:
- net labels added: BUTTONSENSE, D_COLCLK, D_COLLATCH, D_COLSER, D_LED1642_RST, D_PWCLK_P, D_ROW_LAT, E_EN, E_GPIO0, E_RX, E_TX, HC595SEROUT, LEDLOGICVDD, P_BUTTON_SENSE, P_PWCLK, P_SER_CLK, P_SER_DAT, P_SER_HC595_LAT, P_SER_LED1642_LAT, P_SER_RET, P_SPI_CLK, P_SPI_SDI, P_SPI_SDO, VCC
- net labels removed: E_AIN, E_BUTTONSENSE, E_COLCLK, E_COLLATCH, E_COLSER, E_MCLR, E_PGEC, E_PGED, E_RXD, E_SCL, E_SDA, E_TXD, FILTVDD, IR_IN, IR_OUT, P_PWCLK_N, P_PWCLK_P, P_ROW_CLK, P_ROW_DAT, P_ROW_LAT, P_SYNC
- wire segments 158 -> 242
- no-connect marks 5 -> 3
Other:
- note removed: "HW revision strip"

Commit message: Updated to kicad 6.0.0 rc; removed outdated gerber files; Schematic is not complete
Parts:
- removed C88, C90, C91: 0.1u, Capacitors_SMD:C_0603_HandSoldering, symbol C
- removed C89: 1u, Capacitors_SMD:C_0603_HandSoldering, symbol C
- removed C92: 10u, Capacitors_SMD:C_0805_HandSoldering, symbol C
- removed C93, C94: 22p, Capacitors_SMD:C_0603_HandSoldering, symbol C
- removed CONN4: USB_OTG, components:USB-MICRO-B-RECEPT-UNIVERSAL, symbol USB_OTG
- removed D11, D13: D_Schottky_Small, components:SOD-523-mod, symbol D_Schottky_Small
- removed J2: CONN_01X05, Pin_Headers:Pin_Header_Straight_1x05_Pitch2.54mm, symbol CONN_01X05
- removed L5: BLM18RK102SN1 1k @ 100MHz, Resistors_SMD:R_0603_HandSoldering, symbol Ferrite_Bead_Small
- removed R1, R8: 22k, Resistors_SMD:R_0603_HandSoldering, symbol R
- removed R13: 4.7k, Resistors_SMD:R_0603_HandSoldering, symbol R
- removed R130: 10R, Resistors_SMD:R_0603_HandSoldering, symbol R
- removed R137, R138, R139, R140, R141, R2, R3, R4, R5, R6: 120R, Resistors_SMD:R_0603_HandSoldering, symbol R
- removed R7: 10k, Resistors_SMD:R_0603_HandSoldering, symbol R
- removed U19: PIC32MX220F032B-I/ML, components:QFN-28-1EP_6x6mm_Pitch0.65mm_Handsoldering, symbol PIC32MX220F032B-I/ML
- removed Y1: 8MHz, components:Crystal_SMD_HC49-SD_and_MA506_HandSoldering_mod, symbol Crystal_Small
- J1, J3: symbol Conn_01x19_Female -> Connector:Conn_01x19_Female
- J4: symbol Conn_01x14_Female -> Connector:Conn_01x14_Female
- J5: symbol Conn_01x10_Female -> Connector:Conn_01x10_Female
- J7: symbol Conn_01x03_Female -> Connector:Conn_01x03_Female
- J8: symbol Conn_01x08_Female -> Connector:Conn_01x08_Female
- JP1, JP10, JP11, JP12, JP2, JP3, JP4, JP5, JP6, JP7, JP8, JP9: symbol Jumper_NC_Small -> device:Jumper_NC_Small
- Q2, Q4: symbol Q_NPN_BEC -> device:Q_NPN_BEC
- R10, R11, R14, R9: symbol R -> device:R
- U1: symbol ESP32-DEVKIT-C -> DeeComponents:ESP32-DEVKIT-C
- U16: symbol ESP32-WROOM -> DeeComponents:ESP32-WROOM
Connections:
- net labels removed: PIC_VDD, USB_D_N, USB_D_P, USB_VBUS, VCAP
- wire segments 242 -> 189

Commit message: Heavily modifying; Matrix nets under construction
Parts:
- removed J1, J3: Conn_01x19_Female, Pin_Headers:Pin_Header_Straight_1x19_Pitch2.54mm, symbol Connector:Conn_01x19_Female
- removed J4: Conn_01x14_Female, Pin_Headers:Pin_Header_Straight_1x14_Pitch2.54mm, symbol Connector:Conn_01x14_Female
- removed J5: Conn_01x10_Female, Pin_Headers:Pin_Header_Straight_1x10_Pitch2.54mm, symbol Connector:Conn_01x10_Female
- removed J8: Conn_01x08_Female, Pin_Headers:Pin_Header_Straight_1x08_Pitch2.54mm, symbol Connector:Conn_01x08_Female
- removed JP1, JP10, JP11, JP12, JP2, JP3, JP4, JP5, JP6, JP7, JP8, JP9: Jumper_NC_Small, components:SolderJumper, symbol device:Jumper_NC_Small
- removed U1: ESP32-DEVKIT-C, components:ESP32-DEVKIT-C, symbol DeeComponents:ESP32-DEVKIT-C
- added C21, C23, C77: 0.1u, Capacitors_SMD:C_0603_HandSoldering, symbol device:C
- added C22: 1u, Capacitors_SMD:C_0603_HandSoldering, symbol device:C
- added L3: BLM18RK102SN1 1k @ 100MHz, Resistors_SMD:R_0603_HandSoldering, symbol device:Ferrite_Bead_Small
- added P1: CONN_01X06, Pin_Headers:Pin_Header_Straight_1x08_Pitch2.54mm, symbol Connector:Conn_01x06
- added P3, P4: CONN_01X08, Pin_Headers:Pin_Header_Straight_1x08_Pitch2.54mm, symbol Connector:Conn_01x08
- added R118, R122, R125, R126, R127, R3: 10k, Resistors_SMD:R_0603_HandSoldering, symbol device:R
- added R119, R120, R121, R128, R13, R130, R131, R132, R15, R27, R4, R41, R46, R48, R49, R51, R52, R53, R54, R55, R56, R57, R6, R7, R76, R8: 120R, Resistors_SMD:R_0603_HandSoldering, symbol device:R
- added R133, R134, R135, R136, R77, R78, R80, R81: 0, components:SolderJumper, symbol device:R
- added R2, R5, R74, R75: 10R, Resistors_SMD:R_0603_HandSoldering, symbol device:R
- added R34: 100k, Resistors_SMD:R_0603_HandSoldering, symbol device:R
- added R79, R98: 1k, Resistors_SMD:R_0603_HandSoldering, symbol device:R
- added SW1, SW2: SW_PUSH_SMALL_H, Buttons_Switches_SMD:SW_SPST_FSMSM, symbol Switch:SW_Push
- added U1: 74VHC541, components:SOIC-20-0.65mm-w8.0mm, symbol Logic_74xx:74LS541
- added U21, U22: CM1293A-04SO, TO_SOT_Packages_SMD:SOT-23-6_Handsoldering, symbol ESD_Protection:SRV05-4
- added W1, W2, W3, W4, W7: TEST_1P, Measurement_Points:Measurement_Point_Round-SMD-Pad_Small, symbol Connector:Test_Point
- J7: value Conn_01x03_Female -> Conn_01x04_Female; footprint Pin_Headers:Pin_Header_Straight_1x03_Pitch2.54mm -> Pin_Headers:Pin_Header_Straight_1x04_Pitch2.54mm; symbol Connector:Conn_01x03_Female -> Connector:Conn_01x04_Female
- U16: footprint components:ESP32-WROOM-AND-SIDE-PINS -> components:ESP32-WROOM
Connections:
- net labels added: CC_GUARD0, CC_GUARD1, COLCLK, COLLATCH, COLSER, COLSEROUT, E_AIN, HC595CLK, HC595LATCH, HC595SER, I2S_SPK_BCLK, I2S_SPK_DATA, I2S_SPK_GAIN0, I2S_SPK_GAIN1, I2S_SPK_LRCLK, IR_IN, IR_OUT, LED1642VDD, MS_SEL, RC_GUARD0, RC_GUARD1, VSPI_MISO, VSPI_MOSI, VSPI_SCK, VSPI_SS
- net labels removed: D_PWCLK_P, LEDLOGICVDD, P_BUTTON_SENSE, P_ESP_GPIO0, P_ESP_RST, P_LED1642_RST, P_MCLR, P_PGEC, P_PGED, P_PWCLK, P_RX, P_SER_CLK, P_SER_DAT, P_SER_HC595_LAT, P_SER_LED1642_LAT, P_SER_RET, P_SPI_CLK, P_SPI_SDI, P_SPI_SDO, P_TX, VCC
- wire segments 189 -> 235
- no-connect marks 3 -> 7
Other:
- note added: "Master/Slave select"
- note added: "note: WROOM-32D has \nmodule-built-in TXD0's \nouput decoupling resistor 500R."
- note added: "strap pin: IO0 - internally PU'ed"
- note added: "strap pin: IO2 - internally PD'ed"
- note added: "strap pin: IO5 - internally PU'ed"
- note added: "strap pin: MTDI(IO12) - internally PD'ed"
- note added: "strap pin: MTDO(IO15) - internally PU'ed"
