File: dotmatrix_64x48.sch (KiCad schematic (older format))
At the start: 70 parts, among them J1 Conn_01x03_Female, J2 Conn_01x03_Male, J3 Micro_SD_Card, J7 Conn_01x04_Female, P1 CONN_01X06, Q2 Q_NPN_BEC, Q4 Q_NPN_BEC, SW1 SW_PUSH_SMALL_H, SW2 SW_PUSH_SMALL_H, U1 74VHC541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

Commit message: Fixed USB micro-b's mount polarity; Improved SOT-23-6 1-pin silk marker readability
Parts:
- U21, U22, U27: footprint TO_SOT_Packages_SMD:SOT-23-6_Handsoldering -> components:SOT-23-6_Handsoldering_mod
Changed lines of the file:
@@
 F 0 "U22" H 8950 3278 50  0000 C CNN
 F 1 "CM1293A-04SO" H 8950 3187 50  0000 C CNN
-F 2 "TO_SOT_Packages_SMD:SOT-23-6_Handsoldering" H 8950 2600 50  0001 C CNN
+F 2 "components:SOT-23-6_Handsoldering_mod" H 8950 2600 50  0001 C CNN
 F 3 "http://www.onsemi.com/pub/Collateral/SRV05-4-D.PDF" H 8950 2600 50  0001 C CNN
 	1    8950 2600
@@
 F 0 "U21" H 2700 7428 50  0000 C CNN
 F 1 "CM1293A-04SO" H 2700 7337 50  0000 C CNN
-F 2 "TO_SOT_Packages_SMD:SOT-23-6_Handsoldering" H 2700 6750 50  0001 C CNN
+F 2 "components:SOT-23-6_Handsoldering_mod" H 2700 6750 50  0001 C CNN
 F 3 "http://www.onsemi.com/pub/Collateral/SRV05-4-D.PDF" H 2700 6750 50  0001 C CNN
 	1    2700 6750
@@
 F 0 "U27" H 5450 5978 50  0000 C CNN
 F 1 "CM1293A-04SO" H 5450 5887 50  0000 C CNN
-F 2 "TO_SOT_Packages_SMD:SOT-23-6_Handsoldering" H 5450 5300 50  0001 C CNN
+F 2 "components:SOT-23-6_Handsoldering_mod" H 5450 5300 50  0001 C CNN
 F 3 "http://www.onsemi.com/pub/Collateral/SRV05-4-D.PDF" H 5450 5300 50  0001 C CNN
 	1    5450 5300

Commit message: LEDVDD now can be up to 5.0V for blue/white LEDs; DRC clear
Parts:
- removed R119: 120R, Resistor_SMD:R_0603_1608Metric_Pad1.05x0.95mm_HandSolder, symbol dotmatrix_64x48-rescue:R-device
Connections:
- net labels added: HC595SEROUT_LS
- net labels removed: HC595SEROUT
- wire segments 218 -> 217
Changed lines of the file:
@@
-$Comp
-L dotmatrix_64x48-rescue:R-device R?
-U 1 1 5BC0278A
-P 2800 1650
-AR Path="/59A8E319/5BC0278A" Ref="R?"  Part="1"
-AR Path="/5BC0278A" Ref="R119"  Part="1"
-F 0 "R119" V 2800 1550 50  0000 L CNN
-F 1 "120R" V 2850 1350 50  0000 L CNN
-F 2 "Resistor_SMD:R_0603_1608Metric_Pad1.05x0.95mm_HandSolder" V 2730 1650 50  0001 C CNN
-F 3 "" H 2800 1650 50  0000 C CNN
-	1    2800 1650
-	0    1    -1   0
-$EndComp
-Text GLabel 2400 1650 0    60   Input ~ 0
-HC595SEROUT
-Wire Wire Line
-	2950 1650 3100 1650
 $Comp
 L dotmatrix_64x48-rescue:R-device R?
@@
 	0    1    -1   0
 $EndComp
-Wire Wire Line
-	2400 1650 2650 1650
 Wire Wire Line
 	1350 1850 1500 1850
@@
 Text GLabel 5950 5400 2    60   Input ~ 0
 IR_OUT
+Text GLabel 2400 1650 0    60   Input ~ 0
+HC595SEROUT_LS
+Wire Wire Line
+	2400 1650 3100 1650
 $EndSCHEMATC

Commit message: Fixed WROOM-32D footprinco; NO DRC CHECKED
Parts:
- U16: footprint components:ESP32-WROOM -> components:ESP32-WROOM-D
Changed lines of the file:
@@
 F 0 "U16" H 3800 3150 60  0000 C CNN
 F 1 "ESP32-WROOM" H 4300 3150 60  0000 C CNN
-F 2 "components:ESP32-WROOM" H 4400 3200 60  0001 C CNN
+F 2 "components:ESP32-WROOM-D" H 4400 3200 60  0001 C CNN
 F 3 "" H 3600 2300 60  0001 C CNN
 	1    4050 1850
