File: power.sch (KiCad schematic (older format))
At the start: 26 parts, among them P6 CONN_01X03, T1 COMMON_MODE_CHOKE, U14 NJM2845DL1-33

Commit message: Modified to use matrix LEDs; Components layout has almost done, tracks and traces not yet.
Parts:
- removed H4, H5: TEST_1P, components:MountingHole_3.2mm_M3, symbol TEST_1P
Connections:
- wire segments 34 -> 33
Changed lines of the file:
@@
 $Descr A4 11693 8268
 encoding utf-8
-Sheet 10 11
+Sheet 9 10
 Title ""
 Date ""
@@
 $EndDescr
 $Comp
-L TEST_1P H4
-U 1 1 57B06654
-P 4850 1650
-F 0 "H4" H 4908 1724 50  0000 L CNN
-F 1 "TEST_1P" H 4908 1679 50  0001 L CNN
-F 2 "components:MountingHole_3.2mm_M3" H 4908 1679 50  0001 L CNN
-F 3 "" H 5050 1650 50  0000 C CNN
-	1    4850 1650
-	1    0    0    -1
-$EndComp
-$Comp
-L GND #PWR1
-U 1 1 57B05DBF
-P 3900 1650
-F 0 "#PWR1" H 3900 1400 50  0001 C CNN
-F 1 "GND" H 3900 1500 50  0000 C CNN
-F 2 "" H 3900 1650 50  0000 C CNN
-F 3 "" H 3900 1650 50  0000 C CNN
-	1    3900 1650
-	-1   0    0    -1
-$EndComp
-$Comp
-L GND #PWR32
+L GND #PWR0123
 U 1 1 57AD8439
 P 5200 2950
-F 0 "#PWR32" H 5200 2700 50  0001 C CNN
+F 0 "#PWR0123" H 5200 2700 50  0001 C CNN
 F 1 "GND" H 5200 2800 50  0000 C CNN
 F 2 "" H 5200 2950 50  0000 C CNN
@@
 $EndComp
 $Comp
-L GND #PWR26
+L GND #PWR0121
 U 1 1 57AD7D1A
 P 4350 2950
-F 0 "#PWR26" H 4350 2700 50  0001 C CNN
+F 0 "#PWR0121" H 4350 2700 50  0001 C CNN
 F 1 "GND" H 4350 2800 50  0000 C CNN
 F 2 "" H 4350 2950 50  0000 C CNN
@@
 $EndComp
 $Comp
-L GND #PWR24
+L GND #PWR0131
 U 1 1 57AD7A38
 P 3800 3000
-F 0 "#PWR24" H 3800 2750 50  0001 C CNN
+F 0 "#PWR0131" H 3800 2750 50  0001 C CNN
 F 1 "GND" H 3800 2850 50  0000 C CNN
 F 2 "" H 3800 3000 50  0000 C CNN
@@
 $EndComp
 $Comp
-L GND #PWR22
+L GND #PWR0120
 U 1 1 57AD797C
 P 3600 2950
-F 0 "#PWR22" H 3600 2700 50  0001 C CNN
+F 0 "#PWR0120" H 3600 2700 50  0001 C CNN
 F 1 "GND" H 3600 2800 50  0000 C CNN
 F 2 "" H 3600 2950 50  0000 C CNN
@@
 $EndComp
 $Comp
-L GND #PWR30
+L GND #PWR0122
 U 1 1 57A2183A
 P 5000 2950
-F 0 "#PWR30" H 5000 2700 50  0001 C CNN
+F 0 "#PWR0122" H 5000 2700 50  0001 C CNN
 F 1 "GND" H 5000 2800 50  0000 C CNN
 F 2 "" H 5000 2950 50  0000 C CNN
@@
 $EndComp
 $Comp
-L GND #PWR39
+L GND #PWR0132
 U 1 1 57AA37B1
 P 7050 3000
-F 0 "#PWR39" H 7050 2750 50  0001 C CNN
+F 0 "#PWR0132" H 7050 2750 50  0001 C CNN
 F 1 "GND" H 7050 2850 50  0000 C CNN
 F 2 "" H 7050 3000 50  0000 C CNN
@@
 $EndComp
 $Comp
-L VCC #PWR16
+L VCC #PWR0136
 U 1 1 57A2D136
 P 7600 4150
-F 0 "#PWR16" H 7600 4000 50  0001 C CNN
+F 0 "#PWR0136" H 7600 4000 50  0001 C CNN
 F 1 "VCC" H 7617 4323 50  0000 C CNN
 F 2 "" H 7600 4150 50  0000 C CNN
@@
 $EndComp
 $Comp
-L VCC #PWR21
+L VCC #PWR0118
 U 1 1 57A22D12
 P 3450 2200
-F 0 "#PWR21" H 3450 2050 50  0001 C CNN
+F 0 "#PWR0118" H 3450 2050 50  0001 C CNN
 F 1 "VCC" H 3467 2373 50  0000 C CNN
 F 2 "" H 3450 2200 50  0000 C CNN
@@
 $EndComp
 $Comp
-L GND #PWR37
+L GND #PWR0125
 U 1 1 57A21825
 P 6800 2950
-F 0 "#PWR37" H 6800 2700 50  0001 C CNN
+F 0 "#PWR0125" H 6800 2700 50  0001 C CNN
 F 1 "GND" H 6800 2800 50  0000 C CNN
 F 2 "" H 6800 2950 50  0000 C CNN
@@
 $EndComp
 $Comp
-L GND #PWR12
+L GND #PWR0139
 U 1 1 5837D4C6
 P 7150 4600
-F 0 "#PWR12" H 7150 4350 50  0001 C CNN
+F 0 "#PWR0139" H 7150 4350 50  0001 C CNN
 F 1 "GND" H 7150 4450 50  0000 C CNN
 F 2 "" H 7150 4600 50  0000 C CNN
@@
 $EndComp
 $Comp
-L GND #PWR11
+L GND #PWR0138
 U 1 1 5836E9BC
 P 6950 4600
-F 0 "#PWR11" H 6950 4350 50  0001 C CNN
+F 0 "#PWR0138" H 6950 4350 50  0001 C CNN
 F 1 "GND" H 6950 4450 50  0000 C CNN
 F 2 "" H 6950 4600 50  0000 C CNN
@@
 $EndComp
 $Comp
-L GND #PWR13
+L GND #PWR0140
 U 1 1 5836E9B0
 P 7400 4600
-F 0 "#PWR13" H 7400 4350 50  0001 C CNN
+F 0 "#PWR0140" H 7400 4350 50  0001 C CNN
 F 1 "GND" H 7400 4450 50  0000 C CNN
 F 2 "" H 7400 4600 50  0000 C CNN
@@
 $EndComp
 $Comp
-L GND #PWR10
+L GND #PWR0137
 U 1 1 582622CC
 P 6800 4450
-F 0 "#PWR10" H 6800 4200 50  0001 C CNN
+F 0 "#PWR0137" H 6800 4200 50  0001 C CNN
 F 1 "GND" H 6800 4300 50  0000 C CNN
 F 2 "" H 6800 4450 50  0000 C CNN
@@
 $EndComp
 $Comp
-L TEST_1P H5
-U 1 1 581BF01A
-P 5050 1650
-F 0 "H5" H 5108 1724 50  0000 L CNN
-F 1 "TEST_1P" H 5108 1679 50  0001 L CNN
-F 2 "components:MountingHole_3.2mm_M3" H 5108 1679 50  0001 L CNN
-F 3 "" H 5250 1650 50  0000 C CNN
-	1    5050 1650
-	1    0    0    -1
-$EndComp
-$Comp
-L GND #PWR47
+L GND #PWR0135
 U 1 1 58199141
 P 7650 3000
-F 0 "#PWR47" H 7650 2750 50  0001 C CNN
+F 0 "#PWR0135" H 7650 2750 50  0001 C CNN
 F 1 "GND" H 7650 2850 50  0000 C CNN
 F 2 "" H 7650 3000 50  0000 C CNN
@@
 $EndComp
 $Comp
-L GND #PWR44
+L GND #PWR0134
 U 1 1 57AA0DCC
 P 7450 3000
-F 0 "#PWR44" H 7450 2750 50  0001 C CNN
+F 0 "#PWR0134" H 7450 2750 50  0001 C CNN
 F 1 "GND" H 7450 2850 50  0000 C CNN
 F 2 "" H 7450 3000 50  0000 C CNN
@@
 $EndComp
 $Comp
-L GND #PWR41
+L GND #PWR0133
 U 1 1 57A98B8E
 P 7250 3000
-F 0 "#PWR41" H 7250 2750 50  0001 C CNN
+F 0 "#PWR0133" H 7250 2750 50  0001 C CNN
 F 1 "GND" H 7250 2850 50  0000 C CNN
 F 2 "" H 7250 3000 50  0000 C CNN
@@
 $EndComp
 $Comp
-L GND #PWR52
+L GND #PWR0130
 U 1 1 581881BF
 P 8350 2950
-F 0 "#PWR52" H 8350 2700 50  0001 C CNN
+F 0 "#PWR0130" H 8350 2700 50  0001 C CNN
 F 1 "GND" H 8350 2800 50  0000 C CNN
 F 2 "" H 8350 2950 50  0000 C CNN
@@
 $EndComp
 $Comp
-L GND #PWR51
+L GND #PWR0129
 U 1 1 581881B9
 P 8350 2950
-F 0 "#PWR51" H 8350 2700 50  0001 C CNN
+F 0 "#PWR0129" H 8350 2700 50  0001 C CNN
 F 1 "GND" H 8350 2800 50  0000 C CNN
 F 2 "" H 8350 2950 50  0000 C CNN
@@
 $EndComp
 $Comp
-L GND #PWR50
+L GND #PWR0128
 U 1 1 58187AD8
 P 8050 2950
-F 0 "#PWR50" H 8050 2700 50  0001 C CNN
+F 0 "#PWR0128" H 8050 2700 50  0001 C CNN
 F 1 "GND" H 8050 2800 50  0000 C CNN
 F 2 "" H 8050 2950 50  0000 C CNN
@@
 $EndComp
 $Comp
-L GND #PWR49
+L GND #PWR0127
 U 1 1 58187ACC
 P 8050 2950
-F 0 "#PWR49" H 8050 2700 50  0001 C CNN
+F 0 "#PWR0127" H 8050 2700 50  0001 C CNN
 F 1 "GND" H 8050 2800 50  0000 C CNN
 F 2 "" H 8050 2950 50  0000 C CNN
@@
 $EndComp
 $Comp
-L GND #PWR38
+L GND #PWR0126
 U 1 1 58186B9C
 P 6800 2950
-F 0 "#PWR38" H 6800 2700 50  0001 C CNN
+F 0 "#PWR0126" H 6800 2700 50  0001 C CNN
 F 1 "GND" H 6800 2800 50  0000 C CNN
 F 2 "" H 6800 2950 50  0000 C CNN
@@
 $EndComp
 $Comp
-L GND #PWR34
+L GND #PWR0119
 U 1 1 57B28643
 P 5950 2400
-F 0 "#PWR34" H 5950 2150 50  0001 C CNN
+F 0 "#PWR0119" H 5950 2150 50  0001 C CNN
 F 1 "GND" H 5955 2227 50  0000 C CNN
 F 2 "" H 5950 2400 50  0000 C CNN
@@
 $EndComp
 $Comp
-L GND #PWR36
+L GND #PWR0124
 U 1 1 583D6B21
 P 6150 2950
-F 0 "#PWR36" H 6150 2700 50  0001 C CNN
+F 0 "#PWR0124" H 6150 2700 50  0001 C CNN
 F 1 "GND" H 6150 2800 50  0000 C CNN
 F 2 "" H 6150 2950 50  0000 C CNN
@@
 	6950 4300 6950 4250
 Connection ~ 8350 2650
-Wire Wire Line
-	3900 1650 5050 1650
-Connection ~ 4850 1650
 Connection ~ 7050 2650
 Connection ~ 7250 2650

Commit message: This is the MazoClock hw 4.0 series; Uses ESP32 processor instead of ESP8266 used in prior MazoClock hw 3.0 series.
Parts:
- removed C19, C22, C23, C34, C71: 1u, Capacitors_SMD:C_0603_HandSoldering, symbol C
- removed C33, C56, C57: 100u, components:C_Radial_D6.3_L11.2_P2.5_hand_soldering, symbol CP
- removed JP13: Jumper_NC_Small, components:SolderJumper, symbol Jumper_NC_Small
- removed L1: BLM21PG331SN 300R@100MHz, Capacitors_SMD:C_0805_HandSoldering, symbol Ferrite_Bead_Small
- removed P6: CONN_01X03, Pin_Headers:Pin_Header_Straight_1x03, symbol CONN_01X03
- added C19, C22, C23: 100u, components:C_Radial_D6.3_L11.2_P2.5_hand_soldering, symbol CP
- added C28, C30: 1u, Capacitors_SMD:C_0603_HandSoldering, symbol C
- U14: footprint TO_SOT_Packages_SMD:TO-252-2Lead -> TO_SOT_Packages_SMD:TO-252-2
Connections:
- net labels removed: LEDLOGICVDD
- wire segments 33 -> 20

Commit message: Added some DC-DC convertes; DRC clear
Parts:
- added C33, C56, C61: 4.7u, Capacitors_SMD:C_0805_HandSoldering, symbol C
- added C34, C57, C69: 10u, Capacitors_SMD:C_1206_HandSoldering, symbol C
- added C35, C60, C71: 22p, Capacitors_SMD:C_0603_HandSoldering, symbol C
- added J12, J13: Conn_01x03_Female, Pin_Headers:Pin_Header_Straight_1x03_Pitch2.54mm, symbol Conn_01x03_Female
- added L1, L4, L7: 2.2uH, components:Choke_SMD_7.3x7.3_H3.5_handsoldering, symbol L
- added R38, R41, R48: 330k, Resistors_SMD:R_0603_HandSoldering, symbol R
- added R39, R46, R49: 75k, Resistors_SMD:R_0603_HandSoldering, symbol R
- added U20, U21, U22: NCP1529, TO_SOT_Packages_SMD:SOT-23-5_HandSoldering, symbol NCP1529
Connections:
- wire segments 20 -> 68
Other:
- note added: "Vout = 0.6*(1+330/75) = 3.24V"

Commit message: Updated to kicad 6.0.0 rc; removed outdated gerber files; Schematic is not complete
Parts:
- removed C56, C61: 4.7u, Capacitors_SMD:C_0805_HandSoldering, symbol C
- removed C57, C69: 10u, Capacitors_SMD:C_1206_HandSoldering, symbol C
- removed C60, C71: 22p, Capacitors_SMD:C_0603_HandSoldering, symbol C
- removed J12, J13: Conn_01x03_Female, Pin_Headers:Pin_Header_Straight_1x03_Pitch2.54mm, symbol Conn_01x03_Female
- removed L4, L7: 2.2uH, components:Choke_SMD_7.3x7.3_H3.5_handsoldering, symbol L
- removed R41, R48: 330k, Resistors_SMD:R_0603_HandSoldering, symbol R
- removed R46, R49: 75k, Resistors_SMD:R_0603_HandSoldering, symbol R
- removed U21, U22: NCP1529, TO_SOT_Packages_SMD:SOT-23-5_HandSoldering, symbol NCP1529
- C1, C19, C21, C22, C23, C31: symbol CP -> device:CP
- C18, C20, C28, C30, C33, C34, C35, C64, C66, C72: symbol C -> device:C
- CONN1: symbol Barrel_Jack -> Connector:Barrel_Jack
- D7: symbol D_Zener_Small_ALT -> device:D_Zener_Small_ALT
- F1: symbol Polyfuse_Small -> device:Polyfuse_Small
- L1: symbol L -> device:L
- R38, R39: symbol R -> device:R
- T1: symbol COMMON_MODE_CHOKE -> DeeComponents:COMMON_MODE_CHOKE
- U14: symbol LT1129-3.3_SOT223 -> regul:LT1129-3.3_SOT223
- U20: symbol NCP1529 -> DeeComponents:NCP1529
Connections:
- wire segments 68 -> 44

Commit message: Heavily modifying; Matrix nets under construction
Parts:
- removed C1, C19, C21, C22, C23: 100u, components:C_Radial_D6.3_L11.2_P2.5_hand_soldering, symbol device:CP
- removed C18, C20: 1u, Capacitors_SMD:C_0603_HandSoldering, symbol device:C
- removed C31: 1000u 16V LowESR, components:CAP_100_OR_200_P_LAY, symbol device:CP
- removed U14: NJM2845DL1-33, TO_SOT_Packages_SMD:TO-252-2, symbol regul:LT1129-3.3_SOT223
- removed U20: NCP1529, TO_SOT_Packages_SMD:SOT-23-5_HandSoldering, symbol DeeComponents:NCP1529
- added C29, C62, C75, C76: 1u, Capacitors_SMD:C_0603_HandSoldering, symbol device:C
- added C31, C65: 0.1u, Capacitors_SMD:C_0603_HandSoldering, symbol device:C
- added C55: 0.1u, Capacitors_SMD:C_0805_HandSoldering, symbol device:C
- added C56: 22p, Capacitors_SMD:C_0603_HandSoldering, symbol device:C
- added C57, C59, C60, C61: 10u, Capacitors_SMD:C_1206_HandSoldering, symbol device:C
- added L2: 2.2uH, components:Choke_SMD_12x12mm_10.4x10.4mm_compat_h4.5mm_handsoldering, symbol device:L
- added L4: BLM21PG331SN 300R@100MHz, Capacitors_SMD:C_0805_HandSoldering, symbol device:Ferrite_Bead_Small
- added Q29: AO3401, TO_SOT_Packages_SMD:SOT-23_Handsoldering, symbol device:Q_PMOS_GSD
- added Q30: Q_NPN_BEC, TO_SOT_Packages_SMD:SOT-23_Handsoldering, symbol device:Q_NPN_BEC
- added R101, R104: 10k, Resistors_SMD:R_0603_HandSoldering, symbol device:R
- added R102: 100k, Resistors_SMD:R_0603_HandSoldering, symbol device:R
- added R103: 22k, Resistors_SMD:R_0603_HandSoldering, symbol device:R
- added R105, R115: 10R, Resistors_SMD:R_0603_HandSoldering, symbol device:R
- added R114: 4.7k, Resistors_SMD:R_0603_HandSoldering, symbol device:R
- added U19: TPS54428DDA, Housings_SOIC:TI_SO-PowerPAD-8, symbol DeeComponents:TPS54428DDA
- added U2: TPS54202, TO_SOT_Packages_SMD:SOT-23-6, symbol DeeComponents:TPS54202
- C28: value 1u -> 10u; footprint Capacitors_SMD:C_0603_HandSoldering -> Capacitors_SMD:C_0805_HandSoldering
- C30: value 1u -> 0.1u
- C33: value 4.7u -> 10u
- D7: footprint Diodes_SMD:DO-214BA -> Diodes_SMD:D_SMA_Handsoldering
- L1: footprint components:Choke_SMD_7.3x7.3_H3.5_handsoldering -> components:Choke_SMD_12x12mm_10.4x10.4mm_compat_h4.5mm_handsoldering
- R38: value 330k -> 100k
- R39: value 75k -> 22k
Connections:
- net labels added: D_LED1642_RST, LED1642VDD, LEDDC_SW, LEDLOGICVDD, LEDVDD
- wire segments 44 -> 108
Other:
- note added: "3.15V, 4A"
- note added: "3V3 2A"
- note added: "5V"
- note added: "TPS54428DDA for LED Anode, Anode voltage is around 3.1V"
- note added: "Vout = .596*(100000.0/(22000)+1) = 3.305090909090909"
- note removed: "Vout = 0.6*(1+330/75) = 3.24V"
