File: power.sch (KiCad schematic (older format))
At the start: 40 parts, among them Q29 AO3401, Q30 Q_NPN_BEC, T1 COMMON_MODE_CHOKE, U19 TPS54428DDA, U2 TPS54202

Commit message: Almost all components has placed.
Parts:
- C28, C33: value 10u -> 10u 16V
- C75, C76: value 1u -> 1u 16V
- L1: value 2.2uH -> 10uH; footprint components:Choke_SMD_12x12mm_10.4x10.4mm_compat_h4.5mm_handsoldering -> components:Choke_SMD_7.3x7.3_H3.5_handsoldering
- L2: footprint components:Choke_SMD_12x12mm_10.4x10.4mm_compat_h4.5mm_handsoldering -> components:Choke_SMD_7.3x7.3_H3.5_handsoldering
Connections:
- net labels added: DC_IN_N, DC_IN_P
- net labels removed: DC_IN
Other:
- note added: "12V"
- note removed: "5V"
Changed lines of the file:
@@
 EESchema Schematic File Version 4
 LIBS:dotmatrix_64x48-cache
-EELAYER 28 0
+EELAYER 29 0
 EELAYER END
 $Descr A4 11693 8268
@@
 $EndDescr
 Text GLabel 1350 1250 1    60   Input ~ 0
-DC_IN
+DC_IN_P
 $Comp
 L device:Polyfuse_Small F1
@@
 AR Path="/5BB33F0A/59E42088" Ref="C?"  Part="1"
 F 0 "C33" H 1050 2900 50  0000 L CNN
-F 1 "10u" H 1050 2800 50  0000 L CNN
+F 1 "10u 16V" H 1050 2800 50  0000 L CNN
 F 2 "Capacitors_SMD:C_0805_HandSoldering" H 1215 3259 50  0001 L CNN
 F 3 "" H 1100 3350 50  0000 C CNN
@@
 AR Path="/5BB33F0A/59E42358" Ref="L?"  Part="1"
 F 0 "L1" V 3072 3400 50  0000 C CNN
-F 1 "2.2uH" V 3163 3400 50  0000 C CNN
-F 2 "components:Choke_SMD_12x12mm_10.4x10.4mm_compat_h4.5mm_handsoldering" H 3250 3400 50  0001 C CNN
+F 1 "10uH" V 3163 3400 50  0000 C CNN
+F 2 "components:Choke_SMD_7.3x7.3_H3.5_handsoldering" H 3250 3400 50  0001 C CNN
 F 3 "" H 3250 3400 50  0001 C CNN
 	1    3250 3400
@@
 	3850 1050 4200 1050
 Text Notes 4750 950  0    50   ~ 0
-5V
+12V
 $Comp
 L DeeComponents:TPS54428DDA U19
@@
 AR Path="/5BB33F0A/5BBCC3D9" Ref="C?"  Part="1"
 F 0 "C28" H 950 5000 50  0000 L CNN
-F 1 "10u" H 950 4900 50  0000 L CNN
+F 1 "10u 16V" H 950 4900 50  0000 L CNN
 F 2 "Capacitors_SMD:C_0805_HandSoldering" H 1115 5359 50  0001 L CNN
 F 3 "" H 1000 5450 50  0000 C CNN
@@
 F 0 "L2" V 3522 5700 50  0000 C CNN
 F 1 "2.2uH" V 3613 5700 50  0000 C CNN
-F 2 "components:Choke_SMD_12x12mm_10.4x10.4mm_compat_h4.5mm_handsoldering" H 3700 5700 50  0001 C CNN
+F 2 "components:Choke_SMD_7.3x7.3_H3.5_handsoldering" H 3700 5700 50  0001 C CNN
 F 3 "" H 3700 5700 50  0001 C CNN
 	1    3700 5700
@@
 AR Path="/5BB33F0A/5BC62B65" Ref="C?"  Part="1"
 F 0 "C75" H 1200 2950 50  0000 L CNN
-F 1 "1u" H 1250 2850 50  0000 L CNN
+F 1 "1u 16V" H 1250 2850 50  0000 L CNN
 F 2 "Capacitors_SMD:C_0603_HandSoldering" H 1415 3259 50  0001 L CNN
 F 3 "" H 1300 3350 50  0000 C CNN
@@
 AR Path="/5BB33F0A/5BC7105F" Ref="C?"  Part="1"
 F 0 "C76" H 1150 5050 50  0000 L CNN
-F 1 "1u" H 1200 4950 50  0000 L CNN
+F 1 "1u 16V" H 1200 4950 50  0000 L CNN
 F 2 "Capacitors_SMD:C_0603_HandSoldering" H 1365 5359 50  0001 L CNN
 F 3 "" H 1250 5450 50  0000 C CNN
@@
 Text Label 2900 5700 0    50   ~ 0
 LEDDC_SW
+Text Label 2050 1350 0    50   ~ 0
+DC_IN_N
 $EndSCHEMATC

Commit message: Too less PCB space.
Parts:
- added C2: 10u, Capacitors_SMD:C_1206_HandSoldering, symbol device:C
Connections:
- wire segments 108 -> 109
Changed lines of the file:
@@
 Connection ~ 6150 3600
 Wire Wire Line
-	6150 3600 6750 3600
+	6150 3600 6350 3600
 Wire Wire Line
 	4650 3600 5100 3600
@@
 Text Label 2050 1350 0    50   ~ 0
 DC_IN_N
+$Comp
+L device:C C2
+U 1 1 5BDA55B3
+P 6350 3750
+AR Path="/59A82F84/5BDA55B3" Ref="C2"  Part="1"
+AR Path="/5BB33F0A/5BDA55B3" Ref="C?"  Part="1"
+F 0 "C2" H 6500 3600 50  0000 L CNN
+F 1 "10u" H 6500 3500 50  0000 L CNN
+F 2 "Capacitors_SMD:C_1206_HandSoldering" H 6465 3659 50  0001 L CNN
+F 3 "" H 6350 3750 50  0000 C CNN
+	1    6350 3750
+	1    0    0    -1
+$EndComp
+$Comp
+L power:GND #PWR?
+U 1 1 5BDA8B7D
+P 6350 3900
+AR Path="/59A8E319/5BDA8B7D" Ref="#PWR?"  Part="1"
+AR Path="/5BDA8B7D" Ref="#PWR?"  Part="1"
+AR Path="/59A82F84/5BDA8B7D" Ref="#PWR0151"  Part="1"
+F 0 "#PWR0151" H 6350 3650 50  0001 C CNN
+F 1 "GND" H 6355 3727 50  0000 C CNN
+F 2 "" H 6350 3900 50  0000 C CNN
+F 3 "" H 6350 3900 50  0000 C CNN
+	1    6350 3900
+	1    0    0    -1
+$EndComp
+Connection ~ 6350 3600
+Wire Wire Line
+	6350 3600 6750 3600
 $EndSCHEMATC

Commit message: Added stereo power amplifier
Parts:
- CONN1: footprint Connect:BARREL_JACK -> components:BARREL_JACK_HIGH_CURRENT_PJ018
- F1: footprint Resistors_SMD:R_1812_HandSoldering -> Resistors_SMD:R_1812
Connections:
- net labels added: V12_PREFUSE
- wire segments 109 -> 115
Changed lines of the file:
@@
 $Descr A4 11693 8268
 encoding utf-8
-Sheet 9 10
+Sheet 9 11
 Title ""
 Date ""
@@
 L device:Polyfuse_Small F1
 U 1 1 57A2A89C
-P 2250 950
+P 4250 1050
 AR Path="/59A82F84/57A2A89C" Ref="F1"  Part="1"
 AR Path="/5BB33F0A/57A2A89C" Ref="F?"  Part="1"
-F 0 "F1" V 2150 950 50  0000 C CNN
-F 1 "FUSE" V 2050 950 50  0000 C CNN
-F 2 "Resistors_SMD:R_1812_HandSoldering" H 2250 950 50  0001 C CNN
-F 3 "" H 2250 950 50  0000 C CNN
-	1    2250 950
+F 0 "F1" V 4150 1050 50  0000 C CNN
+F 1 "FUSE" V 4050 1050 50  0000 C CNN
+F 2 "Resistors_SMD:R_1812" H 4250 1050 50  0001 C CNN
+F 3 "" H 4250 1050 50  0000 C CNN
+	1    4250 1050
 	0    -1   1    0
 $EndComp
@@
 L power:VCC #PWR0134
 U 1 1 57A2D136
-P 4650 950
+P 4900 950
 AR Path="/59A82F84/57A2D136" Ref="#PWR0134"  Part="1"
 AR Path="/5BB33F0A/57A2D136" Ref="#PWR?"  Part="1"
-F 0 "#PWR0134" H 4650 800 50  0001 C CNN
-F 1 "VCC" H 4667 1123 50  0000 C CNN
-F 2 "" H 4650 950 50  0000 C CNN
-F 3 "" H 4650 950 50  0000 C CNN
-	1    4650 950
+F 0 "#PWR0134" H 4900 800 50  0001 C CNN
+F 1 "VCC" H 4917 1123 50  0000 C CNN
+F 2 "" H 4900 950 50  0000 C CNN
+F 3 "" H 4900 950 50  0000 C CNN
+	1    4900 950
 	1    0    0    -1
 $EndComp
@@
 F 0 "CONN1" H 982 1675 50  0000 C CNN
 F 1 "BARREL_JACK" H 982 1584 50  0000 C CNN
-F 2 "Connect:BARREL_JACK" H 1000 1350 50  0001 C CNN
+F 2 "components:BARREL_JACK_HIGH_CURRENT_PJ018" H 1000 1350 50  0001 C CNN
 F 3 "" H 1000 1350 50  0000 C CNN
 	1    1000 1350
@@
 L power:GND #PWR0137
 U 1 1 5837D4C6
-P 4200 1400
+P 4450 1400
 AR Path="/59A82F84/5837D4C6" Ref="#PWR0137"  Part="1"
 AR Path="/5BB33F0A/5837D4C6" Ref="#PWR?"  Part="1"
-F 0 "#PWR0137" H 4200 1150 50  0001 C CNN
-F 1 "GND" H 4200 1250 50  0000 C CNN
-F 2 "" H 4200 1400 50  0000 C CNN
-F 3 "" H 4200 1400 50  0000 C CNN
-	1    4200 1400
-	-1   0    0    -1
-$EndComp
-$Comp
-L device:C C64
-U 1 1 5836E9C2
-P 4200 1250
-AR Path="/59A82F84/5836E9C2" Ref="C64"  Part="1"
-AR Path="/5BB33F0A/5836E9C2" Ref="C?"  Part="1"
-F 0 "C64" H 4100 850 50  0000 L CNN
-F 1 "1u" H 4150 750 50  0000 L CNN
-F 2 "Capacitors_SMD:C_0603_HandSoldering" H 4315 1159 50  0001 L CNN
-F 3 "" H 4200 1250 50  0000 C CNN
-	1    4200 1250
-	1    0    0    -1
-$EndComp
-$Comp
-L power:GND #PWR0138
-U 1 1 5836E9B0
-P 4450 1400
-AR Path="/59A82F84/5836E9B0" Ref="#PWR0138"  Part="1"
-AR Path="/5BB33F0A/5836E9B0" Ref="#PWR?"  Part="1"
-F 0 "#PWR0138" H 4450 1150 50  0001 C CNN
+F 0 "#PWR0137" H 4450 1150 50  0001 C CNN
 F 1 "GND" H 4450 1250 50  0000 C CNN
 F 2 "" H 4450 1400 50  0000 C CNN
 F 3 "" H 4450 1400 50  0000 C CNN
 	1    4450 1400
+	-1   0    0    -1
+$EndComp
+$Comp
+L device:C C64
+U 1 1 5836E9C2
+P 4450 1250
+AR Path="/59A82F84/5836E9C2" Ref="C64"  Part="1"
+AR Path="/5BB33F0A/5836E9C2" Ref="C?"  Part="1"
+F 0 "C64" H 4350 850 50  0000 L CNN
+F 1 "1u" H 4400 750 50  0000 L CNN
+F 2 "Capacitors_SMD:C_0603_HandSoldering" H 4565 1159 50  0001 L CNN
+F 3 "" H 4450 1250 50  0000 C CNN
+	1    4450 1250
+	1    0    0    -1
+$EndComp
+$Comp
+L power:GND #PWR0138
+U 1 1 5836E9B0
+P 4700 1400
+AR Path="/59A82F84/5836E9B0" Ref="#PWR0138"  Part="1"
+AR Path="/5BB33F0A/5836E9B0" Ref="#PWR?"  Part="1"
+F 0 "#PWR0138" H 4700 1150 50  0001 C CNN
+F 1 "GND" H 4700 1250 50  0000 C CNN
+F 2 "" H 4700 1400 50  0000 C CNN
+F 3 "" H 4700 1400 50  0000 C CNN
+	1    4700 1400
 	-1   0    0    -1
 $EndComp
@@
 L device:C C66
 U 1 1 5837D4CC
-P 4450 1250
+P 4700 1250
 AR Path="/59A82F84/5837D4CC" Ref="C66"  Part="1"
 AR Path="/5BB33F0A/5837D4CC" Ref="C?"  Part="1"
-F 0 "C66" H 4350 850 50  0000 L CNN
-F 1 "0.1u" H 4350 750 50  0000 L CNN
-F 2 "Capacitors_SMD:C_0603_HandSoldering" H 4565 1159 50  0001 L CNN
-F 3 "" H 4450 1250 50  0000 C CNN
-	1    4450 1250
+F 0 "C66" H 4600 850 50  0000 L CNN
+F 1 "0.1u" H 4600 750 50  0000 L CNN
+F 2 "Capacitors_SMD:C_0603_HandSoldering" H 4815 1159 50  0001 L CNN
+F 3 "" H 4700 1250 50  0000 C CNN
+	1    4700 1250
 	1    0    0    -1
 $EndComp
@@
 Wire Wire Line
 	1500 950  1750 950
+Connection ~ 4700 1050
+Wire Wire Line
+	4700 1050 4700 1100
 Connection ~ 4450 1050
 Wire Wire Line
 	4450 1050 4450 1100
-Connection ~ 4200 1050
-Wire Wire Line
-	4200 1050 4200 1100
-Wire Wire Line
-	4650 1050 4650 950
+Wire Wire Line
+	4900 1050 4900 950
 Wire Wire Line
 	1500 1250 1300 1250
@@
 	1600 1350 1600 1450
 Wire Wire Line
-	4450 1050 4650 1050
-Wire Wire Line
-	4200 1050 4450 1050
+	4700 1050 4900 1050
+Wire Wire Line
+	4450 1050 4700 1050
 Wire Wire Line
 	4050 3800 4050 3850
@@
 Wire Wire Line
 	5100 3100 5100 3600
-Wire Wire Line
-	3850 1050 4200 1050
-Text Notes 4750 950  0    50   ~ 0
+Text Notes 5000 950  0    50   ~ 0
 12V
 $Comp
@@
 Wire Wire Line
 	1000 5100 1000 5300
-$Comp
-L power:GND #PWR?
-U 1 1 5BBD1AEF
-P 1650 6050
-AR Path="/59A8E319/5BBD1AEF" Ref="#PWR?"  Part="1"
-AR Path="/5BBD1AEF" Ref="#PWR?"  Part="1"
-AR Path="/59A82F84/5BBD1AEF" Ref="#PWR08"  Part="1"
-F 0 "#PWR08" H 1650 5800 50  0001 C CNN
-F 1 "GND" H 1650 5900 50  0000 C CNN
-F 2 "" H 1650 6050 50  0000 C CNN
-F 3 "" H 1650 6050 50  0000 C CNN
-	1    1650 6050
-	-1   0    0    -1
-$EndComp
 $Comp
 L device:C C?
@@
 $EndComp
 Wire Wire Line
-	1650 6050 1650 6000
-Wire Wire Line
 	1900 5700 1650 5700
 $Comp
@@
 	1    0    0    -1
 $EndComp
-$Comp
-L power:GND #PWR?
-U 1 1 5BBD4E04
-P 1850 6200
-AR Path="/59A8E319/5BBD4E04" Ref="#PWR?"  Part="1"
-AR Path="/5BBD4E04" Ref="#PWR?"  Part="1"
-AR Path="/59A82F84/5BBD4E04" Ref="#PWR09"  Part="1"
-F 0 "#PWR09" H 1850 5950 50  0001 C CNN
-F 1 "GND" H 1855 6027 50  0000 C CNN
-F 2 "" H 1850 6200 50  0000 C CNN
-F 3 "" H 1850 6200 50  0000 C CNN
-	1    1850 6200
-	1    0    0    -1
-$EndComp
-Wire Wire Line
-	1850 6150 1850 6200
 Wire Wire Line
 	1850 5850 1900 5850
@@
 L power:GND #PWR?
 U 1 1 5BBD8503
-P 2400 6100
+P 2400 6400
 AR Path="/59A8E319/5BBD8503" Ref="#PWR?"  Part="1"
 AR Path="/5BBD8503" Ref="#PWR?"  Part="1"
 AR Path="/59A82F84/5BBD8503" Ref="#PWR010"  Part="1"
-F 0 "#PWR010" H 2400 5850 50  0001 C CNN
-F 1 "GND" H 2405 5927 50  0000 C CNN
-F 2 "" H 2400 6100 50  0000 C CNN
-F 3 "" H 2400 6100 50  0000 C CNN
-	1    2400 6100
+F 0 "#PWR010" H 2400 6150 50  0001 C CNN
+F 1 "GND" H 2405 6227 50  0000 C CNN
+F 2 "" H 2400 6400 50  0000 C CNN
+F 3 "" H 2400 6400 50  0000 C CNN
+	1    2400 6400
 	1    0    0    -1
 $EndComp
@@
 	1750 5550 1900 5550
 Wire Wire Line
-	1750 950  2150 950
-Wire Wire Line
 	4650 3600 4650 3400
 Wire Wire Line
@@
 Wire Wire Line
 	2500 1050 2500 950
-Wire Wire Line
-	2500 950  2350 950
 Connection ~ 2700 1050
 $Comp
@@
 Wire Wire Line
 	6350 3600 6750 3600
+Wire Wire Line
+	4350 1050 4450 1050
+Wire Wire Line
+	1750 950  2500 950
+Wire Wire Line
+	3850 1050 3950 1050
+Wire Wire Line
+	3950 700  3950 1050
+Connection ~ 3950 1050
+Wire Wire Line
+	3950 1050 4150 1050
+Text GLabel 3950 700  0    50   Input ~ 0
+V12_PREFUSE
+Wire Wire Line
+	2400 6400 2400 6300
+Wire Wire Line
+	2400 6300 1850 6300
+Wire Wire Line
+	1850 6150 1850 6300
+Wire Wire Line
+	1850 6300 1650 6300
+Wire Wire Line
+	1650 6000 1650 6300
+Connection ~ 1850 6300
+Wire Wire Line
+	2400 6300 2400 6100
+Connection ~ 2400 6300
 $EndSCHEMATC

Commit message: Switched to new kicad libraries
Parts:
- C2, C28, C29, C30, C31, C33, C34, C35, C55, C56, C57, C59, C60, C61, C62, C64, C65, C66, C72, C75, C76: symbol device:C -> dotmatrix_64x48-rescue:C-device
- CONN1: symbol Connector:Barrel_Jack -> dotmatrix_64x48-rescue:Barrel_Jack-Connector
- D7: symbol device:D_Zener_Small_ALT -> dotmatrix_64x48-rescue:D_Zener_Small_ALT-device
- F1: symbol device:Polyfuse_Small -> dotmatrix_64x48-rescue:Polyfuse_Small-device
- L1, L2: symbol device:L -> dotmatrix_64x48-rescue:L-device
- L4: symbol device:Ferrite_Bead_Small -> dotmatrix_64x48-rescue:Ferrite_Bead_Small-device
- Q29: symbol device:Q_PMOS_GSD -> dotmatrix_64x48-rescue:Q_PMOS_GSD-device
- Q30: symbol device:Q_NPN_BEC -> dotmatrix_64x48-rescue:Q_NPN_BEC-device
- R101, R102, R103, R104, R105, R114, R115, R38, R39: symbol device:R -> dotmatrix_64x48-rescue:R-device
Changed lines of the file:
@@
 DC_IN_P
 $Comp
-L device:Polyfuse_Small F1
+L dotmatrix_64x48-rescue:Polyfuse_Small-device F1
 U 1 1 57A2A89C
 P 4250 1050
@@
 $EndComp
 $Comp
-L power:VCC #PWR0134
+L dotmatrix_64x48-rescue:VCC-power #PWR0134
 U 1 1 57A2D136
 P 4900 950
@@
 $EndComp
 $Comp
-L Connector:Barrel_Jack CONN1
+L dotmatrix_64x48-rescue:Barrel_Jack-Connector CONN1
 U 1 1 57A2CB58
 P 1000 1350
 AR Path="/59A82F84/57A2CB58" Ref="CONN1"  Part="1"
 AR Path="/5BB33F0A/57A2CB58" Ref="CONN?"  Part="1"
+AR Path="/57A2CB58" Ref="CONN1"  Part="1"
 F 0 "CONN1" H 982 1675 50  0000 C CNN
 F 1 "BARREL_JACK" H 982 1584 50  0000 C CNN
@@
 $EndComp
 $Comp
-L power:GND #PWR0137
+L dotmatrix_64x48-rescue:GND-power #PWR0137
 U 1 1 5837D4C6
 P 4450 1400
@@
 $EndComp
 $Comp
-L device:C C64
+L dotmatrix_64x48-rescue:C-device C64
 U 1 1 5836E9C2
 P 4450 1250
@@
 $EndComp
 $Comp
-L power:GND #PWR0138
+L dotmatrix_64x48-rescue:GND-power #PWR0138
 U 1 1 5836E9B0
 P 4700 1400
@@
 $EndComp
 $Comp
-L power:GND #PWR0135
+L dotmatrix_64x48-rescue:GND-power #PWR0135
 U 1 1 582622CC
 P 3850 1250
@@
 $EndComp
 $Comp
-L device:D_Zener_Small_ALT D7
+L dotmatrix_64x48-rescue:D_Zener_Small_ALT-device D7
 U 1 1 5859EE13
 P 1750 1100
@@
 $EndComp
 $Comp
-L device:C C72
+L dotmatrix_64x48-rescue:C-device C72
 U 1 1 583E92D5
 P 2700 1200
@@
 $EndComp
 $Comp
-L device:C C66
+L dotmatrix_64x48-rescue:C-device C66
 U 1 1 5837D4CC
 P 4700 1250
@@
 	1500 1250 1300 1250
 $Comp
-L device:C C33
+L dotmatrix_64x48-rescue:C-device C33
 U 1 1 59E42088
 P 1100 3350
@@
 $EndComp
 $Comp
-L power:GND #PWR0146
+L dotmatrix_64x48-rescue:GND-power #PWR0146
 U 1 1 59E4208E
 P 1100 3550
@@
 	1100 3550 1100 3500
 $Comp
-L device:L L1
+L dotmatrix_64x48-rescue:L-device L1
 U 1 1 59E42358
 P 3250 3400
@@
 $EndComp
 $Comp
-L device:C C34
+L dotmatrix_64x48-rescue:C-device C34
 U 1 1 59E426BA
 P 3650 3550
@@
 $EndComp
 $Comp
-L power:GND #PWR0148
+L dotmatrix_64x48-rescue:GND-power #PWR0148
 U 1 1 59E426C0
 P 3650 3900
@@
 	3650 3700 3650 3900
 $Comp
-L device:R R38
+L dotmatrix_64x48-rescue:R-device R38
 U 1 1 59E42F9D
 P 4050 3600
@@
 $EndComp
 $Comp
-L device:R R39
+L dotmatrix_64x48-rescue:R-device R39
 U 1 1 59E430E9
 P 4050 4000
@@
 $EndComp
 $Comp
-L device:C C35
+L dotmatrix_64x48-rescue:C-device C35
 U 1 1 59E4315B
 P 4400 3550
@@
 Connection ~ 1400 3200
 $Comp
-L power:VCC #PWR0145
+L dotmatrix_64x48-rescue:VCC-power #PWR0145
 U 1 1 59E439B6
 P 850 3000
@@
 LEDLOGICVDD
 $Comp
-L power:GND #PWR0147
+L dotmatrix_64x48-rescue:GND-power #PWR0147
 U 1 1 59E441C7
 P 2000 3800
@@
 $EndComp
 $Comp
-L power:GND #PWR0149
+L dotmatrix_64x48-rescue:GND-power #PWR0149
 U 1 1 59E449D3
 P 4050 4150
@@
 	3650 3400 4050 3400
 $Comp
-L device:C C55
+L dotmatrix_64x48-rescue:C-device C55
 U 1 1 5BABFE14
 P 2750 3200
@@
 ESPVDD
 $Comp
-L device:Ferrite_Bead_Small L?
+L dotmatrix_64x48-rescue:Ferrite_Bead_Small-device L?
 U 1 1 5BB82B05
 P 5650 3600
@@
 $EndComp
 $Comp
-L power:GND #PWR?
+L dotmatrix_64x48-rescue:GND-power #PWR?
 U 1 1 5BB82B0D
 P 5900 3950
@@
 $EndComp
 $Comp
-L device:C C?
+L dotmatrix_64x48-rescue:C-device C?
 U 1 1 5BB82B13
 P 5900 3750
@@
 $EndComp
 $Comp
-L device:C C?
+L dotmatrix_64x48-rescue:C-device C?
 U 1 1 5BB82B1A
 P 6150 3750
@@
 $EndComp
 $Comp
-L power:GND #PWR?
+L dotmatrix_64x48-rescue:GND-power #PWR?
 U 1 1 5BB82B21
 P 6150 3950
@@
 3V3 2A
 $Comp
-L device:Q_PMOS_GSD Q29
+L dotmatrix_64x48-rescue:Q_PMOS_GSD-device Q29
 U 1 1 5BB939F2
 P 8500 3250
@@
 	8200 3150 8300 3150
 $Comp
-L device:Q_NPN_BEC Q30
+L dotmatrix_64x48-rescue:Q_NPN_BEC-device Q30
 U 1 1 5BB939FB
 P 9350 3900
@@
 $EndComp
 $Comp
-L device:R R114
+L dotmatrix_64x48-rescue:R-device R114
 U 1 1 5BB93A02
 P 8950 3900
@@
 $EndComp
 $Comp
-L device:R R105
+L dotmatrix_64x48-rescue:R-device R105
 U 1 1 5BB93A09
 P 8250 3900
@@
 $EndComp
 $Comp
-L power:GND #PWR018
+L dotmatrix_64x48-rescue:GND-power #PWR018
 U 1 1 5BB93A10
 P 9450 4150
@@
 	9450 3150 9650 3150
 $Comp
-L device:R R115
+L dotmatrix_64x48-rescue:R-device R115
 U 1 1 5BB93A1E
 P 9450 3500
@@
 $EndComp
 $Comp
-L device:C C28
+L dotmatrix_64x48-rescue:C-device C28
 U 1 1 5BBCC3D9
 P 1000 5450
@@
 $EndComp
 $Comp
-L power:GND #PWR07
+L dotmatrix_64x48-rescue:GND-power #PWR07
 U 1 1 5BBCC3DF
 P 1000 5650
@@
 	1000 5650 1000 5600
 $Comp
-L power:VCC #PWR06
+L dotmatrix_64x48-rescue:VCC-power #PWR06
 U 1 1 5BBCC3E6
 P 1000 5100
@@
 	1000 5100 1000 5300
 $Comp
-L device:C C?
+L dotmatrix_64x48-rescue:C-device C?
 U 1 1 5BBD1AF5
 P 1650 5850
@@
 	1900 5700 1650 5700
 $Comp
-L device:C C?
+L dotmatrix_64x48-rescue:C-device C?
 U 1 1 5BBD4DFE
 P 1850 6000
@@
 	1850 5850 1900 5850
 $Comp
-L power:GND #PWR?
+L dotmatrix_64x48-rescue:GND-power #PWR?
 U 1 1 5BBD8503
 P 2400 6400
@@
 $EndComp
 $Comp
-L device:C C?
+L dotmatrix_64x48-rescue:C-device C?
 U 1 1 5BBDA610
 P 3150 5550
@@
 	3350 5700 3350 5550
 $Comp
-L device:L L2
+L dotmatrix_64x48-rescue:L-device L2
 U 1 1 5BBE36D3
 P 3700 5700
@@
 $EndComp
 $Comp
-L device:C C57
+L dotmatrix_64x48-rescue:C-device C57
 U 1 1 5BBE36D9
 P 4150 5850
@@
 Connection ~ 3350 5700
 $Comp
-L device:C C59
+L dotmatrix_64x48-rescue:C-device C59
 U 1 1 5BBE58F5
 P 4350 5850
@@
 Connection ~ 4350 5700
 $Comp
-L device:C C60
+L dotmatrix_64x48-rescue:C-device C60
 U 1 1 5BBE9B14
 P 4550 5850
@@
 	3850 5700 4000 5700
 $Comp
-L device:C C61
+L dotmatrix_64x48-rescue:C-device C61
 U 1 1 5BBEDEC6
 P 4750 5850
@@
 Connection ~ 4550 5700
 $Comp
-L device:R R102
+L dotmatrix_64x48-rescue:R-device R102
 U 1 1 5BBF4A3E
 P 3850 6000
@@
 $EndComp
 $Comp
-L device:R R103
+L dotmatrix_64x48-rescue:R-device R103
 U 1 1 5BBF9176
 P 3850 6450
@@
 $EndComp
 $Comp
-L power:GND #PWR011
+L dotmatrix_64x48-rescue:GND-power #PWR011
 U 1 1 5BBF917C
 P 3850 6900
@@
 $EndComp
 $Comp
-L power:GND #PWR012
+L dotmatrix_64x48-rescue:GND-power #PWR012
 U 1 1 5BBFB3AB
 P 4150 6000
@@
 $EndComp
 $Comp
-L power:GND #PWR013
+L dotmatrix_64x48-rescue:GND-power #PWR013
 U 1 1 5BBFD5DA
 P 4350 6000
@@
 $EndComp
 $Comp
-L power:GND #PWR014
+L dotmatrix_64x48-rescue:GND-power #PWR014
 U 1 1 5BBFF809
 P 4550 6000
@@
 $EndComp
 $Comp
-L power:GND #PWR015
+L dotmatrix_64x48-rescue:GND-power #PWR015
 U 1 1 5BBFF80F
 P 4750 6000
@@
 $EndComp
 $Comp
-L device:R R104
+L dotmatrix_64x48-rescue:R-device R104
 U 1 1 5BC04AA9
 P 3850 6750
@@
 	3850 6200 3850 6300
 $Comp
-L device:C C56
+L dotmatrix_64x48-rescue:C-device C56
 U 1 1 5BC104FD
 P 3500 6050
@@
 3.15V, 4A
 $Comp
-L device:R R101
+L dotmatrix_64x48-rescue:R-device R101
 U 1 1 5BC29E87
 P 1600 5450
@@
 Connection ~ 2700 1050
 $Comp
-L power:GND #PWR0139
+L dotmatrix_64x48-rescue:GND-power #PWR0139
 U 1 1 5BC62B5B
 P 1300 3500
@@
 $EndComp
 $Comp
-L device:C C75
+L dotmatrix_64x48-rescue:C-device C75
 U 1 1 5BC62B65
 P 1300 3350
@@
 	1000 5300 1250 5300
 $Comp
-L power:GND #PWR0140
+L dotmatrix_64x48-rescue:GND-power #PWR0140
 U 1 1 5BC71055
 P 1250 5600
@@
 $EndComp
 $Comp
-L device:C C76
+L dotmatrix_64x48-rescue:C-device C76
 U 1 1 5BC7105F
 P 1250 5450
@@
 	1250 5300 1600 5300
 $Comp
-L power:GND #PWR?
+L dotmatrix_64x48-rescue:GND-power #PWR?
 U 1 1 5BC7F814
 P 2600 6100
@@
 DC_IN_N
 $Comp
-L device:C C2
+L dotmatrix_64x48-rescue:C-device C2
 U 1 1 5BDA55B3
 P 6350 3750
@@
 $EndComp
 $Comp
-L power:GND #PWR?
+L dotmatrix_64x48-rescue:GND-power #PWR?
 U 1 1 5BDA8B7D
 P 6350 3900

Commit message: Merged production-1.0's LED matrix onto current design.
Parts:
- Q29, Q30: footprint TO_SOT_Packages_SMD:SOT-23_Handsoldering -> Package_TO_SOT_SMD:SOT-23_Handsoldering
- R105, R114, R115: footprint Resistors_SMD:R_0603_HandSoldering -> Resistor_SMD:R_0603_1608Metric_Pad1.05x0.95mm_HandSolder
Changed lines of the file:
@@
 F 0 "Q29" H 8691 3204 50  0000 L CNN
 F 1 "AO3401" H 8691 3295 50  0000 L CNN
-F 2 "TO_SOT_Packages_SMD:SOT-23_Handsoldering" H 8700 3350 50  0001 C CNN
+F 2 "Package_TO_SOT_SMD:SOT-23_Handsoldering" H 8700 3350 50  0001 C CNN
 F 3 "" H 8500 3250 50  0000 C CNN
 	1    8500 3250
@@
 F 0 "Q30" H 9540 3946 50  0000 L CNN
 F 1 "Q_NPN_BEC" H 9540 3855 50  0000 L CNN
-F 2 "TO_SOT_Packages_SMD:SOT-23_Handsoldering" H 9541 3809 50  0001 L CNN
+F 2 "Package_TO_SOT_SMD:SOT-23_Handsoldering" H 9541 3809 50  0001 L CNN
 F 3 "" H 9350 3900 50  0000 C CNN
 	1    9350 3900
@@
 F 0 "R114" V 8950 3800 50  0000 L CNN
 F 1 "4.7k" V 9050 3850 50  0000 L CNN
-F 2 "Resistors_SMD:R_0603_HandSoldering" V 8880 3900 50  0001 C CNN
+F 2 "Resistor_SMD:R_0603_1608Metric_Pad1.05x0.95mm_HandSolder" V 8880 3900 50  0001 C CNN
 F 3 "" H 8950 3900 50  0000 C CNN
 	1    8950 3900
@@
 F 0 "R105" V 8250 3800 50  0000 L CNN
 F 1 "10R" V 8350 3850 50  0000 L CNN
-F 2 "Resistors_SMD:R_0603_HandSoldering" V 8180 3900 50  0001 C CNN
+F 2 "Resistor_SMD:R_0603_1608Metric_Pad1.05x0.95mm_HandSolder" V 8180 3900 50  0001 C CNN
 F 3 "" H 8250 3900 50  0000 C CNN
 	1    8250 3900
@@
 F 0 "R115" H 9520 3546 50  0000 L CNN
 F 1 "10R" H 9520 3455 50  0000 L CNN
-F 2 "Resistors_SMD:R_0603_HandSoldering" V 9380 3500 50  0001 C CNN
+F 2 "Resistor_SMD:R_0603_1608Metric_Pad1.05x0.95mm_HandSolder" V 9380 3500 50  0001 C CNN
 F 3 "" H 9450 3500 50  0000 C CNN
 	1    9450 3500

Commit message: Before removing old style stitching vias
Parts:
- added C18, C19, C3, C36, C63: 10u 10V, Capacitor_SMD:C_0603_1608Metric_Pad1.05x0.95mm_HandSolder, symbol dotmatrix_64x48-rescue:C-device
- added U14: AP1117-33, Package_TO_SOT_SMD:SOT-223-3_TabPin2, symbol regul:AP1117-33
- C2, C34, C57, C59, C60, C61: value 10u -> 10u 10V; footprint Capacitors_SMD:C_1206_HandSoldering -> Capacitor_SMD:C_0603_1608Metric_Pad1.05x0.95mm_HandSolder
- C55: footprint Capacitors_SMD:C_0805_HandSoldering -> Capacitor_SMD:C_0603_1608Metric_Pad1.05x0.95mm_HandSolder
- R38: value 100k -> 75k
- R39: value 22k -> 10k
Connections:
- wire segments 115 -> 122
Other:
- note added: "5V 2A"
- note added: "Vout = .596*(75.0/(10)+1) = 5.066"
- note removed: "3V3 2A"
- note removed: "Vout = .596*(100000.0/(22000)+1) = 3.305090909090909"
- moved on the sheet: C62, C65, L4, Q29, Q30, R105, R114, R115
