File: IR_Sensor.sch (KiCad schematic (older format))
At the start: 27 parts, among them Q1 Q_NPN_BCE RN5006, Q3 NJL7302L-F3, U12 AE-BME280, U17 OSRB38C9AA, U18 BME280

Commit message: This is the MazoClock hw 4.0 series; Uses ESP32 processor instead of ESP8266 used in prior MazoClock hw 3.0 series.
Parts:
- added J11: Conn_01x04_Female, Pin_Headers:Pin_Header_Straight_1x04_Pitch2.54mm, symbol Conn_01x04_Female
Connections:
- wire segments 66 -> 70
Changed lines of the file:
@@
 LIBS:mechanical
 LIBS:microchip_pic32mcu
+LIBS:ESP32-footprints-Shem-Lib
 LIBS:dotmatrix_64x48-cache
 EELAYER 26 0
@@
 SCL
 $Comp
-L GND #PWR32
+L GND #PWR032
 U 1 1 57A9F4D2
 P 7800 2400
-F 0 "#PWR32" H 7800 2150 50  0001 C CNN
+F 0 "#PWR032" H 7800 2150 50  0001 C CNN
 F 1 "GND" H 7805 2227 50  0000 C CNN
 F 2 "" H 7800 2400 50  0000 C CNN
@@
 ESPVDD
 $Comp
-L GND #PWR34
+L GND #PWR034
 U 1 1 57B917E4
 P 1950 2600
-F 0 "#PWR34" H 1950 2350 50  0001 C CNN
+F 0 "#PWR034" H 1950 2350 50  0001 C CNN
 F 1 "GND" H 1955 2427 50  0000 C CNN
 F 2 "" H 1950 2600 50  0000 C CNN
@@
 SCL
 $Comp
-L GND #PWR27
+L GND #PWR027
 U 1 1 57BBCCD6
 P 5950 1500
-F 0 "#PWR27" H 5950 1250 50  0001 C CNN
+F 0 "#PWR027" H 5950 1250 50  0001 C CNN
 F 1 "GND" H 5955 1327 50  0000 C CNN
 F 2 "" H 5950 1500 50  0000 C CNN
@@
 $EndComp
 $Comp
-L GND #PWR28
+L GND #PWR028
 U 1 1 57BBCDE5
 P 4950 1600
-F 0 "#PWR28" H 4950 1350 50  0001 C CNN
+F 0 "#PWR028" H 4950 1350 50  0001 C CNN
 F 1 "GND" H 4955 1427 50  0000 C CNN
 F 2 "" H 4950 1600 50  0000 C CNN
@@
 $EndComp
 $Comp
-L GND #PWR29
+L GND #PWR029
 U 1 1 57BBCFE9
 P 4950 1800
-F 0 "#PWR29" H 4950 1550 50  0001 C CNN
+F 0 "#PWR029" H 4950 1550 50  0001 C CNN
 F 1 "GND" H 4955 1627 50  0000 C CNN
 F 2 "" H 4950 1800 50  0000 C CNN
@@
 ESPVDD
 $Comp
-L GND #PWR31
+L GND #PWR031
 U 1 1 57BBE379
 P 4600 2150
-F 0 "#PWR31" H 4600 1900 50  0001 C CNN
+F 0 "#PWR031" H 4600 1900 50  0001 C CNN
 F 1 "GND" H 4605 1977 50  0000 C CNN
 F 2 "" H 4600 2150 50  0000 C CNN
@@
 $EndComp
 $Comp
-L GND #PWR35
+L GND #PWR035
 U 1 1 5818B2A5
 P 3900 3700
-F 0 "#PWR35" H 3900 3450 50  0001 C CNN
+F 0 "#PWR035" H 3900 3450 50  0001 C CNN
 F 1 "GND" H 3905 3527 50  0000 C CNN
 F 2 "" H 3900 3700 50  0000 C CNN
@@
 	4050 2600 3900 2600
 $Comp
-L GND #PWR33
+L GND #PWR033
 U 1 1 582753E6
 P 8100 2400
-F 0 "#PWR33" H 8100 2150 50  0001 C CNN
+F 0 "#PWR033" H 8100 2150 50  0001 C CNN
 F 1 "GND" H 8105 2227 50  0000 C CNN
 F 2 "" H 8100 2400 50  0000 C CNN
@@
 $EndComp
 $Comp
-L GND #PWR30
+L GND #PWR030
 U 1 1 582DE087
 P 4150 2150
-F 0 "#PWR30" H 4150 1900 50  0001 C CNN
+F 0 "#PWR030" H 4150 1900 50  0001 C CNN
 F 1 "GND" H 4155 1977 50  0000 C CNN
 F 2 "" H 4150 2150 50  0000 C CNN
@@
 $EndComp
 $Comp
-L GND #PWR37
+L GND #PWR037
 U 1 1 59A7F67D
 P 4450 5800
-F 0 "#PWR37" H 4450 5550 50  0001 C CNN
+F 0 "#PWR037" H 4450 5550 50  0001 C CNN
 F 1 "GND" H 4450 5650 50  0000 C CNN
 F 2 "" H 4450 5800 50  0000 C CNN
@@
 $EndComp
 $Comp
-L VCC #PWR36
+L VCC #PWR036
 U 1 1 59A7F683
 P 4950 5000
-F 0 "#PWR36" H 4950 4850 50  0001 C CNN
+F 0 "#PWR036" H 4950 4850 50  0001 C CNN
 F 1 "VCC" H 4967 5173 50  0000 C CNN
 F 2 "" H 4950 5000 50  0000 C CNN
@@
 $EndComp
 $Comp
-L GND #PWR38
+L GND #PWR038
 U 1 1 59A7F6BB
 P 2600 5850
-F 0 "#PWR38" H 2600 5600 50  0001 C CNN
+F 0 "#PWR038" H 2600 5600 50  0001 C CNN
 F 1 "GND" H 2605 5677 50  0000 C CNN
 F 2 "" H 2600 5850 50  0000 C CNN
@@
 	6000 5750 6000 5450
 Connection ~ 5600 5750
+$Comp
+L Conn_01x04_Female J11
+U 1 1 59E053A4
+P 8850 4700
+F 0 "J11" H 8877 4676 50  0000 L CNN
+F 1 "Conn_01x04_Female" H 8877 4585 50  0000 L CNN
+F 2 "Pin_Headers:Pin_Header_Straight_1x04_Pitch2.54mm" H 8850 4700 50  0001 C CNN
+F 3 "" H 8850 4700 50  0001 C CNN
+	1    8850 4700
+	1    0    0    -1
+$EndComp
+Text GLabel 8400 4600 0    60   Input ~ 0
+IR_IN
+Text GLabel 8400 4700 0    60   Input ~ 0
+IR_OUT
+$Comp
+L GND #PWR0144
+U 1 1 59E054D0
+P 8600 4800
+F 0 "#PWR0144" H 8600 4550 50  0001 C CNN
+F 1 "GND" H 8605 4627 50  0000 C CNN
+F 2 "" H 8600 4800 50  0000 C CNN
+F 3 "" H 8600 4800 50  0000 C CNN
+	1    8600 4800
+	0    1    1    0
+$EndComp
+Text GLabel 8400 4900 0    60   Input ~ 0
+E_AIN
+Wire Wire Line
+	8400 4600 8650 4600
+Wire Wire Line
+	8650 4700 8400 4700
+Wire Wire Line
+	8400 4900 8650 4900
+Wire Wire Line
+	8600 4800 8650 4800
 $EndSCHEMATC

Commit message: Updated to kicad 6.0.0 rc; removed outdated gerber files; Schematic is not complete
Parts:
- C2, C3, C32, C36, C4, C58, C63, C68: symbol C -> device:C
- C29: symbol CP -> device:CP
- CONN3: symbol CONN_01X03 -> Connector:Conn_01x03
- D12: symbol D_TVS_x2_AAC -> device:D_TVS_x2_AAC
- D14: symbol D_Schottky_Small -> device:D_Schottky_Small
- J11: symbol Conn_01x04_Female -> Connector:Conn_01x04_Female
- L6: symbol Ferrite_Bead_Small -> device:Ferrite_Bead_Small
- Q1: symbol Q_NPN_BCE -> device:Q_NPN_BCE
- Q3: symbol OPTO_NPN2 -> DeeComponents:OPTO_NPN2
- R12, R123, R124, R129, R40, R42, R43, R44, R45: symbol R -> device:R
- U12: symbol AE-BME280 -> DeeComponents:AE-BME280
- U17: symbol OSRB38C9AA -> DeeComponents:OSRB38C9AA
- U18: symbol BME280 -> DeeComponents:BME280
Connections:
- wire segments 70 -> 98

Commit message: Heavily modifying; Matrix nets under construction
Parts:
- removed C29: 100u, components:C_Radial_D6.3_L11.2_P2.5_hand_soldering, symbol device:CP
- removed J11: Conn_01x04_Female, Pin_Headers:Pin_Header_Straight_1x04_Pitch2.54mm, symbol Connector:Conn_01x04_Female
- added C1, C20: 10u, Capacitors_SMD:C_1206_HandSoldering, symbol device:C
- added C18: 0.1u, Capacitors_SMD:C_0603_HandSoldering, symbol device:C
- added C19: 1u, Capacitors_SMD:C_0603_HandSoldering, symbol device:C
- added LED49, LED50, LED51: IR, LEDs:LED_D5.0mm, symbol device:LED
- added LS1: Speaker, components:SPK_35mm_20mm_RECTANGLE_MOUNT, symbol device:Speaker
- added R100: 0, Resistors_SMD:R_0603_HandSoldering, symbol device:R
- added R16, R17, R26: 10R, Resistors_SMD:R_0603_HandSoldering, symbol device:R
- added R99: 100k, Resistors_SMD:R_0603_HandSoldering, symbol device:R
- added U14: MAX98357, components:QFN-16-1EP_3x3mm_Pitch0.5mm-handsoldering, symbol DeeComponents:MAX98357
- Q1: footprint TO_SOT_Packages_SMD:SOT89-3_Housing_Handsoldering -> TO_SOT_Packages_SMD:SOT-89-3_Handsoldering
- Q3: footprint LEDs:LED-3MM -> LEDs:LED_D3.0mm
Connections:
- net labels added: I2S_SPK_BCLK, I2S_SPK_DATA, I2S_SPK_GAIN0, I2S_SPK_GAIN1, I2S_SPK_LRCLK, LEDLOGICVDD
- wire segments 98 -> 152

Commit message: Almost all components has placed.
Parts:
- removed C36: 1u, Capacitors_SMD:C_0603_HandSoldering, symbol device:C
- removed C63: 0.1u, Capacitors_SMD:C_0603_HandSoldering, symbol device:C
- removed U18: BME280, components:BME280-handsoldering, symbol DeeComponents:BME280
- LS1: footprint components:SPK_35mm_20mm_RECTANGLE_MOUNT -> Wire_Connections_Bridges:WireConnection_1.50mmDrill
Connections:
- net labels added: FILT_VDD, IRLED_K, LEDVDD, SPK_N, SPK_P
- net labels removed: VCC
- wire segments 152 -> 144
