File: IR_Sensor.sch (KiCad schematic (older format))
At the start: 37 parts, among them Q1 Q_NPN_BCE RN5006, Q3 NJL7302L-F3, U12 AE-BME280, U14 MAX98357, U17 OSRB38C9AA

Commit message: Too less PCB space.
Parts:
- removed C2: 0.1u, Capacitors_SMD:C_0603_HandSoldering, symbol device:C
- removed CONN3: Push_Terminal_3P_2.54, components:Push_Terminal_3P_2.54, symbol Connector:Conn_01x03
- removed D12: PESD12VL2BT, TO_SOT_Packages_SMD:SOT-23_Handsoldering, symbol device:D_TVS_x2_AAC
- removed LED50, LED51: IR, LEDs:LED_D5.0mm, symbol device:LED
- removed Q1: Q_NPN_BCE RN5006, TO_SOT_Packages_SMD:SOT-89-3_Handsoldering, symbol device:Q_NPN_BCE
- removed R100: 0, Resistors_SMD:R_0603_HandSoldering, symbol device:R
- removed U14: MAX98357, components:QFN-16-1EP_3x3mm_Pitch0.5mm-handsoldering, symbol DeeComponents:MAX98357
- added C36: 1u, Capacitors_SMD:C_0603_HandSoldering, symbol device:C
- added C63, C78, C83, C84, C85, C86: 0.1u 16V, Capacitors_SMD:C_0603_HandSoldering, symbol device:C
- added C79, C80: 1u 16V, Capacitors_SMD:C_0603_HandSoldering, symbol device:C
- added C81, C82: 10u 16V, Capacitors_SMD:C_1206_HandSoldering, symbol device:C
- added CONN4: Pin_Header_Straight_1x05_Pitch2.54mm, Pin_Headers:Pin_Header_Straight_1x05_Pitch2.54mm, symbol Connector:Conn_01x05
- added J4: Conn_01x02, Wire_Connections_Bridges:WireConnection_1.50mmDrill, symbol Connector:Conn_01x02
- added Q1: AO3401, TO_SOT_Packages_SMD:SOT-23_Handsoldering, symbol device:Q_PMOS_GSD
- added Q31: Q_NPN_BEC, TO_SOT_Packages_SMD:SOT-23_Handsoldering, symbol device:Q_NPN_BEC
- added R1: 4.7k, Resistors_SMD:R_0603_HandSoldering, symbol device:R
- added R139, R140: 10R, Resistors_SMD:R_0603_HandSoldering, symbol device:R
- added U14: TAS5720, components:QFN-32-1EP_4x4mm_Pitch0.4mm_Handsoldering, symbol DeeComponents:TAS5720
- added U26: CM1293A-04SO, TO_SOT_Packages_SMD:SOT-23-6_Handsoldering, symbol ESD_Protection:SRV05-4
- C18: value 0.1u -> 1u
- C20: value 10u -> 1u; footprint Capacitors_SMD:C_1206_HandSoldering -> Capacitors_SMD:C_0603_HandSoldering
- LED49: footprint LEDs:LED_D5.0mm -> LEDs:LED_PLCC_2835_Handsoldering
- R12: value 1k -> 10k
- R42: value 10k DNI -> 10k
- R99: value 100k -> 10k
Connections:
- net labels added: I2S_SPK_MCLK, IRLED_A, VCC
- net labels removed: ESPVDD, I2S_SPK_GAIN0, I2S_SPK_GAIN1, IRLED_K
- wire segments 144 -> 192
Other:
- note added: "12V"

Commit message: Added stereo power amplifier
Parts:
- removed C18, C19, C20, C36: 1u, Capacitors_SMD:C_0603_HandSoldering, symbol device:C
- removed C3: 220p, Capacitors_SMD:C_0603_HandSoldering, symbol device:C
- removed C63, C78, C83, C84, C85, C86: 0.1u 16V, Capacitors_SMD:C_0603_HandSoldering, symbol device:C
- removed C79, C80: 1u 16V, Capacitors_SMD:C_0603_HandSoldering, symbol device:C
- removed C81, C82: 10u 16V, Capacitors_SMD:C_1206_HandSoldering, symbol device:C
- removed J4: Conn_01x02, Wire_Connections_Bridges:WireConnection_1.50mmDrill, symbol Connector:Conn_01x02
- removed LS1: Speaker, Wire_Connections_Bridges:WireConnection_1.50mmDrill, symbol device:Speaker
- removed Q31: Q_NPN_BEC, TO_SOT_Packages_SMD:SOT-23_Handsoldering, symbol device:Q_NPN_BEC
- removed R12, R42, R99: 10k, Resistors_SMD:R_0603_HandSoldering, symbol device:R
- removed U14: TAS5720, components:QFN-32-1EP_4x4mm_Pitch0.4mm_Handsoldering, symbol DeeComponents:TAS5720
Connections:
- net labels removed: SPK_N, SPK_P, VCC
- wire segments 192 -> 93
Other:
- note removed: "12V"

Commit message: Switched to new kicad libraries
Parts:
- C1, C32, C4, C58, C68: symbol device:C -> dotmatrix_64x48-rescue:C-device
- CONN4: symbol Connector:Conn_01x05 -> dotmatrix_64x48-rescue:Conn_01x05-Connector
- D14: symbol device:D_Schottky_Small -> dotmatrix_64x48-rescue:D_Schottky_Small-device
- L6: symbol device:Ferrite_Bead_Small -> dotmatrix_64x48-rescue:Ferrite_Bead_Small-device
- LED49: symbol device:LED -> dotmatrix_64x48-rescue:LED-device
- Q1: symbol device:Q_PMOS_GSD -> dotmatrix_64x48-rescue:Q_PMOS_GSD-device
- R1, R123, R124, R129, R139, R140, R16, R17, R26, R40, R43, R44, R45: symbol device:R -> dotmatrix_64x48-rescue:R-device
- U26: symbol ESD_Protection:SRV05-4 -> dotmatrix_64x48-rescue:SRV05-4-ESD_Protection
Changed lines of the file:
@@
 SCL
 $Comp
-L power:GND #PWR032
+L dotmatrix_64x48-rescue:GND-power #PWR032
 U 1 1 57A9F4D2
 P 7750 1500
@@
 $EndComp
 $Comp
-L device:R R40
+L dotmatrix_64x48-rescue:R-device R40
 U 1 1 57B8F5DB
 P 1350 950
@@
 $EndComp
 $Comp
-L power:GND #PWR034
+L dotmatrix_64x48-rescue:GND-power #PWR034
 U 1 1 57B917E4
 P 1850 1800
@@
 $EndComp
 $Comp
-L device:C C32
+L dotmatrix_64x48-rescue:C-device C32
 U 1 1 57B9F506
 P 2000 1600
@@
 IR_IN
 $Comp
-L device:R R43
+L dotmatrix_64x48-rescue:R-device R43
 U 1 1 5818B29E
 P 4900 950
@@
 $EndComp
 $Comp
-L power:GND #PWR035
+L dotmatrix_64x48-rescue:GND-power #PWR035
 U 1 1 5818B2A5
 P 4900 1900
@@
 Longer lead side
 $Comp
-L device:R R44
+L dotmatrix_64x48-rescue:R-device R44
 U 1 1 581BE703
 P 5100 950
@@
 $EndComp
 $Comp
-L device:R R45
+L dotmatrix_64x48-rescue:R-device R45
 U 1 1 581BE747
 P 5300 950
@@
 	5050 800  4900 800
 $Comp
-L power:GND #PWR033
+L dotmatrix_64x48-rescue:GND-power #PWR033
 U 1 1 582753E6
 P 8050 1500
@@
 $EndComp
 $Comp
-L device:R R123
+L dotmatrix_64x48-rescue:R-device R123
 U 1 1 5836657C
 P 2550 1250
@@
 $EndComp
 $Comp
-L device:R R124
+L dotmatrix_64x48-rescue:R-device R124
 U 1 1 583665D6
 P 2550 1350
@@
 Connection ~ 2750 1350
 $Comp
-L device:C C68
+L dotmatrix_64x48-rescue:C-device C68
 U 1 1 583D96AC
 P 3000 1500
@@
 Connection ~ 3000 1350
 $Comp
-L device:R R129
+L dotmatrix_64x48-rescue:R-device R129
 U 1 1 594A71FB
 P 4600 1550
@@
 $EndComp
 $Comp
-L device:C C58
+L dotmatrix_64x48-rescue:C-device C58
 U 1 1 5818B2AB
 P 4350 1550
@@
 Connection ~ 4600 1800
 $Comp
-L device:C C4
+L dotmatrix_64x48-rescue:C-device C4
 U 1 1 59A7F689
 P 2100 2900
@@
 IR_OUT
 $Comp
-L device:Ferrite_Bead_Small L6
+L dotmatrix_64x48-rescue:Ferrite_Bead_Small-device L6
 U 1 1 59A7F6A6
 P 1750 2750
@@
 $EndComp
 $Comp
-L device:D_Schottky_Small D14
+L dotmatrix_64x48-rescue:D_Schottky_Small-device D14
 U 1 1 59A7F6B4
 P 1550 3550
@@
 $EndComp
 $Comp
-L power:GND #PWR038
+L dotmatrix_64x48-rescue:GND-power #PWR038
 U 1 1 59A7F6BB
 P 1550 3650
@@
 	1550 3300 1700 3300
 $Comp
-L device:LED LED49
+L dotmatrix_64x48-rescue:LED-device LED49
 U 1 1 5BB50E0E
 P 4100 3350
@@
 $EndComp
 $Comp
-L device:R R16
+L dotmatrix_64x48-rescue:R-device R16
 U 1 1 5BB5618C
 P 3750 2750
@@
 $EndComp
 $Comp
-L device:C C?
+L dotmatrix_64x48-rescue:C-device C?
 U 1 1 5BBD3352
 P 2350 1550
@@
 	1850 2750 2100 2750
 $Comp
-L power:GND #PWR0144
+L dotmatrix_64x48-rescue:GND-power #PWR0144
 U 1 1 5BE206B6
 P 2100 3050
@@
 Connection ~ 2100 2750
 $Comp
-L device:R R1
+L dotmatrix_64x48-rescue:R-device R1
 U 1 1 5BDCDF20
 P 2700 2900
@@
 I2S_SPK_MCLK
 $Comp
-L Connector:Conn_01x05 CONN4
+L dotmatrix_64x48-rescue:Conn_01x05-Connector CONN4
 U 1 1 5C135F0D
 P 10500 4550
@@
 $EndComp
 $Comp
-L power:GND #PWR0154
+L dotmatrix_64x48-rescue:GND-power #PWR0154
 U 1 1 5C14CA3D
 P 8400 4750
@@
 $EndComp
 $Comp
-L ESD_Protection:SRV05-4 U?
+L dotmatrix_64x48-rescue:SRV05-4-ESD_Protection U?
 U 1 1 5C1694C3
 P 9400 5650
@@
 $EndComp
 $Comp
-L power:GND #PWR?
+L dotmatrix_64x48-rescue:GND-power #PWR?
 U 1 1 5C1694C9
 P 9400 6150
@@
 	1350 700  1350 650
 $Comp
-L device:R R26
+L dotmatrix_64x48-rescue:R-device R26
 U 1 1 5BE01611
 P 3850 2750
@@
 	3850 2900 3750 2900
 $Comp
-L device:R R139
+L dotmatrix_64x48-rescue:R-device R139
 U 1 1 5BDF6F9A
 P 3950 2750
@@
 $EndComp
 $Comp
-L device:R R140
+L dotmatrix_64x48-rescue:R-device R140
 U 1 1 5BDF6FA4
 P 4050 2750
@@
 	3950 2600 3850 2600
 $Comp
-L device:R R17
+L dotmatrix_64x48-rescue:R-device R17
 U 1 1 5BE1614C
 P 1850 3300
@@
 	3300 2600 3750 2600
 $Comp
-L device:Q_PMOS_GSD Q?
+L dotmatrix_64x48-rescue:Q_PMOS_GSD-device Q?
 U 1 1 5BE39F04
 P 2400 2850
@@
 	2400 3050 2400 3300
 $Comp
-L power:GND #PWR037
+L dotmatrix_64x48-rescue:GND-power #PWR037
 U 1 1 5BE44566
 P 3400 3500

Commit message: Layout fixup
Parts:
- added C20: 1u, Capacitor_SMD:C_0603_1608Metric_Pad1.05x0.95mm_HandSolder, symbol dotmatrix_64x48-rescue:C-device
Connections:
- wire segments 93 -> 99
Changed lines of the file:
@@
 L dotmatrix_64x48-rescue:GND-power #PWR032
 U 1 1 57A9F4D2
-P 7750 1500
-F 0 "#PWR032" H 7750 1250 50  0001 C CNN
-F 1 "GND" H 7755 1327 50  0000 C CNN
-F 2 "" H 7750 1500 50  0000 C CNN
-F 3 "" H 7750 1500 50  0000 C CNN
-	1    7750 1500
-	1    0    0    -1
-$EndComp
-Text GLabel 7650 1500 3    60   Input ~ 0
+P 7750 1750
+F 0 "#PWR032" H 7750 1500 50  0001 C CNN
+F 1 "GND" H 7755 1577 50  0000 C CNN
+F 2 "" H 7750 1750 50  0000 C CNN
+F 3 "" H 7750 1750 50  0000 C CNN
+	1    7750 1750
+	1    0    0    -1
+$EndComp
+Text GLabel 7400 1800 3    60   Input ~ 0
 LEDLOGICVDD
 NoConn ~ 7850 1500
@@
 Wire Wire Line
 	2700 3500 3400 3500
+$Comp
+L dotmatrix_64x48-rescue:C-device C20
+U 1 1 5BF3C5D2
+P 7550 1650
+F 0 "C20" H 7665 1696 50  0000 L CNN
+F 1 "1u" H 7665 1605 50  0000 L CNN
+F 2 "Capacitor_SMD:C_0603_1608Metric_Pad1.05x0.95mm_HandSolder" H 7665 1559 50  0001 L CNN
+F 3 "" H 7550 1650 50  0000 C CNN
+	1    7550 1650
+	0    1    1    0
+$EndComp
+Wire Wire Line
+	7750 1750 7750 1650
+Wire Wire Line
+	7650 1500 7400 1500
+Wire Wire Line
+	7400 1500 7400 1650
+Connection ~ 7400 1650
+Wire Wire Line
+	7400 1650 7400 1800
+Wire Wire Line
+	7700 1650 7750 1650
+Connection ~ 7750 1650
+Wire Wire Line
+	7750 1650 7750 1500
 $EndSCHEMATC

Commit message: Merged production-1.0's LED matrix onto current design.
Parts:
- C1: footprint Capacitors_SMD:C_1206_HandSoldering -> Capacitor_SMD:C_1206_3216Metric_Pad1.42x1.75mm_HandSolder
- C32: footprint Capacitors_SMD:C_0603_HandSoldering -> Capacitor_SMD:C_0603_1608Metric_Pad1.05x0.95mm_HandSolder
- Q3: footprint LEDs:LED_D3.0mm -> LED_THT:LED_D3.0mm
- R129, R40, R43, R44, R45: footprint Resistors_SMD:R_0603_HandSoldering -> Resistor_SMD:R_0603_1608Metric_Pad1.05x0.95mm_HandSolder
Changed lines of the file:
@@
 F 0 "R40" V 1350 850 50  0000 L CNN
 F 1 "22k" V 1250 850 50  0000 L CNN
-F 2 "Resistors_SMD:R_0603_HandSoldering" V 1280 950 50  0001 C CNN
+F 2 "Resistor_SMD:R_0603_1608Metric_Pad1.05x0.95mm_HandSolder" V 1280 950 50  0001 C CNN
 F 3 "" H 1350 950 50  0000 C CNN
 	1    1350 950
@@
 F 0 "C32" H 2115 1646 50  0000 L CNN
 F 1 "1u" H 2115 1555 50  0000 L CNN
-F 2 "Capacitors_SMD:C_0603_HandSoldering" H 2115 1509 50  0001 L CNN
+F 2 "Capacitor_SMD:C_0603_1608Metric_Pad1.05x0.95mm_HandSolder" H 2115 1509 50  0001 L CNN
 F 3 "" H 2000 1600 50  0000 C CNN
 	1    2000 1600
@@
 F 0 "R43" V 4900 900 50  0000 L CNN
 F 1 "10k" V 5000 850 50  0000 L CNN
-F 2 "Resistors_SMD:R_0603_HandSoldering" V 4830 950 50  0001 C CNN
+F 2 "Resistor_SMD:R_0603_1608Metric_Pad1.05x0.95mm_HandSolder" V 4830 950 50  0001 C CNN
 F 3 "" H 4900 950 50  0000 C CNN
 	1    4900 950
@@
 F 0 "Q3" H 4976 1641 50  0000 L CNN
 F 1 "NJL7302L-F3" H 4976 1550 50  0000 L CNN
-F 2 "LEDs:LED_D3.0mm" H 4976 1459 50  0000 L CNN
+F 2 "LED_THT:LED_D3.0mm" H 4976 1459 50  0000 L CNN
 F 3 "" H 4800 1550 50  0000 C CNN
 	1    4800 1550
@@
 F 0 "R44" V 5100 900 50  0000 L CNN
 F 1 "10k" V 5200 850 50  0000 L CNN
-F 2 "Resistors_SMD:R_0603_HandSoldering" V 5030 950 50  0001 C CNN
+F 2 "Resistor_SMD:R_0603_1608Metric_Pad1.05x0.95mm_HandSolder" V 5030 950 50  0001 C CNN
 F 3 "" H 5100 950 50  0000 C CNN
 	1    5100 950
@@
 F 0 "R45" V 5300 900 50  0000 L CNN
 F 1 "10k" V 5400 850 50  0000 L CNN
-F 2 "Resistors_SMD:R_0603_HandSoldering" V 5230 950 50  0001 C CNN
+F 2 "Resistor_SMD:R_0603_1608Metric_Pad1.05x0.95mm_HandSolder" V 5230 950 50  0001 C CNN
 F 3 "" H 5300 950 50  0000 C CNN
 	1    5300 950
@@
 F 0 "R129" V 4600 1450 50  0000 L CNN
 F 1 "10k" V 4700 1450 50  0000 L CNN
-F 2 "Resistors_SMD:R_0603_HandSoldering" V 4530 1550 50  0001 C CNN
+F 2 "Resistor_SMD:R_0603_1608Metric_Pad1.05x0.95mm_HandSolder" V 4530 1550 50  0001 C CNN
 F 3 "" H 4600 1550 50  0000 C CNN
 	1    4600 1550
@@
 F 0 "C1" H 2500 1550 50  0000 L CNN
 F 1 "10u" H 2500 1450 50  0000 L CNN
-F 2 "Capacitors_SMD:C_1206_HandSoldering" H 2465 1459 50  0001 L CNN
+F 2 "Capacitor_SMD:C_1206_3216Metric_Pad1.42x1.75mm_HandSolder" H 2465 1459 50  0001 L CNN
 F 3 "" H 2350 1550 50  0000 C CNN
 	1    2350 1550

Commit message: Before removing old style stitching vias
Parts:
- C1: value 10u -> 10u 10V; footprint Capacitor_SMD:C_1206_3216Metric_Pad1.42x1.75mm_HandSolder -> Capacitor_SMD:C_0603_1608Metric_Pad1.05x0.95mm_HandSolder
Connections:
- net labels added: LED1642VDD
- wire segments 99 -> 98
Changed lines of the file:
@@
 AR Path="/57BB11DB/5BBD3352" Ref="C1"  Part="1"
 F 0 "C1" H 2500 1550 50  0000 L CNN
-F 1 "10u" H 2500 1450 50  0000 L CNN
-F 2 "Capacitor_SMD:C_1206_3216Metric_Pad1.42x1.75mm_HandSolder" H 2465 1459 50  0001 L CNN
+F 1 "10u 10V" H 2500 1450 50  0000 L CNN
+F 2 "Capacitor_SMD:C_0603_1608Metric_Pad1.05x0.95mm_HandSolder" H 2465 1459 50  0001 L CNN
 F 3 "" H 2350 1550 50  0000 C CNN
 	1    2350 1550
@@
 Wire Wire Line
 	9950 4650 10300 4650
-Text GLabel 10250 5050 2    60   Input ~ 0
-LEDLOGICVDD
 Wire Wire Line
 	9400 5150 10250 5150
-Wire Wire Line
-	10250 5150 10250 5050
 Text GLabel 1350 650  0    60   Input ~ 0
 LEDLOGICVDD
@@
 Wire Wire Line
 	7750 1650 7750 1500
+Text GLabel 10250 5150 2    60   Input ~ 0
+LED1642VDD
 $EndSCHEMATC

Commit message: Almost done drawing pcb tracks
Parts:
- removed L6: BLM21PG331SN 300R@100MHz, Capacitors_SMD:C_0805_HandSoldering, symbol dotmatrix_64x48-rescue:Ferrite_Bead_Small-device
Connections:
- wire segments 98 -> 97
Changed lines of the file:
@@
 IR_OUT
-$Comp
-L dotmatrix_64x48-rescue:Ferrite_Bead_Small-device L6
-U 1 1 59A7F6A6
-P 1750 2750
-F 0 "L6" V 1572 2750 50  0000 C CNN
-F 1 "BLM21PG331SN 300R@100MHz" V 1450 2750 50  0000 C CNN
-F 2 "Capacitors_SMD:C_0805_HandSoldering" H 1750 2750 50  0001 C CNN
-F 3 "" H 1750 2750 50  0000 C CNN
-	1    1750 2750
-	0    -1   1    0
-$EndComp
 $Comp
 L dotmatrix_64x48-rescue:D_Schottky_Small-device D14
@@
 Text Label 3300 650  0    50   ~ 0
 FILT_VDD
-Wire Wire Line
-	1350 2750 1650 2750
-Wire Wire Line
-	1850 2750 2100 2750
 $Comp
 L dotmatrix_64x48-rescue:GND-power #PWR0144
@@
 Text GLabel 10250 5150 2    60   Input ~ 0
 LED1642VDD
+Wire Wire Line
+	1350 2750 2100 2750
 $EndSCHEMATC
