File: column_driver.sch (KiCad schematic (older format))
At the start: 41 parts, among them U10 LED1642GW, U3 LED1642GW, U4 LED1642GW, U5 LED1642GW, U6 LED1642GW, U7 LED1642GW, U8 LED1642GW, U9 LED1642GW

Commit message: Modified to use matrix LEDs; Components layout has almost done, tracks and traces not yet.
Parts:
- added Q29: AO3401, TO_SOT_Packages_SMD:SOT-23_Handsoldering, symbol Q_PMOS_GSD
- added Q30: Q_NPN_BEC, TO_SOT_Packages_SMD:SOT-23_Handsoldering, symbol Q_NPN_BEC
- added R146: 10R, Resistors_SMD:R_0603_HandSoldering, symbol R
- added R147: 4.7k, Resistors_SMD:R_0603_HandSoldering, symbol R
Connections:
- net labels added: LED1642VDD, P_LED1642_RST
- wire segments 78 -> 86

Commit message: This is the MazoClock hw 4.0 series; Uses ESP32 processor instead of ESP8266 used in prior MazoClock hw 3.0 series.
Connections:
- net labels added: D_LED1642_RST
- net labels removed: P_LED1642_RST
Changed lines of the file:
@@
 LIBS:mechanical
 LIBS:microchip_pic32mcu
+LIBS:ESP32-footprints-Shem-Lib
 LIBS:dotmatrix_64x48-cache
 EELAYER 26 0
@@
 Connection ~ 7650 5250
 $Comp
-L GND #PWR62
+L GND #PWR062
 U 1 1 5943C2CA
 P 8850 5150
-F 0 "#PWR62" H 8850 4900 50  0001 C CNN
+F 0 "#PWR062" H 8850 4900 50  0001 C CNN
 F 1 "GND" H 8855 4977 50  0000 C CNN
 F 2 "" H 8850 5150 50  0000 C CNN
@@
 $EndComp
 $Comp
-L GND #PWR66
+L GND #PWR066
 U 1 1 59439C71
 P 8500 5750
-F 0 "#PWR66" H 8500 5500 50  0001 C CNN
+F 0 "#PWR066" H 8500 5500 50  0001 C CNN
 F 1 "GND" H 8505 5577 50  0000 C CNN
 F 2 "" H 8500 5750 50  0000 C CNN
@@
 $EndComp
 $Comp
-L GND #PWR61
+L GND #PWR061
 U 1 1 5943AA65
 P 6750 5150
-F 0 "#PWR61" H 6750 4900 50  0001 C CNN
+F 0 "#PWR061" H 6750 4900 50  0001 C CNN
 F 1 "GND" H 6755 4977 50  0000 C CNN
 F 2 "" H 6750 5150 50  0000 C CNN
@@
 $EndComp
 $Comp
-L GND #PWR65
+L GND #PWR065
 U 1 1 5943AA6B
 P 6250 5750
-F 0 "#PWR65" H 6250 5500 50  0001 C CNN
+F 0 "#PWR065" H 6250 5500 50  0001 C CNN
 F 1 "GND" H 6255 5577 50  0000 C CNN
 F 2 "" H 6250 5750 50  0000 C CNN
@@
 $EndComp
 $Comp
-L GND #PWR60
+L GND #PWR060
 U 1 1 5943ABA3
 P 4650 5150
-F 0 "#PWR60" H 4650 4900 50  0001 C CNN
+F 0 "#PWR060" H 4650 4900 50  0001 C CNN
 F 1 "GND" H 4655 4977 50  0000 C CNN
 F 2 "" H 4650 5150 50  0000 C CNN
@@
 $EndComp
 $Comp
-L GND #PWR64
+L GND #PWR064
 U 1 1 5943ABA9
 P 4150 5750
-F 0 "#PWR64" H 4150 5500 50  0001 C CNN
+F 0 "#PWR064" H 4150 5500 50  0001 C CNN
 F 1 "GND" H 4155 5577 50  0000 C CNN
 F 2 "" H 4150 5750 50  0000 C CNN
@@
 $EndComp
 $Comp
-L GND #PWR58
+L GND #PWR058
 U 1 1 5943ACE1
 P 10300 4050
-F 0 "#PWR58" H 10300 3800 50  0001 C CNN
+F 0 "#PWR058" H 10300 3800 50  0001 C CNN
 F 1 "GND" H 10305 3877 50  0000 C CNN
 F 2 "" H 10300 4050 50  0000 C CNN
@@
 $EndComp
 $Comp
-L GND #PWR57
+L GND #PWR057
 U 1 1 5943ACE7
 P 10000 4050
-F 0 "#PWR57" H 10000 3800 50  0001 C CNN
+F 0 "#PWR057" H 10000 3800 50  0001 C CNN
 F 1 "GND" H 10005 3877 50  0000 C CNN
 F 2 "" H 10000 4050 50  0000 C CNN
@@
 $EndComp
 $Comp
-L GND #PWR59
+L GND #PWR059
 U 1 1 5943AFDB
 P 2550 5150
-F 0 "#PWR59" H 2550 4900 50  0001 C CNN
+F 0 "#PWR059" H 2550 4900 50  0001 C CNN
 F 1 "GND" H 2555 4977 50  0000 C CNN
 F 2 "" H 2550 5150 50  0000 C CNN
@@
 $EndComp
 $Comp
-L GND #PWR63
+L GND #PWR063
 U 1 1 5943AFE1
 P 2050 5750
-F 0 "#PWR63" H 2050 5500 50  0001 C CNN
+F 0 "#PWR063" H 2050 5500 50  0001 C CNN
 F 1 "GND" H 2055 5577 50  0000 C CNN
 F 2 "" H 2050 5750 50  0000 C CNN
@@
 $EndComp
 $Comp
-L GND #PWR42
+L GND #PWR042
 U 1 1 5943B229
 P 8850 2350
-F 0 "#PWR42" H 8850 2100 50  0001 C CNN
+F 0 "#PWR042" H 8850 2100 50  0001 C CNN
 F 1 "GND" H 8855 2177 50  0000 C CNN
 F 2 "" H 8850 2350 50  0000 C CNN
@@
 $EndComp
 $Comp
-L GND #PWR50
+L GND #PWR050
 U 1 1 5943B22F
 P 8350 2950
-F 0 "#PWR50" H 8350 2700 50  0001 C CNN
+F 0 "#PWR050" H 8350 2700 50  0001 C CNN
 F 1 "GND" H 8355 2777 50  0000 C CNN
 F 2 "" H 8350 2950 50  0000 C CNN
@@
 $EndComp
 $Comp
-L GND #PWR41
+L GND #PWR041
 U 1 1 5943B345
 P 6750 2350
-F 0 "#PWR41" H 6750 2100 50  0001 C CNN
+F 0 "#PWR041" H 6750 2100 50  0001 C CNN
 F 1 "GND" H 6755 2177 50  0000 C CNN
 F 2 "" H 6750 2350 50  0000 C CNN
@@
 $EndComp
 $Comp
-L GND #PWR49
+L GND #PWR049
 U 1 1 5943B34B
 P 6250 2950
-F 0 "#PWR49" H 6250 2700 50  0001 C CNN
+F 0 "#PWR049" H 6250 2700 50  0001 C CNN
 F 1 "GND" H 6255 2777 50  0000 C CNN
 F 2 "" H 6250 2950 50  0000 C CNN
@@
 $EndComp
 $Comp
-L GND #PWR40
+L GND #PWR040
 U 1 1 5943B4A5
 P 4650 2350
-F 0 "#PWR40" H 4650 2100 50  0001 C CNN
+F 0 "#PWR040" H 4650 2100 50  0001 C CNN
 F 1 "GND" H 4655 2177 50  0000 C CNN
 F 2 "" H 4650 2350 50  0000 C CNN
@@
 $EndComp
 $Comp
-L GND #PWR48
+L GND #PWR048
 U 1 1 5943B4AB
 P 4150 2950
-F 0 "#PWR48" H 4150 2700 50  0001 C CNN
+F 0 "#PWR048" H 4150 2700 50  0001 C CNN
 F 1 "GND" H 4155 2777 50  0000 C CNN
 F 2 "" H 4150 2950 50  0000 C CNN
@@
 $EndComp
 $Comp
-L GND #PWR39
+L GND #PWR039
 U 1 1 5943B803
 P 2550 2350
-F 0 "#PWR39" H 2550 2100 50  0001 C CNN
+F 0 "#PWR039" H 2550 2100 50  0001 C CNN
 F 1 "GND" H 2555 2177 50  0000 C CNN
 F 2 "" H 2550 2350 50  0000 C CNN
@@
 $EndComp
 $Comp
-L GND #PWR47
+L GND #PWR047
 U 1 1 5943B809
 P 2050 2950
-F 0 "#PWR47" H 2050 2700 50  0001 C CNN
+F 0 "#PWR047" H 2050 2700 50  0001 C CNN
 F 1 "GND" H 2055 2777 50  0000 C CNN
 F 2 "" H 2050 2950 50  0000 C CNN
@@
 $EndComp
 $Comp
-L GND #PWR56
+L GND #PWR056
 U 1 1 5943BAD9
 P 9700 4050
-F 0 "#PWR56" H 9700 3800 50  0001 C CNN
+F 0 "#PWR056" H 9700 3800 50  0001 C CNN
 F 1 "GND" H 9705 3877 50  0000 C CNN
 F 2 "" H 9700 4050 50  0000 C CNN
@@
 $EndComp
 $Comp
-L GND #PWR55
+L GND #PWR055
 U 1 1 5943BADF
 P 9400 4050
-F 0 "#PWR55" H 9400 3800 50  0001 C CNN
+F 0 "#PWR055" H 9400 3800 50  0001 C CNN
 F 1 "GND" H 9405 3877 50  0000 C CNN
 F 2 "" H 9400 4050 50  0000 C CNN
@@
 $EndComp
 $Comp
-L GND #PWR46
+L GND #PWR046
 U 1 1 5943BB07
 P 10300 2750
-F 0 "#PWR46" H 10300 2500 50  0001 C CNN
+F 0 "#PWR046" H 10300 2500 50  0001 C CNN
 F 1 "GND" H 10305 2577 50  0000 C CNN
 F 2 "" H 10300 2750 50  0000 C CNN
@@
 $EndComp
 $Comp
-L GND #PWR45
+L GND #PWR045
 U 1 1 5943BB0D
 P 10000 2750
-F 0 "#PWR45" H 10000 2500 50  0001 C CNN
+F 0 "#PWR045" H 10000 2500 50  0001 C CNN
 F 1 "GND" H 10005 2577 50  0000 C CNN
 F 2 "" H 10000 2750 50  0000 C CNN
@@
 $EndComp
 $Comp
-L GND #PWR44
+L GND #PWR044
 U 1 1 5943BB13
 P 9700 2750
-F 0 "#PWR44" H 9700 2500 50  0001 C CNN
+F 0 "#PWR044" H 9700 2500 50  0001 C CNN
 F 1 "GND" H 9705 2577 50  0000 C CNN
 F 2 "" H 9700 2750 50  0000 C CNN
@@
 $EndComp
 $Comp
-L GND #PWR43
+L GND #PWR043
 U 1 1 5943BB19
 P 9400 2750
-F 0 "#PWR43" H 9400 2500 50  0001 C CNN
+F 0 "#PWR043" H 9400 2500 50  0001 C CNN
 F 1 "GND" H 9405 2577 50  0000 C CNN
 F 2 "" H 9400 2750 50  0000 C CNN
@@
 $EndComp
 $Comp
-L GND #PWR51
+L GND #PWR051
 U 1 1 596DACFA
 P 1800 3000
-F 0 "#PWR51" H 1800 2750 50  0001 C CNN
+F 0 "#PWR051" H 1800 2750 50  0001 C CNN
 F 1 "GND" H 1805 2827 50  0000 C CNN
 F 2 "" H 1800 3000 50  0000 C CNN
@@
 $EndComp
 $Comp
-L GND #PWR53
+L GND #PWR053
 U 1 1 596DB008
 P 6000 3000
-F 0 "#PWR53" H 6000 2750 50  0001 C CNN
+F 0 "#PWR053" H 6000 2750 50  0001 C CNN
 F 1 "GND" H 6005 2827 50  0000 C CNN
 F 2 "" H 6000 3000 50  0000 C CNN
@@
 	1650 5500 1800 5500
 $Comp
-L GND #PWR67
+L GND #PWR067
 U 1 1 596DB237
 P 1800 5800
-F 0 "#PWR67" H 1800 5550 50  0001 C CNN
+F 0 "#PWR067" H 1800 5550 50  0001 C CNN
 F 1 "GND" H 1805 5627 50  0000 C CNN
 F 2 "" H 1800 5800 50  0000 C CNN
@@
 	5850 5500 6000 5500
 $Comp
-L GND #PWR69
+L GND #PWR069
 U 1 1 596DB31C
 P 6000 5800
-F 0 "#PWR69" H 6000 5550 50  0001 C CNN
+F 0 "#PWR069" H 6000 5550 50  0001 C CNN
 F 1 "GND" H 6005 5627 50  0000 C CNN
 F 2 "" H 6000 5800 50  0000 C CNN
@@
 	3750 5500 3900 5500
 $Comp
-L GND #PWR68
+L GND #PWR068
 U 1 1 596DB575
 P 3900 5800
-F 0 "#PWR68" H 3900 5550 50  0001 C CNN
+F 0 "#PWR068" H 3900 5550 50  0001 C CNN
 F 1 "GND" H 3905 5627 50  0000 C CNN
 F 2 "" H 3900 5800 50  0000 C CNN
@@
 	7950 5500 8100 5500
 $Comp
-L GND #PWR70
+L GND #PWR070
 U 1 1 596DB780
 P 8100 5800
-F 0 "#PWR70" H 8100 5550 50  0001 C CNN
+F 0 "#PWR070" H 8100 5550 50  0001 C CNN
 F 1 "GND" H 8105 5627 50  0000 C CNN
 F 2 "" H 8100 5800 50  0000 C CNN
@@
 	3750 2700 3900 2700
 $Comp
-L GND #PWR52
+L GND #PWR052
 U 1 1 596DC341
 P 3900 3000
-F 0 "#PWR52" H 3900 2750 50  0001 C CNN
+F 0 "#PWR052" H 3900 2750 50  0001 C CNN
 F 1 "GND" H 3905 2827 50  0000 C CNN
 F 2 "" H 3900 3000 50  0000 C CNN
@@
 	7950 2700 8100 2700
 $Comp
-L GND #PWR54
+L GND #PWR054
 U 1 1 596DC3EA
 P 8100 3000
-F 0 "#PWR54" H 8100 2750 50  0001 C CNN
+F 0 "#PWR054" H 8100 2750 50  0001 C CNN
 F 1 "GND" H 8105 2827 50  0000 C CNN
 F 2 "" H 8100 3000 50  0000 C CNN
@@
 $EndComp
 $Comp
-L GND #PWR71
+L GND #PWR071
 U 1 1 59B021F9
 P 3400 7450
-F 0 "#PWR71" H 3400 7200 50  0001 C CNN
+F 0 "#PWR071" H 3400 7200 50  0001 C CNN
 F 1 "GND" H 3405 7277 50  0000 C CNN
 F 2 "" H 3400 7450 50  0000 C CNN
@@
 	3400 7400 3400 7450
 Text GLabel 1950 7200 0    60   Input ~ 0
-P_LED1642_RST
+D_LED1642_RST
 Wire Wire Line
 	2050 7200 1950 7200

Commit message: Updated to kicad 6.0.0 rc; removed outdated gerber files; Schematic is not complete
Parts:
- C10, C11, C12, C5, C6, C7, C8, C80, C81, C82, C83, C84, C85, C86, C87, C9: symbol C -> device:C
- Q29: symbol Q_PMOS_GSD -> device:Q_PMOS_GSD
- Q30: symbol Q_NPN_BEC -> device:Q_NPN_BEC
- R146, R147, R18, R19, R20, R21, R22, R23, R24, R25: symbol R -> device:R
- U10, U3, U4, U5, U6, U7, U8, U9: symbol LED1642GW -> DeeComponents:LED1642GW
- W10, W12, W13, W14, W15, W16, W17, W18, W19: symbol TEST_1P -> Connector:Test_Point
Connections:
- wire segments 86 -> 97

Commit message: Heavily modifying; Matrix nets under construction
Parts:
- removed C80, C81, C82, C83, C84, C85, C86, C87: 3p, Capacitors_SMD:C_0603_HandSoldering, symbol device:C
- removed Q29: AO3401, TO_SOT_Packages_SMD:SOT-23_Handsoldering, symbol device:Q_PMOS_GSD
- removed Q30: Q_NPN_BEC, TO_SOT_Packages_SMD:SOT-23_Handsoldering, symbol device:Q_NPN_BEC
- removed R146: 10R, Resistors_SMD:R_0603_HandSoldering, symbol device:R
- removed R147: 4.7k, Resistors_SMD:R_0603_HandSoldering, symbol device:R
Connections:
- net labels removed: COLPWCLK0, COLPWCLK1, D_LED1642_RST, LEDLOGICVDD
- wire segments 97 -> 94

Commit message: Almost all components has placed.
Parts:
- removed W10, W12, W13, W14, W15, W16, W17, W18, W19: TEST_1P, Measurement_Points:Measurement_Point_Round-SMD-Pad_Small, symbol Connector:Test_Point
Connections:
- wire segments 94 -> 77
Changed lines of the file:
@@
 EESchema Schematic File Version 4
 LIBS:dotmatrix_64x48-cache
-EELAYER 28 0
+EELAYER 29 0
 EELAYER END
 $Descr A4 11693 8268
@@
 	1350 2350 1350 2450
 Wire Wire Line
-	1250 2350 1250 2450
-Wire Wire Line
 	3350 2600 1750 2600
 Wire Wire Line
-	7550 2350 7550 2450
-Wire Wire Line
 	7550 2600 5950 2600
 Wire Wire Line
 	5950 2600 5950 2350
 Wire Wire Line
-	5450 2350 5450 2450
-Wire Wire Line
 	5450 2600 3850 2600
 Wire Wire Line
 	3850 2600 3850 2350
-Wire Wire Line
-	3350 2350 3350 2450
 Wire Wire Line
 	1750 2600 1750 2350
@@
 	1350 5150 1350 5250
 Wire Wire Line
-	1250 5150 1250 5250
-Wire Wire Line
 	3350 5400 1750 5400
 Wire Wire Line
-	7550 5150 7550 5250
-Wire Wire Line
 	7550 5400 5950 5400
 Wire Wire Line
 	5950 5400 5950 5150
 Wire Wire Line
-	5450 5150 5450 5250
-Wire Wire Line
 	5450 5400 3850 5400
 Wire Wire Line
 	3850 5400 3850 5150
-Wire Wire Line
-	3350 5150 3350 5250
 Wire Wire Line
 	1750 5400 1750 5150
@@
 	1    0    0    -1
 $EndComp
-$Comp
-L Connector:Test_Point W10
-U 1 1 58ABAB2B
-P 1200 2450
-F 0 "W10" V 1250 2500 50  0000 C CNN
-F 1 "TEST_1P" V 1304 2524 50  0001 C CNN
-F 2 "Measurement_Points:Measurement_Point_Round-SMD-Pad_Small" H 1400 2450 50  0001 C CNN
-F 3 "" H 1400 2450 50  0000 C CNN
-	1    1200 2450
-	-1   0    0    1
-$EndComp
-Wire Wire Line
-	1200 2450 1250 2450
-Connection ~ 1250 2450
-$Comp
-L Connector:Test_Point W13
-U 1 1 58ABB0BD
-P 3300 2450
-F 0 "W13" V 3350 2500 50  0000 C CNN
-F 1 "TEST_1P" V 3404 2524 50  0001 C CNN
-F 2 "Measurement_Points:Measurement_Point_Round-SMD-Pad_Small" H 3500 2450 50  0001 C CNN
-F 3 "" H 3500 2450 50  0000 C CNN
-	1    3300 2450
-	-1   0    0    1
-$EndComp
-Wire Wire Line
-	3300 2450 3350 2450
-Connection ~ 3350 2450
-$Comp
-L Connector:Test_Point W15
-U 1 1 58ABB383
-P 5400 2450
-F 0 "W15" V 5450 2500 50  0000 C CNN
-F 1 "TEST_1P" V 5504 2524 50  0001 C CNN
-F 2 "Measurement_Points:Measurement_Point_Round-SMD-Pad_Small" H 5600 2450 50  0001 C CNN
-F 3 "" H 5600 2450 50  0000 C CNN
-	1    5400 2450
-	-1   0    0    1
-$EndComp
-Wire Wire Line
-	5400 2450 5450 2450
-Connection ~ 5450 2450
-$Comp
-L Connector:Test_Point W17
-U 1 1 58ABB414
-P 7500 2450
-F 0 "W17" V 7550 2500 50  0000 C CNN
-F 1 "TEST_1P" V 7604 2524 50  0001 C CNN
-F 2 "Measurement_Points:Measurement_Point_Round-SMD-Pad_Small" H 7700 2450 50  0001 C CNN
-F 3 "" H 7700 2450 50  0000 C CNN
-	1    7500 2450
-	-1   0    0    1
-$EndComp
-Wire Wire Line
-	7500 2450 7550 2450
-Connection ~ 7550 2450
-$Comp
-L Connector:Test_Point W12
-U 1 1 58ABB953
-P 1200 5250
-F 0 "W12" V 1250 5300 50  0000 C CNN
-F 1 "TEST_1P" V 1304 5324 50  0001 C CNN
-F 2 "Measurement_Points:Measurement_Point_Round-SMD-Pad_Small" H 1400 5250 50  0001 C CNN
-F 3 "" H 1400 5250 50  0000 C CNN
-	1    1200 5250
-	-1   0    0    1
-$EndComp
-Wire Wire Line
-	1200 5250 1250 5250
-Connection ~ 1250 5250
-$Comp
-L Connector:Test_Point W14
-U 1 1 58ABB9DC
-P 3300 5250
-F 0 "W14" V 3350 5300 50  0000 C CNN
-F 1 "TEST_1P" V 3404 5324 50  0001 C CNN
-F 2 "Measurement_Points:Measurement_Point_Round-SMD-Pad_Small" H 3500 5250 50  0001 C CNN
-F 3 "" H 3500 5250 50  0000 C CNN
-	1    3300 5250
-	-1   0    0    1
-$EndComp
-Wire Wire Line
-	3300 5250 3350 5250
-Connection ~ 3350 5250
-$Comp
-L Connector:Test_Point W16
-U 1 1 58ABBC10
-P 5400 5250
-F 0 "W16" V 5450 5300 50  0000 C CNN
-F 1 "TEST_1P" V 5504 5324 50  0001 C CNN
-F 2 "Measurement_Points:Measurement_Point_Round-SMD-Pad_Small" H 5600 5250 50  0001 C CNN
-F 3 "" H 5600 5250 50  0000 C CNN
-	1    5400 5250
-	-1   0    0    1
-$EndComp
-Wire Wire Line
-	5400 5250 5450 5250
-Connection ~ 5450 5250
-$Comp
-L Connector:Test_Point W18
-U 1 1 58ABBDEF
-P 7500 5250
-F 0 "W18" V 7500 5500 50  0000 C CNN
-F 1 "TEST_1P" V 7604 5324 50  0001 C CNN
-F 2 "Measurement_Points:Measurement_Point_Round-SMD-Pad_Small" H 7700 5250 50  0001 C CNN
-F 3 "" H 7700 5250 50  0000 C CNN
-	1    7500 5250
-	-1   0    0    1
-$EndComp
-Wire Wire Line
-	7500 5250 7550 5250
-Connection ~ 7550 5250
-$Comp
-L Connector:Test_Point W19
-U 1 1 58ABBF5D
-P 7600 5250
-F 0 "W19" V 7500 5350 50  0000 C CNN
-F 1 "TEST_1P" V 7704 5324 50  0001 C CNN
-F 2 "Measurement_Points:Measurement_Point_Round-SMD-Pad_Small" H 7800 5250 50  0001 C CNN
-F 3 "" H 7800 5250 50  0000 C CNN
-	1    7600 5250
-	-1   0    0    1
-$EndComp
-Wire Wire Line
-	7600 5250 7650 5250
 Connection ~ 7650 5250
 $Comp
@@
 LED1642VDD
 Wire Wire Line
-	1250 2450 1250 2650
-Wire Wire Line
-	3350 2450 3350 2600
-Wire Wire Line
-	5450 2450 5450 2600
-Wire Wire Line
-	7550 2450 7550 2600
-Wire Wire Line
-	1250 5250 1250 6050
-Wire Wire Line
-	3350 5250 3350 5400
-Wire Wire Line
-	5450 5250 5450 5400
-Wire Wire Line
-	7550 5250 7550 5400
-Wire Wire Line
 	7650 5250 7650 5450
 Wire Wire Line
@@
 Wire Wire Line
 	7850 5250 7650 5250
+Wire Wire Line
+	1250 5150 1250 6050
+Wire Wire Line
+	3350 5150 3350 5400
+Wire Wire Line
+	5450 5150 5450 5400
+Wire Wire Line
+	7550 5150 7550 5400
+Wire Wire Line
+	7550 2350 7550 2600
+Wire Wire Line
+	5450 2350 5450 2600
+Wire Wire Line
+	3350 2350 3350 2600
+Wire Wire Line
+	1250 2350 1250 2650
 $EndSCHEMATC
