File: column_driver.sch (KiCad schematic (older format))
At the start: 24 parts, among them U10 LED1642GW, U3 LED1642GW, U4 LED1642GW, U5 LED1642GW, U6 LED1642GW, U7 LED1642GW, U8 LED1642GW, U9 LED1642GW

Commit message: Switched to new kicad libraries
Parts:
- C10, C11, C12, C5, C6, C7, C8, C9: symbol device:C -> dotmatrix_64x48-rescue:C-device
- R18, R19, R20, R21, R22, R23, R24, R25: symbol device:R -> dotmatrix_64x48-rescue:R-device
Changed lines of the file:
@@
 $EndDescr
 $Comp
-L device:R R24
+L dotmatrix_64x48-rescue:R-device R24
 U 1 1 58122B4C
 P 8350 2800
@@
 $EndComp
 $Comp
-L device:R R22
+L dotmatrix_64x48-rescue:R-device R22
 U 1 1 58122B59
 P 6250 2800
@@
 $EndComp
 $Comp
-L device:R R20
+L dotmatrix_64x48-rescue:R-device R20
 U 1 1 58122B66
 P 4150 2800
@@
 $EndComp
 $Comp
-L device:R R18
+L dotmatrix_64x48-rescue:R-device R18
 U 1 1 58122B73
 P 2050 2800
@@
 COLSEROUT
 $Comp
-L device:R R25
+L dotmatrix_64x48-rescue:R-device R25
 U 1 1 5811DEF4
 P 8500 5600
@@
 $EndComp
 $Comp
-L device:R R23
+L dotmatrix_64x48-rescue:R-device R23
 U 1 1 5811DF00
 P 6250 5600
@@
 $EndComp
 $Comp
-L device:R R21
+L dotmatrix_64x48-rescue:R-device R21
 U 1 1 5811DF0C
 P 4150 5600
@@
 $EndComp
 $Comp
-L device:R R19
+L dotmatrix_64x48-rescue:R-device R19
 U 1 1 5811DF18
 P 2050 5600
@@
 ce10
 $Comp
-L device:C C5
+L dotmatrix_64x48-rescue:C-device C5
 U 1 1 581833BD
 P 9400 2600
@@
 LED1642VDD
 $Comp
-L device:C C7
+L dotmatrix_64x48-rescue:C-device C7
 U 1 1 58183AA7
 P 9700 2600
@@
 $EndComp
 $Comp
-L device:C C9
+L dotmatrix_64x48-rescue:C-device C9
 U 1 1 58183AFE
 P 10000 2600
@@
 $EndComp
 $Comp
-L device:C C11
+L dotmatrix_64x48-rescue:C-device C11
 U 1 1 58183B0B
 P 10300 2600
@@
 $EndComp
 $Comp
-L device:C C6
+L dotmatrix_64x48-rescue:C-device C6
 U 1 1 58183BCC
 P 9400 3900
@@
 $EndComp
 $Comp
-L device:C C8
+L dotmatrix_64x48-rescue:C-device C8
 U 1 1 58183BD9
 P 9700 3900
@@
 $EndComp
 $Comp
-L device:C C10
+L dotmatrix_64x48-rescue:C-device C10
 U 1 1 58183BE6
 P 10000 3900
@@
 $EndComp
 $Comp
-L device:C C12
+L dotmatrix_64x48-rescue:C-device C12
 U 1 1 58183BF3
 P 10300 3900
@@
 Connection ~ 7650 5250
 $Comp
-L power:GND #PWR062
+L dotmatrix_64x48-rescue:GND-power #PWR062
 U 1 1 5943C2CA
 P 8850 5150
@@
 $EndComp
 $Comp
-L power:GND #PWR066
+L dotmatrix_64x48-rescue:GND-power #PWR066
 U 1 1 59439C71
 P 8500 5750
@@
 $EndComp
 $Comp
-L power:GND #PWR061
+L dotmatrix_64x48-rescue:GND-power #PWR061
 U 1 1 5943AA65
 P 6750 5150
@@
 $EndComp
 $Comp
-L power:GND #PWR065
+L dotmatrix_64x48-rescue:GND-power #PWR065
 U 1 1 5943AA6B
 P 6250 5750
@@
 $EndComp
 $Comp
-L power:GND #PWR060
+L dotmatrix_64x48-rescue:GND-power #PWR060
 U 1 1 5943ABA3
 P 4650 5150
@@
 $EndComp
 $Comp
-L power:GND #PWR064
+L dotmatrix_64x48-rescue:GND-power #PWR064
 U 1 1 5943ABA9
 P 4150 5750
@@
 $EndComp
 $Comp
-L power:GND #PWR058
+L dotmatrix_64x48-rescue:GND-power #PWR058
 U 1 1 5943ACE1
 P 10300 4050
@@
 $EndComp
 $Comp
-L power:GND #PWR057
+L dotmatrix_64x48-rescue:GND-power #PWR057
 U 1 1 5943ACE7
 P 10000 4050
@@
 $EndComp
 $Comp
-L power:GND #PWR059
+L dotmatrix_64x48-rescue:GND-power #PWR059
 U 1 1 5943AFDB
 P 2550 5150
@@
 $EndComp
 $Comp
-L power:GND #PWR063
+L dotmatrix_64x48-rescue:GND-power #PWR063
 U 1 1 5943AFE1
 P 2050 5750
@@
 $EndComp
 $Comp
-L power:GND #PWR042
+L dotmatrix_64x48-rescue:GND-power #PWR042
 U 1 1 5943B229
 P 8850 2350
@@
 $EndComp
 $Comp
-L power:GND #PWR050
+L dotmatrix_64x48-rescue:GND-power #PWR050
 U 1 1 5943B22F
 P 8350 2950
@@
 $EndComp
 $Comp
-L power:GND #PWR041
+L dotmatrix_64x48-rescue:GND-power #PWR041
 U 1 1 5943B345
 P 6750 2350
@@
 $EndComp
 $Comp
-L power:GND #PWR049
+L dotmatrix_64x48-rescue:GND-power #PWR049
 U 1 1 5943B34B
 P 6250 2950
@@
 $EndComp
 $Comp
-L power:GND #PWR040
+L dotmatrix_64x48-rescue:GND-power #PWR040
 U 1 1 5943B4A5
 P 4650 2350
@@
 $EndComp
 $Comp
-L power:GND #PWR048
+L dotmatrix_64x48-rescue:GND-power #PWR048
 U 1 1 5943B4AB
 P 4150 2950
@@
 $EndComp
 $Comp
-L power:GND #PWR039
+L dotmatrix_64x48-rescue:GND-power #PWR039
 U 1 1 5943B803
 P 2550 2350
@@
 $EndComp
 $Comp
-L power:GND #PWR047
+L dotmatrix_64x48-rescue:GND-power #PWR047
 U 1 1 5943B809
 P 2050 2950
@@
 $EndComp
 $Comp
-L power:GND #PWR056
+L dotmatrix_64x48-rescue:GND-power #PWR056
 U 1 1 5943BAD9
 P 9700 4050
@@
 $EndComp
 $Comp
-L power:GND #PWR055
+L dotmatrix_64x48-rescue:GND-power #PWR055
 U 1 1 5943BADF
 P 9400 4050
@@
 $EndComp
 $Comp
-L power:GND #PWR046
+L dotmatrix_64x48-rescue:GND-power #PWR046
 U 1 1 5943BB07
 P 10300 2750
@@
 $EndComp
 $Comp
-L power:GND #PWR045
+L dotmatrix_64x48-rescue:GND-power #PWR045
 U 1 1 5943BB0D
 P 10000 2750
@@
 $EndComp
 $Comp
-L power:GND #PWR044
+L dotmatrix_64x48-rescue:GND-power #PWR044
 U 1 1 5943BB13
 P 9700 2750
@@
 $EndComp
 $Comp
-L power:GND #PWR043
+L dotmatrix_64x48-rescue:GND-power #PWR043
 U 1 1 5943BB19
 P 9400 2750

Commit message: Changed footprints from old 4.x's R/C to 5.x's
Parts:
- C10, C11, C12, C5, C6, C7, C8, C9: value 1u -> 1u/35V; footprint Capacitors_SMD:C_0603_HandSoldering -> Capacitor_SMD:C_0603_1608Metric_Pad1.05x0.95mm_HandSolder
- R18, R19, R20, R21, R22, R23, R24, R25: footprint Resistors_SMD:R_0603_HandSoldering -> Resistor_SMD:R_0603_1608Metric_Pad1.05x0.95mm_HandSolder
Changed lines of the file:
@@
 F 0 "R24" H 8420 2846 50  0000 L CNN
 F 1 "22k" H 8420 2755 50  0000 L CNN
-F 2 "Resistors_SMD:R_0603_HandSoldering" V 8280 2800 50  0001 C CNN
+F 2 "Resistor_SMD:R_0603_1608Metric_Pad1.05x0.95mm_HandSolder" V 8280 2800 50  0001 C CNN
 F 3 "" H 8350 2800 50  0000 C CNN
 	1    8350 2800
@@
 F 0 "R22" H 6320 2846 50  0000 L CNN
 F 1 "22k" H 6320 2755 50  0000 L CNN
-F 2 "Resistors_SMD:R_0603_HandSoldering" V 6180 2800 50  0001 C CNN
+F 2 "Resistor_SMD:R_0603_1608Metric_Pad1.05x0.95mm_HandSolder" V 6180 2800 50  0001 C CNN
 F 3 "" H 6250 2800 50  0000 C CNN
 	1    6250 2800
@@
 F 0 "R20" H 4220 2846 50  0000 L CNN
 F 1 "22k" H 4220 2755 50  0000 L CNN
-F 2 "Resistors_SMD:R_0603_HandSoldering" V 4080 2800 50  0001 C CNN
+F 2 "Resistor_SMD:R_0603_1608Metric_Pad1.05x0.95mm_HandSolder" V 4080 2800 50  0001 C CNN
 F 3 "" H 4150 2800 50  0000 C CNN
 	1    4150 2800
@@
 F 0 "R18" H 2120 2846 50  0000 L CNN
 F 1 "22k" H 2120 2755 50  0000 L CNN
-F 2 "Resistors_SMD:R_0603_HandSoldering" V 1980 2800 50  0001 C CNN
+F 2 "Resistor_SMD:R_0603_1608Metric_Pad1.05x0.95mm_HandSolder" V 1980 2800 50  0001 C CNN
 F 3 "" H 2050 2800 50  0000 C CNN
 	1    2050 2800
@@
 F 0 "R25" H 8570 5646 50  0000 L CNN
 F 1 "22k" H 8570 5555 50  0000 L CNN
-F 2 "Resistors_SMD:R_0603_HandSoldering" V 8430 5600 50  0001 C CNN
+F 2 "Resistor_SMD:R_0603_1608Metric_Pad1.05x0.95mm_HandSolder" V 8430 5600 50  0001 C CNN
 F 3 "" H 8500 5600 50  0000 C CNN
 	1    8500 5600
@@
 F 0 "R23" H 6320 5646 50  0000 L CNN
 F 1 "22k" H 6320 5555 50  0000 L CNN
-F 2 "Resistors_SMD:R_0603_HandSoldering" V 6180 5600 50  0001 C CNN
+F 2 "Resistor_SMD:R_0603_1608Metric_Pad1.05x0.95mm_HandSolder" V 6180 5600 50  0001 C CNN
 F 3 "" H 6250 5600 50  0000 C CNN
 	1    6250 5600
@@
 F 0 "R21" H 4220 5646 50  0000 L CNN
 F 1 "22k" H 4220 5555 50  0000 L CNN
-F 2 "Resistors_SMD:R_0603_HandSoldering" V 4080 5600 50  0001 C CNN
+F 2 "Resistor_SMD:R_0603_1608Metric_Pad1.05x0.95mm_HandSolder" V 4080 5600 50  0001 C CNN
 F 3 "" H 4150 5600 50  0000 C CNN
 	1    4150 5600
@@
 F 0 "R19" H 2120 5646 50  0000 L CNN
 F 1 "22k" H 2120 5555 50  0000 L CNN
-F 2 "Resistors_SMD:R_0603_HandSoldering" V 1980 5600 50  0001 C CNN
+F 2 "Resistor_SMD:R_0603_1608Metric_Pad1.05x0.95mm_HandSolder" V 1980 5600 50  0001 C CNN
 F 3 "" H 2050 5600 50  0000 C CNN
 	1    2050 5600
@@
 P 9400 2600
 F 0 "C5" H 9515 2646 50  0000 L CNN
-F 1 "1u" H 9515 2555 50  0000 L CNN
-F 2 "Capacitors_SMD:C_0603_HandSoldering" H 9515 2509 50  0001 L CNN
+F 1 "1u/35V" H 9515 2555 50  0000 L CNN
+F 2 "Capacitor_SMD:C_0603_1608Metric_Pad1.05x0.95mm_HandSolder" H 9515 2509 50  0001 L CNN
 F 3 "" H 9400 2600 50  0000 C CNN
 	1    9400 2600
@@
 P 9700 2600
 F 0 "C7" H 9815 2646 50  0000 L CNN
-F 1 "1u" H 9815 2555 50  0000 L CNN
-F 2 "Capacitors_SMD:C_0603_HandSoldering" H 9815 2509 50  0001 L CNN
+F 1 "1u/35V" H 9815 2555 50  0000 L CNN
+F 2 "Capacitor_SMD:C_0603_1608Metric_Pad1.05x0.95mm_HandSolder" H 9815 2509 50  0001 L CNN
 F 3 "" H 9700 2600 50  0000 C CNN
 	1    9700 2600
@@
 P 10000 2600
 F 0 "C9" H 10115 2646 50  0000 L CNN
-F 1 "1u" H 10115 2555 50  0000 L CNN
-F 2 "Capacitors_SMD:C_0603_HandSoldering" H 10115 2509 50  0001 L CNN
+F 1 "1u/35V" H 10115 2555 50  0000 L CNN
+F 2 "Capacitor_SMD:C_0603_1608Metric_Pad1.05x0.95mm_HandSolder" H 10115 2509 50  0001 L CNN
 F 3 "" H 10000 2600 50  0000 C CNN
 	1    10000 2600
@@
 P 10300 2600
 F 0 "C11" H 10415 2646 50  0000 L CNN
-F 1 "1u" H 10415 2555 50  0000 L CNN
-F 2 "Capacitors_SMD:C_0603_HandSoldering" H 10415 2509 50  0001 L CNN
+F 1 "1u/35V" H 10415 2555 50  0000 L CNN
+F 2 "Capacitor_SMD:C_0603_1608Metric_Pad1.05x0.95mm_HandSolder" H 10415 2509 50  0001 L CNN
 F 3 "" H 10300 2600 50  0000 C CNN
 	1    10300 2600
@@
 P 9400 3900
 F 0 "C6" H 9515 3946 50  0000 L CNN
-F 1 "1u" H 9515 3855 50  0000 L CNN
-F 2 "Capacitors_SMD:C_0603_HandSoldering" H 9515 3809 50  0001 L CNN
+F 1 "1u/35V" H 9515 3855 50  0000 L CNN
+F 2 "Capacitor_SMD:C_0603_1608Metric_Pad1.05x0.95mm_HandSolder" H 9515 3809 50  0001 L CNN
 F 3 "" H 9400 3900 50  0000 C CNN
 	1    9400 3900
@@
 P 9700 3900
 F 0 "C8" H 9815 3946 50  0000 L CNN
-F 1 "1u" H 9815 3855 50  0000 L CNN
-F 2 "Capacitors_SMD:C_0603_HandSoldering" H 9815 3809 50  0001 L CNN
+F 1 "1u/35V" H 9815 3855 50  0000 L CNN
+F 2 "Capacitor_SMD:C_0603_1608Metric_Pad1.05x0.95mm_HandSolder" H 9815 3809 50  0001 L CNN
 F 3 "" H 9700 3900 50  0000 C CNN
 	1    9700 3900
@@
 P 10000 3900
 F 0 "C10" H 10115 3946 50  0000 L CNN
-F 1 "1u" H 10115 3855 50  0000 L CNN
-F 2 "Capacitors_SMD:C_0603_HandSoldering" H 10115 3809 50  0001 L CNN
+F 1 "1u/35V" H 10115 3855 50  0000 L CNN
+F 2 "Capacitor_SMD:C_0603_1608Metric_Pad1.05x0.95mm_HandSolder" H 10115 3809 50  0001 L CNN
 F 3 "" H 10000 3900 50  0000 C CNN
 	1    10000 3900
@@
 P 10300 3900
 F 0 "C12" H 10415 3946 50  0000 L CNN
-F 1 "1u" H 10415 3855 50  0000 L CNN
-F 2 "Capacitors_SMD:C_0603_HandSoldering" H 10415 3809 50  0001 L CNN
+F 1 "1u/35V" H 10415 3855 50  0000 L CNN
+F 2 "Capacitor_SMD:C_0603_1608Metric_Pad1.05x0.95mm_HandSolder" H 10415 3809 50  0001 L CNN
 F 3 "" H 10300 3900 50  0000 C CNN
 	1    10300 3900
