File: fet-driver.sch (KiCad schematic (older format))
At the start: 40 parts, among them Q13 AO3401, Q22 AO3401, Q23 AO3401, Q24 AO3401, Q25 AO3401, Q26 AO3401, Q27 AO3401, Q28 AO3401

Commit message: Modified to use matrix LEDs; Components layout has almost done, tracks and traces not yet.
Parts:
- removed R100, R101, R102, R103, R104, R105, R98, R99: 2.2k DNI, Resistors_SMD:R_0603_HandSoldering, symbol R
Connections:
- wire segments 104 -> 88

Commit message: Updated to kicad 6.0.0 rc; removed outdated gerber files; Schematic is not complete
Parts:
- C16, C17, C24, C25, C26, C27, C37, C38: symbol C -> device:C
- Q13, Q22, Q23, Q24, Q25, Q26, Q27, Q28: symbol Q_PMOS_GSD -> device:Q_PMOS_GSD
- R106, R107, R108, R109, R110, R111, R112, R113, R90, R91, R92, R93, R94, R95, R96, R97: symbol R -> device:R
Changed lines of the file:
@@
-EESchema Schematic File Version 3
-LIBS:power
-LIBS:device
-LIBS:linear
-LIBS:regul
-LIBS:adc-dac
-LIBS:dsp
-LIBS:analog_switches
-LIBS:audio
-LIBS:interface
-LIBS:siliconi
-LIBS:opto
-LIBS:contrib
-LIBS:DeeComponents
-LIBS:bb-ch340t
-LIBS:wroom-02
-LIBS:silabs
-LIBS:ac-dc
-LIBS:ir
-LIBS:Zilog
-LIBS:dc-dc
-LIBS:references
-LIBS:sensors
-LIBS:bbd
-LIBS:bosch
-LIBS:zetex
-LIBS:hc11
-LIBS:ESD_Protection
-LIBS:Oscillators
-LIBS:pspice
-LIBS:wiznet
-LIBS:ESP32-footprints-Shem-Lib
-LIBS:Altera
-LIBS:Battery_Management
-LIBS:Connector
-LIBS:DSP_Microchip_DSPIC33
-LIBS:Diode
-LIBS:Display
-LIBS:Espressif
-LIBS:FPGA_Actel
-LIBS:Graphic
-LIBS:LED
-LIBS:LEM
-LIBS:Lattice
-LIBS:Logic_74xgxx
-LIBS:Logic_74xx
-LIBS:Logic_CMOS_4000
-LIBS:Logic_CMOS_IEEE
-LIBS:Logic_TTL_IEEE
-LIBS:MCU_Microchip_PIC10
-LIBS:MCU_Microchip_PIC12
-LIBS:MCU_Microchip_PIC16
-LIBS:MCU_Microchip_PIC18
-LIBS:MCU_Microchip_PIC24
-LIBS:MCU_Microchip_PIC32
-LIBS:MCU_NXP_Kinetis
-LIBS:MCU_NXP_LPC
-LIBS:MCU_NXP_S08
-LIBS:MCU_ST_STM8
-LIBS:MCU_ST_STM32
-LIBS:MCU_Texas_MSP430
-LIBS:Mechanical
-LIBS:Motor
-LIBS:Power_Management
-LIBS:RFSolutions
-LIBS:Relay
-LIBS:Sensor_Current
-LIBS:Switch
-LIBS:Transformer
-LIBS:Transistor
-LIBS:Valve
-LIBS:Worldsemi
-LIBS:Xicor
-LIBS:analog_devices
-LIBS:atmel
-LIBS:brooktre
-LIBS:cypress
-LIBS:digital-audio
-LIBS:driver_gate
-LIBS:elec-unifil
-LIBS:ftdi
-LIBS:gennum
-LIBS:infineon
-LIBS:intel
-LIBS:intersil
-LIBS:logic_programmable
-LIBS:maxim
-LIBS:memory
-LIBS:microchip
-LIBS:microcontrollers
-LIBS:modules
-LIBS:motor_drivers
-LIBS:motorola
-LIBS:nordicsemi
-LIBS:nxp
-LIBS:onsemi
-LIBS:philips
-LIBS:powerint
-LIBS:rfcom
-LIBS:supertex
-LIBS:texas
-LIBS:triac_thyristor
-LIBS:video
-LIBS:xilinx
-LIBS:dotmatrix_64x48-cache
+EESchema Schematic File Version 4
 EELAYER 26 0
 EELAYER END
@@
 	4400 3800 4400 3750
 $Comp
-L Q_PMOS_GSD Q13
+L device:Q_PMOS_GSD Q13
 U 1 1 58170F54
 P 4300 1300
@@
 	4400 5350 4400 5300
 $Comp
-L R R90
+L device:R R90
 U 1 1 581715D9
 P 3450 1300
@@
 $EndComp
 $Comp
-L R R91
+L device:R R91
 U 1 1 581716D7
 P 3450 2050
@@
 $EndComp
 $Comp
-L R R92
+L device:R R92
 U 1 1 58171711
 P 3450 2800
@@
 $EndComp
 $Comp
-L R R93
+L device:R R93
 U 1 1 58171776
 P 3450 3550
@@
 $EndComp
 $Comp
-L R R94
+L device:R R94
 U 1 1 58171B04
 P 3450 4350
@@
 $EndComp
 $Comp
-L R R95
+L device:R R95
 U 1 1 58171B0A
 P 3450 5100
@@
 $EndComp
 $Comp
-L R R96
+L device:R R96
 U 1 1 58171B10
 P 3450 5850
@@
 $EndComp
 $Comp
-L R R97
+L device:R R97
 U 1 1 58171B16
 P 3450 6600
@@
 $EndComp
 $Comp
-L R R110
+L device:R R110
 U 1 1 58171C74
 P 5500 4750
@@
 Connection ~ 4700 4600
 $Comp
-L R R111
+L device:R R111
 U 1 1 58172045
 P 5500 5500
@@
 	5350 5500 4700 5500
 $Comp
-L R R112
+L device:R R112
 U 1 1 581720DE
 P 5500 6250
@@
 	5350 6250 4700 6250
 $Comp
-L R R113
+L device:R R113
 U 1 1 581721A0
 P 5500 7000
@@
 	5350 7000 4700 7000
 $Comp
-L R R106
+L device:R R106
 U 1 1 5817233D
 P 5500 1700
@@
 	5350 1700 4700 1700
 $Comp
-L R R107
+L device:R R107
 U 1 1 58172888
 P 5500 2450
@@
 	5350 2450 4700 2450
 $Comp
-L R R108
+L device:R R108
 U 1 1 5817296B
 P 5500 3200
@@
 	5350 3200 4700 3200
 $Comp
-L R R109
+L device:R R109
 U 1 1 58172A3B
 P 5500 3950
@@
 	5350 3950 4700 3950
 $Comp
-L Q_PMOS_GSD Q22
+L device:Q_PMOS_GSD Q22
 U 1 1 58185931
 P 4300 2050
@@
 $EndComp
 $Comp
-L Q_PMOS_GSD Q23
+L device:Q_PMOS_GSD Q23
 U 1 1 58185A11
 P 4300 2800
@@
 $EndComp
 $Comp
-L Q_PMOS_GSD Q24
+L device:Q_PMOS_GSD Q24
 U 1 1 58185B83
 P 4300 3550
@@
 $EndComp
 $Comp
-L Q_PMOS_GSD Q25
+L device:Q_PMOS_GSD Q25
 U 1 1 58185CB1
 P 4300 4350
@@
 $EndComp
 $Comp
-L Q_PMOS_GSD Q26
+L device:Q_PMOS_GSD Q26
 U 1 1 58185D8F
 P 4300 5100
@@
 $EndComp
 $Comp
-L Q_PMOS_GSD Q27
+L device:Q_PMOS_GSD Q27
 U 1 1 58185F92
 P 4300 5850
@@
 $EndComp
 $Comp
-L Q_PMOS_GSD Q28
+L device:Q_PMOS_GSD Q28
 U 1 1 5818602B
 P 4300 6600
@@
 LEDVDD
 $Comp
-L C C16
+L device:C C16
 U 1 1 58185CB0
 P 5800 1400
@@
 LEDVDD
 $Comp
-L C C17
+L device:C C17
 U 1 1 581864C9
 P 5800 2150
@@
 LEDVDD
 $Comp
-L C C24
+L device:C C24
 U 1 1 58186564
 P 5800 2900
@@
 LEDVDD
 $Comp
-L C C25
+L device:C C25
 U 1 1 581865F8
 P 5800 3650
@@
 LEDVDD
 $Comp
-L C C26
+L device:C C26
 U 1 1 58186806
 P 5800 4450
@@
 LEDVDD
 $Comp
-L C C27
+L device:C C27
 U 1 1 581868F4
 P 5800 5200
@@
 LEDVDD
 $Comp
-L C C37
+L device:C C37
 U 1 1 58186B25
 P 5800 5950
@@
 LEDVDD
 $Comp
-L C C38
+L device:C C38
 U 1 1 58186DEC
 P 5800 6700
@@
 	3000 6600 3300 6600
 $Comp
-L GND #PWR092
+L power:GND #PWR092
 U 1 1 5943CA8A
 P 5800 1700
@@
 $EndComp
 $Comp
-L GND #PWR093
+L power:GND #PWR093
 U 1 1 5943CD8E
 P 5800 2450
@@
 $EndComp
 $Comp
-L GND #PWR094
+L power:GND #PWR094
 U 1 1 5943CDBC
 P 5800 3200
@@
 $EndComp
 $Comp
-L GND #PWR095
+L power:GND #PWR095
 U 1 1 5943CFF2
 P 5800 3950
@@
 $EndComp
 $Comp
-L GND #PWR096
+L power:GND #PWR096
 U 1 1 5943D1B0
 P 5800 4750
@@
 $EndComp
 $Comp
-L GND #PWR097
+L power:GND #PWR097
 U 1 1 5943D1DE
 P 5800 5500
@@
 $EndComp
 $Comp
-L GND #PWR098
+L power:GND #PWR098
 U 1 1 5943D414
 P 5800 6250
@@
 $EndComp
 $Comp
-L GND #PWR099
+L power:GND #PWR099
 U 1 1 5943D442
 P 5800 7000

Commit message: Heavily modifying; Matrix nets under construction
Connections:
- wire segments 88 -> 104
Changed lines of the file:
@@
 EESchema Schematic File Version 4
-EELAYER 26 0
+LIBS:dotmatrix_64x48-cache
+EELAYER 28 0
 EELAYER END
 $Descr A4 11693 8268
@@
 OUT2
 Wire Wire Line
-	4400 3050 4950 3050
+	4400 3050 4700 3050
 Wire Wire Line
 	4400 3050 4400 3000
@@
 OUT3
 Wire Wire Line
-	4400 3800 4950 3800
+	4400 3800 4700 3800
 Wire Wire Line
 	4400 3800 4400 3750
@@
 OUT0
 Wire Wire Line
-	4400 1550 4950 1550
+	4400 1550 4700 1550
 Wire Wire Line
 	4400 1550 4400 1500
@@
 OUT1
 Wire Wire Line
-	4400 2300 4950 2300
+	4400 2300 4700 2300
 Wire Wire Line
 	4400 2300 4400 2250
@@
 OUT6
 Wire Wire Line
-	4400 6100 4950 6100
+	4400 6100 4700 6100
 Wire Wire Line
 	4400 6100 4400 6050
@@
 OUT7
 Wire Wire Line
-	4400 6850 4950 6850
+	4400 6850 4700 6850
 Wire Wire Line
 	4400 6850 4400 6800
@@
 OUT4
 Wire Wire Line
-	4400 4600 4950 4600
+	4400 4600 4700 4600
 Wire Wire Line
 	4400 4600 4400 4550
@@
 OUT5
 Wire Wire Line
-	4400 5350 4950 5350
+	4400 5350 4700 5350
 Wire Wire Line
 	4400 5350 4400 5300
@@
 $EndComp
 Wire Wire Line
-	4400 1050 5900 1050
-Wire Wire Line
-	4400 1800 5900 1800
-Wire Wire Line
-	4400 2550 5900 2550
-Wire Wire Line
-	4400 3300 5900 3300
-Wire Wire Line
-	4400 4100 5900 4100
-Wire Wire Line
-	4400 4850 5900 4850
-Wire Wire Line
-	4400 5600 5900 5600
-Wire Wire Line
-	4400 6350 5900 6350
+	4400 1050 5800 1050
+Wire Wire Line
+	4400 1800 5800 1800
+Wire Wire Line
+	4400 2550 5800 2550
+Wire Wire Line
+	4400 3300 5800 3300
+Wire Wire Line
+	4400 4100 5800 4100
+Wire Wire Line
+	4400 4850 5800 4850
+Wire Wire Line
+	4400 5600 5800 5600
+Wire Wire Line
+	4400 6350 5800 6350
+Wire Wire Line
+	4700 4600 4950 4600
+Wire Wire Line
+	4700 6850 4950 6850
+Wire Wire Line
+	4700 6100 4950 6100
+Wire Wire Line
+	4700 5350 4950 5350
+Wire Wire Line
+	4700 3800 4950 3800
+Wire Wire Line
+	4700 3050 4950 3050
+Wire Wire Line
+	4700 2300 4950 2300
+Wire Wire Line
+	4700 1550 4950 1550
+Wire Wire Line
+	5800 1050 5900 1050
+Wire Wire Line
+	5800 1800 5900 1800
+Wire Wire Line
+	5800 2550 5900 2550
+Wire Wire Line
+	5800 3300 5900 3300
+Wire Wire Line
+	5800 4100 5900 4100
+Wire Wire Line
+	5800 4850 5900 4850
+Wire Wire Line
+	5800 5600 5900 5600
+Wire Wire Line
+	5800 6350 5900 6350
 $EndSCHEMATC
