File: row_driver.sch (KiCad schematic (older format))
At the start: 29 parts, among them SW3 SW_PUSH_SMALL_H, SW4 SW_PUSH_SMALL_H, SW5 SW_PUSH_SMALL_H, SW6 SW_PUSH_SMALL_H, SW7 SW_PUSH_SMALL_H, SW8 SW_PUSH_SMALL_H, U11 74HCT595, U13 74HCT595, U15 74HCT595

Commit message: Modified to use matrix LEDs; Components layout has almost done, tracks and traces not yet.
Parts:
- removed H1, H2: TEST_1P, components:MountingHole_stud-M3, symbol TEST_1P
Connections:
- net labels added: ESPVDD
- net labels removed: LEDLOGICVDD
- wire segments 90 -> 88
Other:
- note added: "3.3V"
Changed lines of the file:
@@
 $Descr A4 11693 8268
 encoding utf-8
-Sheet 5 11
+Sheet 5 10
 Title ""
 Date ""
@@
 Wire Wire Line
 	7050 2950 7050 2800
-Text GLabel 7050 2800 2    60   Input ~ 0
-LEDLOGICVDD
 $Comp
 L C C14
@@
 $EndComp
 $Comp
-L VCC #PWR105
+L VCC #PWR081
 U 1 1 584A8233
 P 6650 4950
-F 0 "#PWR105" H 6650 4800 50  0001 C CNN
+F 0 "#PWR081" H 6650 4800 50  0001 C CNN
 F 1 "VCC" H 6667 5123 50  0000 C CNN
 F 2 "" H 6650 4950 50  0000 C CNN
@@
 $EndComp
 $Comp
-L VCC #PWR107
+L VCC #PWR082
 U 1 1 584A84D9
 P 6950 4950
-F 0 "#PWR107" H 6950 4800 50  0001 C CNN
+F 0 "#PWR082" H 6950 4800 50  0001 C CNN
 F 1 "VCC" H 6967 5123 50  0000 C CNN
 F 2 "" H 6950 4950 50  0000 C CNN
@@
 $EndComp
 $Comp
-L VCC #PWR109
+L VCC #PWR083
 U 1 1 584A84FF
 P 7250 4950
-F 0 "#PWR109" H 7250 4800 50  0001 C CNN
+F 0 "#PWR083" H 7250 4800 50  0001 C CNN
 F 1 "VCC" H 7267 5123 50  0000 C CNN
 F 2 "" H 7250 4950 50  0000 C CNN
@@
 $EndComp
 $Comp
-L VCC #PWR98
+L VCC #PWR085
 U 1 1 584A8637
 P 2800 5250
-F 0 "#PWR98" H 2800 5100 50  0001 C CNN
+F 0 "#PWR085" H 2800 5100 50  0001 C CNN
 F 1 "VCC" H 2817 5423 50  0000 C CNN
 F 2 "" H 2800 5250 50  0000 C CNN
@@
 $EndComp
 $Comp
-L VCC #PWR100
+L VCC #PWR076
 U 1 1 584A865D
 P 3700 4350
-F 0 "#PWR100" H 3700 4200 50  0001 C CNN
+F 0 "#PWR076" H 3700 4200 50  0001 C CNN
 F 1 "VCC" H 3717 4523 50  0000 C CNN
 F 2 "" H 3700 4350 50  0000 C CNN
@@
 $EndComp
 $Comp
-L VCC #PWR96
+L VCC #PWR073
 U 1 1 584A88B2
 P 2350 4350
-F 0 "#PWR96" H 2350 4200 50  0001 C CNN
+F 0 "#PWR073" H 2350 4200 50  0001 C CNN
 F 1 "VCC" H 2367 4523 50  0000 C CNN
 F 2 "" H 2350 4350 50  0000 C CNN
@@
 $EndComp
 $Comp
-L VCC #PWR103
+L VCC #PWR079
 U 1 1 584A8A58
 P 5050 4350
-F 0 "#PWR103" H 5050 4200 50  0001 C CNN
+F 0 "#PWR079" H 5050 4200 50  0001 C CNN
 F 1 "VCC" H 5067 4523 50  0000 C CNN
 F 2 "" H 5050 4350 50  0000 C CNN
@@
 	8950 5150 10650 5150
 $Comp
-L VCC #PWR111
+L VCC #PWR084
 U 1 1 584AB1DF
 P 8400 5150
-F 0 "#PWR111" H 8400 5000 50  0001 C CNN
+F 0 "#PWR084" H 8400 5000 50  0001 C CNN
 F 1 "VCC" H 8417 5323 50  0000 C CNN
 F 2 "" H 8400 5150 50  0000 C CNN
@@
 	1    0    0    -1
 $EndComp
-$Comp
-L GND #PWR112
-U 1 1 58E2244E
-P 8900 6300
-F 0 "#PWR112" H 8900 6050 50  0001 C CNN
-F 1 "GND" H 8905 6127 50  0000 C CNN
-F 2 "" H 8900 6300 50  0000 C CNN
-F 3 "" H 8900 6300 50  0000 C CNN
-	1    8900 6300
-	-1   0    0    -1
-$EndComp
-Wire Wire Line
-	8900 6100 8900 6300
-$Comp
-L TEST_1P H1
-U 1 1 58E2104F
-P 9550 6100
-F 0 "H1" H 9608 6174 50  0000 L CNN
-F 1 "TEST_1P" H 9608 6129 50  0001 L CNN
-F 2 "components:MountingHole_stud-M3" H 9608 6129 50  0001 L CNN
-F 3 "" H 9750 6100 50  0000 C CNN
-	1    9550 6100
-	1    0    0    -1
-$EndComp
-$Comp
-L TEST_1P H2
-U 1 1 58E21056
-P 9800 6100
-F 0 "H2" H 9858 6174 50  0000 L CNN
-F 1 "TEST_1P" H 9858 6129 50  0001 L CNN
-F 2 "components:MountingHole_stud-M3" H 9858 6129 50  0001 L CNN
-F 3 "" H 10000 6100 50  0000 C CNN
-	1    9800 6100
-	1    0    0    -1
-$EndComp
-Connection ~ 9550 6100
 Wire Wire Line
 	4150 4350 4150 4750
@@
 Connection ~ 4150 4750
 Connection ~ 2800 4750
-Wire Wire Line
-	8900 6100 9800 6100
-$Comp
-L GND #PWR106
+$Comp
+L GND #PWR086
 U 1 1 5943AB4A
 P 6650 5250
-F 0 "#PWR106" H 6650 5000 50  0001 C CNN
+F 0 "#PWR086" H 6650 5000 50  0001 C CNN
 F 1 "GND" H 6655 5077 50  0000 C CNN
 F 2 "" H 6650 5250 50  0000 C CNN
@@
 $EndComp
 $Comp
-L GND #PWR108
+L GND #PWR087
 U 1 1 5943AB76
 P 6950 5250
-F 0 "#PWR108" H 6950 5000 50  0001 C CNN
+F 0 "#PWR087" H 6950 5000 50  0001 C CNN
 F 1 "GND" H 6955 5077 50  0000 C CNN
 F 2 "" H 6950 5250 50  0000 C CNN
@@
 $EndComp
 $Comp
-L GND #PWR110
+L GND #PWR088
 U 1 1 5943ABA2
 P 7250 5250
-F 0 "#PWR110" H 7250 5000 50  0001 C CNN
+F 0 "#PWR088" H 7250 5000 50  0001 C CNN
 F 1 "GND" H 7255 5077 50  0000 C CNN
 F 2 "" H 7250 5250 50  0000 C CNN
@@
 $EndComp
 $Comp
-L GND #PWR113
+L GND #PWR089
 U 1 1 5943AE2E
 P 9250 5450
-F 0 "#PWR113" H 9250 5200 50  0001 C CNN
+F 0 "#PWR089" H 9250 5200 50  0001 C CNN
 F 1 "GND" H 9255 5277 50  0000 C CNN
 F 2 "" H 9250 5450 50  0000 C CNN
@@
 $EndComp
 $Comp
-L GND #PWR114
+L GND #PWR090
 U 1 1 5943AE34
 P 9650 5450
-F 0 "#PWR114" H 9650 5200 50  0001 C CNN
+F 0 "#PWR090" H 9650 5200 50  0001 C CNN
 F 1 "GND" H 9655 5277 50  0000 C CNN
 F 2 "" H 9650 5450 50  0000 C CNN
@@
 $EndComp
 $Comp
-L GND #PWR115
+L GND #PWR091
 U 1 1 5943AE3A
 P 10050 5450
-F 0 "#PWR115" H 10050 5200 50  0001 C CNN
+F 0 "#PWR091" H 10050 5200 50  0001 C CNN
 F 1 "GND" H 10055 5277 50  0000 C CNN
 F 2 "" H 10050 5450 50  0000 C CNN
@@
 $EndComp
 $Comp
-L GND #PWR104
+L GND #PWR080
 U 1 1 5943B74E
 P 5200 4350
-F 0 "#PWR104" H 5200 4100 50  0001 C CNN
+F 0 "#PWR080" H 5200 4100 50  0001 C CNN
 F 1 "GND" H 5205 4177 50  0000 C CNN
 F 2 "" H 5200 4350 50  0000 C CNN
@@
 $EndComp
 $Comp
-L GND #PWR102
+L GND #PWR078
 U 1 1 5943B77A
 P 4900 4350
-F 0 "#PWR102" H 4900 4100 50  0001 C CNN
+F 0 "#PWR078" H 4900 4100 50  0001 C CNN
 F 1 "GND" H 4905 4177 50  0000 C CNN
 F 2 "" H 4900 4350 50  0000 C CNN
@@
 $EndComp
 $Comp
-L GND #PWR101
+L GND #PWR077
 U 1 1 5943B994
 P 3850 4350
-F 0 "#PWR101" H 3850 4100 50  0001 C CNN
+F 0 "#PWR077" H 3850 4100 50  0001 C CNN
 F 1 "GND" H 3855 4177 50  0000 C CNN
 F 2 "" H 3850 4350 50  0000 C CNN
@@
 $EndComp
 $Comp
-L GND #PWR99
+L GND #PWR075
 U 1 1 5943B9C0
 P 3550 4350
-F 0 "#PWR99" H 3550 4100 50  0001 C CNN
+F 0 "#PWR075" H 3550 4100 50  0001 C CNN
 F 1 "GND" H 3555 4177 50  0000 C CNN
 F 2 "" H 3550 4350 50  0000 C CNN
@@
 $EndComp
 $Comp
-L GND #PWR97
+L GND #PWR074
 U 1 1 5943B9EC
 P 2500 4350
-F 0 "#PWR97" H 2500 4100 50  0001 C CNN
+F 0 "#PWR074" H 2500 4100 50  0001 C CNN
 F 1 "GND" H 2505 4177 50  0000 C CNN
 F 2 "" H 2500 4350 50  0000 C CNN
@@
 $EndComp
 $Comp
-L GND #PWR95
+L GND #PWR072
 U 1 1 5943BA18
 P 2200 4350
-F 0 "#PWR95" H 2200 4100 50  0001 C CNN
+F 0 "#PWR072" H 2200 4100 50  0001 C CNN
 F 1 "GND" H 2205 4177 50  0000 C CNN
 F 2 "" H 2200 4350 50  0000 C CNN
@@
 	-1   0    0    -1
 $EndComp
+Text Notes 7050 2950 0    60   ~ 0
+3.3V
+Text GLabel 7050 2800 1    60   Input ~ 0
+ESPVDD
 $EndSCHEMATC

Commit message: This is the MazoClock hw 4.0 series; Uses ESP32 processor instead of ESP8266 used in prior MazoClock hw 3.0 series.
Parts:
- added J10, J9: Conn_01x07_Female, Pin_Headers:Pin_Header_Straight_1x07_Pitch2.54mm, symbol Conn_01x07_Female
Connections:
- net labels added: SWPAD_CANCEL, SWPAD_COM, SWPAD_DOWN, SWPAD_LEFT, SWPAD_OK, SWPAD_RIGHT, SWPAD_UP
- wire segments 88 -> 108

Commit message: Added quick-and-dirty class-D amplifier circuit for just testing
Parts:
- added R50: 10k DNI, Resistors_SMD:R_0603_HandSoldering, symbol R
Connections:
- wire segments 108 -> 110
Changed lines of the file:
@@
 LIBS:power
 LIBS:device
-LIBS:transistors
-LIBS:conn
 LIBS:linear
 LIBS:regul
-LIBS:74xx
-LIBS:cmos4000
 LIBS:adc-dac
 LIBS:dsp
@@
 LIBS:audio
 LIBS:interface
-LIBS:display
 LIBS:siliconi
 LIBS:opto
 LIBS:contrib
-LIBS:valves
 LIBS:DeeComponents
 LIBS:bb-ch340t
 LIBS:wroom-02
-LIBS:actel
 LIBS:silabs
 LIBS:ac-dc
 LIBS:ir
-LIBS:74xgxx
 LIBS:Zilog
 LIBS:dc-dc
 LIBS:references
-LIBS:cmos_ieee
 LIBS:sensors
 LIBS:bbd
@@
 LIBS:ESD_Protection
 LIBS:Oscillators
-LIBS:allegro
-LIBS:switches
 LIBS:pspice
-LIBS:transf
-LIBS:relays
-LIBS:ttl_ieee
-LIBS:diode
 LIBS:wiznet
-LIBS:mechanical
-LIBS:microchip_pic32mcu
 LIBS:ESP32-footprints-Shem-Lib
+LIBS:Altera
+LIBS:Battery_Management
+LIBS:Connector
+LIBS:DSP_Microchip_DSPIC33
+LIBS:Diode
+LIBS:Display
+LIBS:Espressif
+LIBS:FPGA_Actel
+LIBS:Graphic
+LIBS:LED
+LIBS:LEM
+LIBS:Lattice
+LIBS:Logic_74xgxx
+LIBS:Logic_74xx
+LIBS:Logic_CMOS_4000
+LIBS:Logic_CMOS_IEEE
+LIBS:Logic_TTL_IEEE
+LIBS:MCU_Microchip_PIC10
+LIBS:MCU_Microchip_PIC12
+LIBS:MCU_Microchip_PIC16
+LIBS:MCU_Microchip_PIC18
+LIBS:MCU_Microchip_PIC24
+LIBS:MCU_Microchip_PIC32
+LIBS:MCU_NXP_Kinetis
+LIBS:MCU_NXP_LPC
+LIBS:MCU_NXP_S08
+LIBS:MCU_ST_STM8
+LIBS:MCU_ST_STM32
+LIBS:MCU_Texas_MSP430
+LIBS:Mechanical
+LIBS:Motor
+LIBS:Power_Management
+LIBS:RFSolutions
+LIBS:Relay
+LIBS:Sensor_Current
+LIBS:Switch
+LIBS:Transformer
+LIBS:Transistor
+LIBS:Valve
+LIBS:Worldsemi
+LIBS:Xicor
+LIBS:analog_devices
+LIBS:atmel
+LIBS:brooktre
+LIBS:cypress
+LIBS:digital-audio
+LIBS:driver_gate
+LIBS:elec-unifil
+LIBS:ftdi
+LIBS:gennum
+LIBS:infineon
+LIBS:intel
+LIBS:intersil
+LIBS:logic_programmable
+LIBS:maxim
+LIBS:memory
+LIBS:microchip
+LIBS:microcontrollers
+LIBS:modules
+LIBS:motor_drivers
+LIBS:motorola
+LIBS:nordicsemi
+LIBS:nxp
+LIBS:onsemi
+LIBS:philips
+LIBS:powerint
+LIBS:rfcom
+LIBS:supertex
+LIBS:texas
+LIBS:triac_thyristor
+LIBS:video
+LIBS:xilinx
 LIBS:dotmatrix_64x48-cache
 EELAYER 26 0
@@
 	8500 750  8500 900
 Wire Wire Line
-	7500 750  8500 750
+	7250 750  8500 750
 Wire Wire Line
 	7850 750  7850 1000
@@
 Wire Wire Line
 	9650 2150 9450 2150
+$Comp
+L R R50
+U 1 1 59E6F4DB
+P 7250 1050
+F 0 "R50" V 7250 1000 50  0000 L CNN
+F 1 "10k DNI" V 7350 850 50  0000 L CNN
+F 2 "Resistors_SMD:R_0603_HandSoldering" V 7180 1050 50  0001 C CNN
+F 3 "" H 7250 1050 50  0000 C CNN
+	1    7250 1050
+	1    0    0    -1
+$EndComp
+$Comp
+L GND #PWR0160
+U 1 1 59E6F925
+P 7250 1450
+F 0 "#PWR0160" H 7250 1200 50  0001 C CNN
+F 1 "GND" H 7255 1277 50  0000 C CNN
+F 2 "" H 7250 1450 50  0000 C CNN
+F 3 "" H 7250 1450 50  0000 C CNN
+	1    7250 1450
+	-1   0    0    -1
+$EndComp
+Wire Wire Line
+	7250 1450 7250 1200
+Wire Wire Line
+	7250 900  7250 750
+Connection ~ 7500 750
 $EndSCHEMATC

Commit message: Updated to kicad 6.0.0 rc; removed outdated gerber files; Schematic is not complete
Parts:
- C13, C14, C15, C65, C67: symbol C -> device:C
- C59: symbol CP -> device:CP
- D1, D2, D3, D4, D5, D6: symbol D_Schottky_Small -> device:D_Schottky_Small
- J10, J9: symbol Conn_01x07_Female -> Connector:Conn_01x07_Female
- L2: symbol INDUCTOR -> pspice:INDUCTOR
- R28, R47, R50: symbol R -> device:R
- SW3, SW4, SW5, SW6, SW7, SW8: symbol SW_Push -> Switch:SW_Push
- U11, U13, U15: symbol 74HC595-alt-vdd -> DeeComponents:74HC595-alt-vdd
- W20, W21, W22: symbol TEST_1P -> Connector:Test_Point
Connections:
- wire segments 110 -> 122

Commit message: Heavily modifying; Matrix nets under construction
Parts:
- removed C59: 3300u 16V LowESR, components:CAP_200_OR_300_P_LAY, symbol device:CP
- removed C65: 1u, Capacitors_SMD:C_0603_HandSoldering, symbol device:C
- removed C67: 0.1u, Capacitors_SMD:C_0603_HandSoldering, symbol device:C
- removed J10, J9: Conn_01x07_Female, Pin_Headers:Pin_Header_Straight_1x07_Pitch2.54mm, symbol Connector:Conn_01x07_Female
- removed L2: 56uH, components:Choke_SMD_12x12mm_10.4x10.4mm_compat_h4.5mm_handsoldering, symbol pspice:INDUCTOR
- removed W20, W21, W22: TEST_1P, Measurement_Points:Measurement_Point_Round-SMD-Pad_Small, symbol Connector:Test_Point
- added U23, U24: CM1293A-04SO, TO_SOT_Packages_SMD:SOT-23-6_Handsoldering, symbol ESD_Protection:SRV05-4
- SW3, SW4, SW5, SW6, SW7, SW8: footprint components:TACT-SW-4P -> components:SW_PUSH_6mm-2pin
- U11, U13, U15: value 74HCT595 -> 74HC595
Connections:
- net labels removed: VCC
- wire segments 122 -> 144

Commit message: Almost all components has placed.
Connections:
- net labels added: LEDLOGICVDD
- net labels removed: ESPVDD
Changed lines of the file:
@@
 EESchema Schematic File Version 4
 LIBS:dotmatrix_64x48-cache
-EELAYER 28 0
+EELAYER 29 0
 EELAYER END
 $Descr A4 11693 8268
@@
 3.3V
 Text GLabel 10500 1000 0    60   Input ~ 0
-ESPVDD
+LEDLOGICVDD
 Text Label 9700 1650 0    60   ~ 0
 SWPAD_COM
@@
 $EndComp
 Text GLabel 8550 2600 0    60   Input ~ 0
-ESPVDD
+LEDLOGICVDD
 Wire Wire Line
 	8550 2600 8650 2600
@@
 $EndComp
 Text GLabel 9800 2600 0    60   Input ~ 0
-ESPVDD
+LEDLOGICVDD
 Wire Wire Line
 	9800 2600 10000 2600
