File: row_driver.sch (KiCad schematic (older format))
At the start: 24 parts, among them SW3 SW_PUSH_SMALL_H, SW4 SW_PUSH_SMALL_H, SW5 SW_PUSH_SMALL_H, SW6 SW_PUSH_SMALL_H, SW7 SW_PUSH_SMALL_H, SW8 SW_PUSH_SMALL_H, U11 74HC595, U13 74HC595, U15 74HC595, U23 CM1293A-04SO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

Commit message: Changed HC595's vdd from LEDVDD to LEDLOGICVDD; Fixed silk refdes'; DRC clean ?(unchecked)
Connections:
- net labels removed: LEDVDD
Changed lines of the file:
@@
 Wire Wire Line
 	7500 1650 9350 1650
-Text GLabel 1450 4950 3    60   Input ~ 0
-LEDVDD
-Text GLabel 2800 4950 3    60   Input ~ 0
-LEDVDD
-Text GLabel 4150 4950 3    60   Input ~ 0
-LEDVDD
 Wire Wire Line
 	4150 4950 4150 4450
@@
 Wire Wire Line
 	1450 4950 1450 4450
-Text GLabel 1900 5350 3    60   Input ~ 0
-LEDVDD
-Text GLabel 6650 4950 1    60   Input ~ 0
-LEDVDD
-Text GLabel 6950 4950 1    60   Input ~ 0
-LEDVDD
-Text GLabel 7250 4950 1    60   Input ~ 0
-LEDVDD
 Wire Wire Line
 	4000 3050 3750 3050
@@
 Text Notes 10250 4300 0    50   ~ 0
 place near TVSs
+Text GLabel 7250 4950 1    60   Input ~ 0
+LEDLOGICVDD
+Text GLabel 6950 4950 1    60   Input ~ 0
+LEDLOGICVDD
+Text GLabel 6650 4950 1    60   Input ~ 0
+LEDLOGICVDD
+Text GLabel 4150 4950 3    60   Input ~ 0
+LEDLOGICVDD
+Text GLabel 2800 4950 3    60   Input ~ 0
+LEDLOGICVDD
+Text GLabel 1450 4950 3    60   Input ~ 0
+LEDLOGICVDD
+Text GLabel 1900 5350 3    60   Input ~ 0
+LEDLOGICVDD
 $EndSCHEMATC

Commit message: Fixed USB micro-b's mount polarity; Improved SOT-23-6 1-pin silk marker readability
Parts:
- U23, U24: footprint TO_SOT_Packages_SMD:SOT-23-6_Handsoldering -> components:SOT-23-6_Handsoldering_mod
Changed lines of the file:
@@
 F 0 "U23" H 8650 3778 50  0000 C CNN
 F 1 "CM1293A-04SO" H 8650 3687 50  0000 C CNN
-F 2 "TO_SOT_Packages_SMD:SOT-23-6_Handsoldering" H 8650 3100 50  0001 C CNN
+F 2 "components:SOT-23-6_Handsoldering_mod" H 8650 3100 50  0001 C CNN
 F 3 "http://www.onsemi.com/pub/Collateral/SRV05-4-D.PDF" H 8650 3100 50  0001 C CNN
 	1    8650 3100
@@
 F 0 "U24" H 10000 3778 50  0000 C CNN
 F 1 "CM1293A-04SO" H 10000 3687 50  0000 C CNN
-F 2 "TO_SOT_Packages_SMD:SOT-23-6_Handsoldering" H 10000 3100 50  0001 C CNN
+F 2 "components:SOT-23-6_Handsoldering_mod" H 10000 3100 50  0001 C CNN
 F 3 "http://www.onsemi.com/pub/Collateral/SRV05-4-D.PDF" H 10000 3100 50  0001 C CNN
 	1    10000 3100

Commit message: LEDVDD now can be up to 5.0V for blue/white LEDs; DRC clear
Parts:
- added R119: 10k, Resistor_SMD:R_0603_1608Metric_Pad1.05x0.95mm_HandSolder, symbol dotmatrix_64x48-rescue:R-device
- added R46: 22k DNI, Resistor_SMD:R_0603_1608Metric_Pad1.05x0.95mm_HandSolder, symbol dotmatrix_64x48-rescue:R-device
- U11, U13, U15: value 74HC595 -> 74HCT595
Connections:
- net labels added: HC595SEROUT_LS, LEDVDD
- wire segments 145 -> 150
Other:
- note added: "3.1V to 5.0V"
- note added: "R46 must be installed when HC595SEROUT does not match to 3.3V levels"
- note added: "for LEDVDD > 4.5V : use 74HCT595; otherwise use 74HC595"
Changed lines of the file:
@@
 P 1750 3750
 F 0 "U11" V 1900 3700 50  0000 L CNN
-F 1 "74HC595" V 1800 3400 50  0000 L CNN
+F 1 "74HCT595" V 1800 3400 50  0000 L CNN
 F 2 "components:SOIC-16-1.27mm" V 1700 3200 50  0000 L CNN
 F 3 "" H 1750 3750 50  0000 C CNN
@@
 P 3100 3750
 F 0 "U13" V 3250 3700 50  0000 L CNN
-F 1 "74HC595" V 3150 3400 50  0000 L CNN
+F 1 "74HCT595" V 3150 3400 50  0000 L CNN
 F 2 "components:SOIC-16-1.27mm" V 3050 3200 50  0000 L CNN
 F 3 "" H 3100 3750 50  0000 C CNN
@@
 P 4450 3750
 F 0 "U15" V 4600 3700 50  0000 L CNN
-F 1 "74HC595" V 4500 3400 50  0000 L CNN
+F 1 "74HCT595" V 4500 3400 50  0000 L CNN
 F 2 "components:SOIC-16-1.27mm" V 4400 3200 50  0000 L CNN
 F 3 "" H 4450 3750 50  0000 C CNN
@@
 place near TVSs
 Text GLabel 7250 4950 1    60   Input ~ 0
-LEDLOGICVDD
+LEDVDD
 Text GLabel 6950 4950 1    60   Input ~ 0
-LEDLOGICVDD
+LEDVDD
 Text GLabel 6650 4950 1    60   Input ~ 0
-LEDLOGICVDD
+LEDVDD
 Text GLabel 4150 4950 3    60   Input ~ 0
-LEDLOGICVDD
+LEDVDD
 Text GLabel 2800 4950 3    60   Input ~ 0
-LEDLOGICVDD
+LEDVDD
 Text GLabel 1450 4950 3    60   Input ~ 0
-LEDLOGICVDD
+LEDVDD
 Text GLabel 1900 5350 3    60   Input ~ 0
-LEDLOGICVDD
+LEDVDD
+$Comp
+L dotmatrix_64x48-rescue:R-device R?
+U 1 1 5BC0278A
+P 9150 5050
+AR Path="/59A8E319/5BC0278A" Ref="R?"  Part="1"
+AR Path="/5BC0278A" Ref="R119"  Part="1"
+AR Path="/58141380/5BC0278A" Ref="R119"  Part="1"
+F 0 "R119" V 9150 4950 50  0000 L CNN
+F 1 "10k" V 9200 4750 50  0000 L CNN
+F 2 "Resistor_SMD:R_0603_1608Metric_Pad1.05x0.95mm_HandSolder" V 9080 5050 50  0001 C CNN
+F 3 "" H 9150 5050 50  0000 C CNN
+	1    9150 5050
+	0    1    -1   0
+$EndComp
+Text GLabel 8850 5050 0    60   Input ~ 0
+HC595SEROUT
+Text GLabel 9600 5050 2    60   Input ~ 0
+HC595SEROUT_LS
+$Comp
+L dotmatrix_64x48-rescue:R-device R?
+U 1 1 5DE6F14B
+P 9500 5350
+AR Path="/59A8E319/5DE6F14B" Ref="R?"  Part="1"
+AR Path="/5DE6F14B" Ref="R?"  Part="1"
+AR Path="/58141380/5DE6F14B" Ref="R46"  Part="1"
+F 0 "R46" V 9500 5250 50  0000 L CNN
+F 1 "22k DNI" V 9600 5050 50  0000 L CNN
+F 2 "Resistor_SMD:R_0603_1608Metric_Pad1.05x0.95mm_HandSolder" V 9430 5350 50  0001 C CNN
+F 3 "" H 9500 5350 50  0000 C CNN
+	1    9500 5350
+	-1   0    0    -1
+$EndComp
+$Comp
+L dotmatrix_64x48-rescue:GND-power #PWR015
+U 1 1 5DE70132
+P 9500 5700
+F 0 "#PWR015" H 9500 5450 50  0001 C CNN
+F 1 "GND" H 9505 5527 50  0000 C CNN
+F 2 "" H 9500 5700 50  0000 C CNN
+F 3 "" H 9500 5700 50  0000 C CNN
+	1    9500 5700
+	-1   0    0    -1
+$EndComp
+Wire Wire Line
+	8850 5050 9000 5050
+Wire Wire Line
+	9300 5050 9500 5050
+Wire Wire Line
+	9500 5200 9500 5050
+Connection ~ 9500 5050
+Wire Wire Line
+	9500 5050 9600 5050
+Wire Wire Line
+	9500 5500 9500 5700
+Text Notes 7400 6200 0    50   ~ 0
+R46 must be installed when HC595SEROUT does not match to 3.3V levels
+Text Notes 8150 5000 0    50   ~ 0
+3.1V to 5.0V
+Text Notes 9850 5000 0    50   ~ 0
+3.3V
+Text Notes 5200 3900 0    50   ~ 0
+for LEDVDD > 4.5V : use 74HCT595; otherwise use 74HC595
 $EndSCHEMATC

Commit message: Wrote note about making LEDVDD > 4.5V
Parts:
- R119: value 10k -> 4.7k
- R46: value 22k DNI -> 10k DNI
Changed lines of the file:
@@
 AR Path="/58141380/5BC0278A" Ref="R119"  Part="1"
 F 0 "R119" V 9150 4950 50  0000 L CNN
-F 1 "10k" V 9200 4750 50  0000 L CNN
+F 1 "4.7k" V 9200 4750 50  0000 L CNN
 F 2 "Resistor_SMD:R_0603_1608Metric_Pad1.05x0.95mm_HandSolder" V 9080 5050 50  0001 C CNN
 F 3 "" H 9150 5050 50  0000 C CNN
@@
 AR Path="/58141380/5DE6F14B" Ref="R46"  Part="1"
 F 0 "R46" V 9500 5250 50  0000 L CNN
-F 1 "22k DNI" V 9600 5050 50  0000 L CNN
+F 1 "10k DNI" V 9600 5050 50  0000 L CNN
 F 2 "Resistor_SMD:R_0603_1608Metric_Pad1.05x0.95mm_HandSolder" V 9430 5350 50  0001 C CNN
 F 3 "" H 9500 5350 50  0000 C CNN
@@
 Wire Wire Line
 	9500 5500 9500 5700
-Text Notes 7400 6200 0    50   ~ 0
+Text Notes 8100 6200 0    50   ~ 0
 R46 must be installed when HC595SEROUT does not match to 3.3V levels
 Text Notes 8150 5000 0    50   ~ 0
