File: ledmatrix.sch (KiCad schematic (older format))
At the start: 1 part

Commit message: Modified to use matrix LEDs; Components layout has almost done, tracks and traces not yet.
Parts:
- removed LED1: LED64x48, components:LED1608_Handsoldering_64x48, symbol LED64x48
- added LED1, LED10, LED11, LED12, LED13, LED14, LED15, LED16, LED17, LED18, LED19, LED2, LED20, LED21, LED22, LED23, LED24, LED25, LED26, LED27, LED28, LED29, LED3, LED30, LED31, LED32, LED33, LED34, LED35, LED36, LED37, LED38, LED39, LED4, LED40, LED41, LED42, LED43, LED44, LED45, LED46, LED47, LED48, LED5, LED6, LED7, LED8, LED9: LED8x8, components:LED8x8,0.8x0.8inch, symbol LED8x8
Connections:
- wire segments 64 -> 0

Commit message: Updated to kicad 6.0.0 rc; removed outdated gerber files; Schematic is not complete
Parts:
- LED1, LED10, LED11, LED12, LED13, LED14, LED15, LED16, LED17, LED18, LED19, LED2, LED20, LED21, LED22, LED23, LED24, LED25, LED26, LED27, LED28, LED29, LED3, LED30, LED31, LED32, LED33, LED34, LED35, LED36, LED37, LED38, LED39, LED4, LED40, LED41, LED42, LED43, LED44, LED45, LED46, LED47, LED48, LED5, LED6, LED7, LED8, LED9: symbol LED8x8 -> DeeComponents:LED8x8
Changed lines of the file:
@@
-EESchema Schematic File Version 3
-LIBS:power
-LIBS:device
-LIBS:linear
-LIBS:regul
-LIBS:adc-dac
-LIBS:dsp
-LIBS:analog_switches
-LIBS:audio
-LIBS:interface
-LIBS:siliconi
-LIBS:opto
-LIBS:contrib
-LIBS:DeeComponents
-LIBS:bb-ch340t
-LIBS:wroom-02
-LIBS:silabs
-LIBS:ac-dc
-LIBS:ir
-LIBS:Zilog
-LIBS:dc-dc
-LIBS:references
-LIBS:sensors
-LIBS:bbd
-LIBS:bosch
-LIBS:zetex
-LIBS:hc11
-LIBS:ESD_Protection
-LIBS:Oscillators
-LIBS:pspice
-LIBS:wiznet
-LIBS:ESP32-footprints-Shem-Lib
-LIBS:Altera
-LIBS:Battery_Management
-LIBS:Connector
-LIBS:DSP_Microchip_DSPIC33
-LIBS:Diode
-LIBS:Display
-LIBS:Espressif
-LIBS:FPGA_Actel
-LIBS:Graphic
-LIBS:LED
-LIBS:LEM
-LIBS:Lattice
-LIBS:Logic_74xgxx
-LIBS:Logic_74xx
-LIBS:Logic_CMOS_4000
-LIBS:Logic_CMOS_IEEE
-LIBS:Logic_TTL_IEEE
-LIBS:MCU_Microchip_PIC10
-LIBS:MCU_Microchip_PIC12
-LIBS:MCU_Microchip_PIC16
-LIBS:MCU_Microchip_PIC18
-LIBS:MCU_Microchip_PIC24
-LIBS:MCU_Microchip_PIC32
-LIBS:MCU_NXP_Kinetis
-LIBS:MCU_NXP_LPC
-LIBS:MCU_NXP_S08
-LIBS:MCU_ST_STM8
-LIBS:MCU_ST_STM32
-LIBS:MCU_Texas_MSP430
-LIBS:Mechanical
-LIBS:Motor
-LIBS:Power_Management
-LIBS:RFSolutions
-LIBS:Relay
-LIBS:Sensor_Current
-LIBS:Switch
-LIBS:Transformer
-LIBS:Transistor
-LIBS:Valve
-LIBS:Worldsemi
-LIBS:Xicor
-LIBS:analog_devices
-LIBS:atmel
-LIBS:brooktre
-LIBS:cypress
-LIBS:digital-audio
-LIBS:driver_gate
-LIBS:elec-unifil
-LIBS:ftdi
-LIBS:gennum
-LIBS:infineon
-LIBS:intel
-LIBS:intersil
-LIBS:logic_programmable
-LIBS:maxim
-LIBS:memory
-LIBS:microchip
-LIBS:microcontrollers
-LIBS:modules
-LIBS:motor_drivers
-LIBS:motorola
-LIBS:nordicsemi
-LIBS:nxp
-LIBS:onsemi
-LIBS:philips
-LIBS:powerint
-LIBS:rfcom
-LIBS:supertex
-LIBS:texas
-LIBS:triac_thyristor
-LIBS:video
-LIBS:xilinx
-LIBS:dotmatrix_64x48-cache
+EESchema Schematic File Version 4
 EELAYER 26 0
 EELAYER END
@@
 r23
 $Comp
-L LED8x8 LED1
+L DeeComponents:LED8x8 LED1
 U 1 1 59A97C81
 P 1000 900
@@
 r7
 $Comp
-L LED8x8 LED9
+L DeeComponents:LED8x8 LED9
 U 1 1 59AAA060
 P 1000 2350
@@
 r7
 $Comp
-L LED8x8 LED2
+L DeeComponents:LED8x8 LED2
 U 1 1 59AAA0CE
 P 2200 900
@@
 r7
 $Comp
-L LED8x8 LED10
+L DeeComponents:LED8x8 LED10
 U 1 1 59AAA0DC
 P 2200 2350
@@
 r7
 $Comp
-L LED8x8 LED3
+L DeeComponents:LED8x8 LED3
 U 1 1 59AAA1BE
 P 3400 900
@@
 r7
 $Comp
-L LED8x8 LED11
+L DeeComponents:LED8x8 LED11
 U 1 1 59AAA1CC
 P 3400 2350
@@
 r7
 $Comp
-L LED8x8 LED4
+L DeeComponents:LED8x8 LED4
 U 1 1 59AAA1DA
 P 4600 900
@@
 r7
 $Comp
-L LED8x8 LED12
+L DeeComponents:LED8x8 LED12
 U 1 1 59AAA1E8
 P 4600 2350
@@
 r7
 $Comp
-L LED8x8 LED5
+L DeeComponents:LED8x8 LED5
 U 1 1 59AAA33E
 P 5800 900
@@
 r7
 $Comp
-L LED8x8 LED13
+L DeeComponents:LED8x8 LED13
 U 1 1 59AAA34C
 P 5800 2350
@@
 r7
 $Comp
-L LED8x8 LED6
+L DeeComponents:LED8x8 LED6
 U 1 1 59AAA35A
 P 7000 900
@@
 r7
 $Comp
-L LED8x8 LED14
+L DeeComponents:LED8x8 LED14
 U 1 1 59AAA368
 P 7000 2350
@@
 r7
 $Comp
-L LED8x8 LED7
+L DeeComponents:LED8x8 LED7
 U 1 1 59AAA396
 P 8200 900
@@
 r7
 $Comp
-L LED8x8 LED15
+L DeeComponents:LED8x8 LED15
 U 1 1 59AAA3A4
 P 8200 2350
@@
 r7
 $Comp
-L LED8x8 LED8
+L DeeComponents:LED8x8 LED8
 U 1 1 59AAA3B2
 P 9400 900
@@
 r7
 $Comp
-L LED8x8 LED16
+L DeeComponents:LED8x8 LED16
 U 1 1 59AAA3C0
 P 9400 2350
@@
 co63
 $Comp
-L LED8x8 LED17
+L DeeComponents:LED8x8 LED17
 U 1 1 59AAA9CE
 P 1000 3800
@@
 $EndComp
 $Comp
-L LED8x8 LED25
+L DeeComponents:LED8x8 LED25
 U 1 1 59AAA9DC
 P 1000 5250
@@
 $EndComp
 $Comp
-L LED8x8 LED18
+L DeeComponents:LED8x8 LED18
 U 1 1 59AAA9EA
 P 2200 3800
@@
 $EndComp
 $Comp
-L LED8x8 LED26
+L DeeComponents:LED8x8 LED26
 U 1 1 59AAA9F8
 P 2200 5250
@@
 $EndComp
 $Comp
-L LED8x8 LED19
+L DeeComponents:LED8x8 LED19
 U 1 1 59AAAA06
 P 3400 3800
@@
 $EndComp
 $Comp
-L LED8x8 LED27
+L DeeComponents:LED8x8 LED27
 U 1 1 59AAAA14
 P 3400 5250
@@
 $EndComp
 $Comp
-L LED8x8 LED20
+L DeeComponents:LED8x8 LED20
 U 1 1 59AAAA22
 P 4600 3800
@@
 $EndComp
 $Comp
-L LED8x8 LED28
+L DeeComponents:LED8x8 LED28
 U 1 1 59AAAA30
 P 4600 5250
@@
 $EndComp
 $Comp
-L LED8x8 LED21
+L DeeComponents:LED8x8 LED21
 U 1 1 59AAAA3E
 P 5800 3800
@@
 $EndComp
 $Comp
-L LED8x8 LED29
+L DeeComponents:LED8x8 LED29
 U 1 1 59AAAA4C
 P 5800 5250
@@
 $EndComp
 $Comp
-L LED8x8 LED22
+L DeeComponents:LED8x8 LED22
 U 1 1 59AAAA5A
 P 7000 3800
@@
 $EndComp
 $Comp
-L LED8x8 LED30
+L DeeComponents:LED8x8 LED30
 U 1 1 59AAAA68
 P 7000 5250
@@
 $EndComp
 $Comp
-L LED8x8 LED23
+L DeeComponents:LED8x8 LED23
 U 1 1 59AAAA76
 P 8200 3800
@@
 $EndComp
 $Comp
-L LED8x8 LED31
+L DeeComponents:LED8x8 LED31
 U 1 1 59AAAA84
 P 8200 5250
@@
 $EndComp
 $Comp
-L LED8x8 LED24
+L DeeComponents:LED8x8 LED24
 U 1 1 59AAAA92
 P 9400 3800
@@
 $EndComp
 $Comp
-L LED8x8 LED32
+L DeeComponents:LED8x8 LED32
 U 1 1 59AAAAA0
 P 9400 5250
@@
 co63
 $Comp
-L LED8x8 LED33
+L DeeComponents:LED8x8 LED33
 U 1 1 59AAB966
 P 1000 6700
@@
 $EndComp
 $Comp
-L LED8x8 LED41
+L DeeComponents:LED8x8 LED41
 U 1 1 59AAB96C
 P 1000 8150
@@
 $EndComp
 $Comp
-L LED8x8 LED34
+L DeeComponents:LED8x8 LED34
 U 1 1 59AAB972
 P 2200 6700
@@
 $EndComp
 $Comp
-L LED8x8 LED42
+L DeeComponents:LED8x8 LED42
 U 1 1 59AAB978
 P 2200 8150
@@
 $EndComp
 $Comp
-L LED8x8 LED35
+L DeeComponents:LED8x8 LED35
 U 1 1 59AAB97E
 P 3400 6700
@@
 $EndComp
 $Comp
-L LED8x8 LED43
+L DeeComponents:LED8x8 LED43
 U 1 1 59AAB984
 P 3400 8150
@@
 $EndComp
 $Comp
-L LED8x8 LED36
+L DeeComponents:LED8x8 LED36
 U 1 1 59AAB98A
 P 4600 6700
@@
 $EndComp
 $Comp
-L LED8x8 LED44
+L DeeComponents:LED8x8 LED44
 U 1 1 59AAB990
 P 4600 8150
@@
 $EndComp
 $Comp
-L LED8x8 LED38
+L DeeComponents:LED8x8 LED38
 U 1 1 59AAB9A2
 P 7000 6700
@@
 $EndComp
 $Comp
-L LED8x8 LED46
+L DeeComponents:LED8x8 LED46
 U 1 1 59AAB9A8
 P 7000 8150
@@
 $EndComp
 $Comp
-L LED8x8 LED39
+L DeeComponents:LED8x8 LED39
 U 1 1 59AAB9AE
 P 8200 6700
@@
 $EndComp
 $Comp
-L LED8x8 LED47
+L DeeComponents:LED8x8 LED47
 U 1 1 59AAB9B4
 P 8200 8150
@@
 $EndComp
 $Comp
-L LED8x8 LED40
+L DeeComponents:LED8x8 LED40
 U 1 1 59AAB9BA
 P 9400 6700
@@
 $EndComp
 $Comp
-L LED8x8 LED48
+L DeeComponents:LED8x8 LED48
 U 1 1 59AAB9C0
 P 9400 8150
@@
 $EndComp
 $Comp
-L LED8x8 LED45
+L DeeComponents:LED8x8 LED45
 U 1 1 59AAB99C
 P 5800 8150
@@
 $EndComp
 $Comp
-L LED8x8 LED37
+L DeeComponents:LED8x8 LED37
 U 1 1 59AAB996
 P 5800 6700
