File: ledmatrix.sch (KiCad schematic (older format))
At the start: 48 parts

Commit message: Prior to merge production-1.0's led matrix pattern
Parts:
- removed LED1, LED10, LED11, LED12, LED13, LED14, LED15, LED16, LED17, LED18, LED19, LED2, LED20, LED21, LED22, LED23, LED24, LED25, LED26, LED27, LED28, LED29, LED3, LED30, LED31, LED32, LED33, LED34, LED35, LED36, LED37, LED38, LED39, LED4, LED40, LED41, LED42, LED43, LED44, LED45, LED46, LED47, LED48, LED5, LED6, LED7, LED8, LED9: LED8x8, components:LED8x8,0.8x0.8inch, symbol DeeComponents:LED8x8
- added LED1: LED64x48, components:LEDMATRIX_64x48-3.0, symbol matrix-dotmatrix_64x48:LED64x48

Commit message: Merged production-1.0's LED matrix onto current design.
Parts:
- LED1: footprint components:LEDMATRIX_64x48-3.0 -> components:LED1608_Handsoldering_64x48
Changed lines of the file:
@@
 F 0 "LED1" H 8828 -96 60  0000 L CNN
 F 1 "LED64x48" H 8828 -203 60  0000 L CNN
-F 2 "components:LEDMATRIX_64x48-3.0" H 1900 1450 60  0001 C CNN
+F 2 "components:LED1608_Handsoldering_64x48" H 1900 1450 60  0001 C CNN
 F 3 "" H 1900 1450 60  0001 C CNN
 	1    1900 1450
