File: dotmatrix_64x48.kicad_pcb (KiCad board)
At the start: 2 copper layers, 207 x 120 mm, 372 parts, among them J7 Conn_01x04_Female, P1 CONN_01X06, P2 CONN_01X06, P3 CONN_01X08, P4 CONN_01X08, Q1 Q_NPN_BCE RN5006, Q10 AO3401, Q11 AO3401, Q12 AO3401, Q13 AO3401, Q14 AO3401, Q15 AO3401, Q16 AO3401, Q17 AO3401, Q18 AO3401, Q19 AO3401, Q2 Q_NPN_BEC, Q20 AO3401, Q21 AO3401, Q22 AO3401, Q23 AO3401, Q24 AO3401, Q25 AO3401, Q26 AO3401, Q27 AO3401, Q28 AO3401, Q29 AO3401, Q3 NJL7302L-F3, Q30 Q_NPN_BEC, Q4 Q_NPN_BEC, Q5 AO3401, Q6 AO3401, Q7 AO3401, Q8 AO3401, Q9 AO3401, SW1 SW_PUSH_SMALL_H, SW2 SW_PUSH_SMALL_H, SW3 SW_PUSH_SMALL_H, SW4 SW_PUSH_SMALL_H, SW5 SW_PUSH_SMALL_H, SW6 SW_PUSH_SMALL_H, SW7 SW_PUSH_SMALL_H, SW8 SW_PUSH_SMALL_H, T1 COMMON_MODE_CHOKE, U1 74VHC541, U10 LED1642GW, U11 74HC595, U12 AE-BME280, U13 74HC595, U14 MAX98357, U15 74HC595, U16 ESP32-WROOM, U17 OSRB38C9AA, U18 BME280, U19 TPS54428DDA, U2 TPS54202, U20 CP2102N-A01-GQFN28, U21 CM1293A-04SO, U22 CM1293A-04SO, U23 CM1293A-04SO, U24 CM1293A-04SO, U25 CM1293A-04SO, U3 LED1642GW, U4 LED1642GW, U5 LED1642GW, U6 LED1642GW, U7 LED1642GW, U8 LED1642GW, U9 LED1642GW

Commit message: Getting very mojai
Parts:
- moved R65 150.1 mm to (121.8, 63.4), turned to 90 degrees
- moved C38 148.7 mm to (121.7, 67.5), turned to 90 degrees
- moved Q12 146.4 mm to (119.4, 66.1), turned to 90 degrees
- moved R37 139.5 mm to (119.7, 70.0)
- moved R63 128.1 mm to (138.3, 63.0), turned to 90 degrees
- moved R64 127.1 mm to (165.2, 62.1), turned to 90 degrees
- moved C27 126.9 mm to (139.0, 66.8), turned to 90 degrees
- moved C37 124.9 mm to (165.4, 65.9), turned to 90 degrees
- moved R61 124.5 mm to (128.3, 62.6), turned to 90 degrees
- moved C25 123.8 mm to (128.3, 66.5), turned to 90 degrees
- moved Q10 123.7 mm to (136.7, 66.5), turned to 90 degrees
- moved Q11 123.1 mm to (162.8, 65.0), turned to 90 degrees
- moved Q8 120.7 mm to (125.8, 64.7), turned to 90 degrees
- moved R62 119.4 mm to (151.9, 61.2), turned to 90 degrees
- moved R35 117.8 mm to (137.1, 69.9)
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Routing:
- net GND: track 829.2 -> 1334.7 mm, vias 38 -> 75
- net LEDVDD: track 531.7 -> 635.3 mm, vias 20 -> 28
- net r2: track 317.5 -> 370.1 mm, vias 8 -> 11
- net r6: track 336.3 -> 380.4 mm, vias 6 -> 9
- net r1: track 354.3 -> 397.1 mm, vias 13 -> 14
- net r15: track 357.0 -> 389.9 mm, vias 15 -> 21
- net r7: track 330.9 -> 361.9 mm, vias 8 -> 11
- net r5: track 336.4 -> 363.9 mm, vias 9 -> 12
- net r4: track 331.7 -> 351.7 mm, vias 5 -> 8
- net r3: track 344.3 -> 359.5 mm, vias 11 -> 12
- net co18: track 94.7 -> 104.9 mm, vias 3 -> 8
- net r12: track 354.1 -> 361.9 mm, vias 5 -> 7
- net r22: track 341.7 -> 349.4 mm, vias 7 -> 8
- net r14: track 363.2 -> 369.7 mm, vias 19 -> 18
- net ce52: track 110.5 -> 116.9 mm, vias 8 -> 10
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
Commit message: Almost all components has placed.
Parts:
- removed C36: 1u, Capacitors_SMD:C_0603_HandSoldering
- removed C63: 0.1u, Capacitors_SMD:C_0603_HandSoldering
- removed P3, P4: CONN_01X08, Pin_Headers:Pin_Header_Straight_1x08_Pitch2.54mm
- removed R1: 1k, Resistors_SMD:R_0603_HandSoldering
- removed U18: BME280, components:BME280-handsoldering
- removed W1, W10, W12, W13, W14, W15, W16, W17, W18, W19, W2, W3, W4, W7: TEST_1P, Measurement_Points:Measurement_Point_Round-SMD-Pad_Small
- added J1: Conn_02x04_Odd_Even, Pin_Headers:Pin_Header_Angled_2x04_Pitch2.54mm, F.Cu at (107.0, 22.2)
- added J2: Conn_02x04_Odd_Even, Pin_Headers:Pin_Header_Angled_2x04_Pitch2.54mm, F.Cu at (114.6, 123.0)
- added REF**: SPK_DAEX25FHE-4_adhesive_circle, components:SPK_DAEX25FHE-4_adhesive_circle, F.Cu at (185.7, 75.9)
- C2, C21, C22, C23, C3, C4, C62, C64, C65, C66, C72, D12, D14, D7, F1, L3, L6, LED49, LED50, LED51, Q1, Q3, R100, R11, R118, R119, R12, R120, R121, R125, R126, R127, R128, R13, R130, R131, R132, R14, R15, R2, R27, R34, R4, R41, R42, R46, R49, R5, R51, R54, R55, R57, R6, R7, R74, R75, R76, R8, U1, U12, U16: moved to B.Cu
- C28, C33: value 10u -> 10u 16V
- C75, C76: value 1u -> 1u 16V
- L1: value 2.2uH -> 10uH; footprint components:Choke_SMD_12x12mm_10.4x10.4mm_compat_h4.5mm_handsoldering -> components:Choke_SMD_7.3x7.3_H3.5_handsoldering
- L2: footprint components:Choke_SMD_12x12mm_10.4x10.4mm_compat_h4.5mm_handsoldering -> components:Choke_SMD_7.3x7.3_H3.5_handsoldering
- LS1: footprint components:SPK_35mm_20mm_RECTANGLE_MOUNT -> Wire_Connections_Bridges:WireConnection_1.50mmDrill
- R80, R81: moved to F.Cu
- moved U25 694.8 mm to (86.2, 46.5)
- moved R34 659.0 mm to (103.2, 18.6), turned to 90 degrees
- moved R118 656.7 mm to (104.5, 20.8), turned to 90 degrees
- moved R127 650.6 mm to (107.2, 17.2)
- moved R121 649.6 mm to (106.8, 28.1), turned to 270 degrees
- moved R119 649.6 mm to (103.0, 28.1), turned to 90 degrees
- moved R120 647.9 mm to (104.2, 28.1), turned to 90 degrees
- moved R128 647.6 mm to (98.0, 53.4), turned to 90 degrees
- moved R132 647.4 mm to (108.8, 53.4), turned to 90 degrees
- moved R130 644.4 mm to (105.8, 53.4), turned to 90 degrees
- moved U22 644.1 mm to (94.7, 104.9), turned to 90 degrees
- moved R126 642.5 mm to (111.1, 17.2)
- moved R122 640.6 mm to (117.1, 21.0), turned to 90 degrees
- moved U21 640.1 mm to (103.0, 132.0), turned to 90 degrees
- moved R125 639.4 mm to (114.9, 17.2), turned to 180 degrees
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Connections:
- net DC_IN renamed DC_IN_P
- net Net-(C72-Pad2) renamed /power/DC_IN_N
- net Net-(CONN3-Pad2) renamed /IR_Sensor/IRLED_K
- net Net-(LS1-Pad1) renamed /IR_Sensor/SPK_P
- net Net-(LS1-Pad2) renamed /IR_Sensor/SPK_N
- C1 pad 1: Net-(C1-Pad1) -> /IR_Sensor/FILT_VDD
- C32 pad 1: Net-(C1-Pad1) -> /IR_Sensor/FILT_VDD
- C4 pad 1: VCC -> LEDVDD
- C67 pad 1: GND -> /USB_UART/USB3V3
- C70 pad 1: GND -> /USB_UART/USB3V3
- C73 pad 1: GND -> /USB_UART/USB3V3
- J7 pad 4: ESPVDD -> LEDLOGICVDD
- L6 pad 1: VCC -> LEDVDD
- P2 pad 1: GND -> /USB_UART/USB3V3
- R10 pad 2: ESPVDD -> LEDLOGICVDD
- R117 pad 2: GND -> /USB_UART/USB3V3
- R123 pad 1: Net-(C1-Pad1) -> /IR_Sensor/FILT_VDD
- R124 pad 1: Net-(C1-Pad1) -> /IR_Sensor/FILT_VDD
- R16 pad 2: VCC -> LEDVDD
- R17 pad 2: VCC -> LEDVDD
- R26 pad 2: VCC -> LEDVDD
- R28 pad 1: ESPVDD -> LEDLOGICVDD
- R45 pad 2: ESPVDD -> /IR_Sensor/FILT_VDD
- R9 pad 2: ESPVDD -> LEDLOGICVDD
- U12 pad 1: ESPVDD -> LEDLOGICVDD
- U17 pad 3: Net-(C1-Pad1) -> /IR_Sensor/FILT_VDD
- U20 pad 6: GND -> /USB_UART/USB3V3
- U21 pad 5: ESPVDD -> LEDLOGICVDD
- U22 pad 5: ESPVDD -> LEDLOGICVDD
- U23 pad 5: ESPVDD -> LEDLOGICVDD
- U24 pad 5: ESPVDD -> LEDLOGICVDD
Routing:
- net GND: track 1334.7 -> 2184.6 mm, vias 75 -> 117
- net /IR_Sensor/IRLED_K: track 0.00 -> 286.9 mm, vias 0 -> 2
- net /CC_GUARD1: track 0.00 -> 272.0 mm, vias 0 -> 8
- net /CC_GUARD0: track 2.03 -> 272.9 mm, vias 0 -> 8
- net Net-(R121-Pad2): track 239.7 -> 0.00 mm, vias 6 -> 0
- net Net-(R119-Pad1): track 237.7 -> 0.00 mm, vias 6 -> 0
- net IR_IN: track 0.00 -> 234.7 mm, vias 0 -> 12
- net /IR_Sensor/FILT_VDD: track 0.00 -> 217.1 mm, vias 0 -> 8
- net E_AIN: track 0.00 -> 213.7 mm, vias 0 -> 11
- net HC595SEROUT: track 0.00 -> 198.7 mm, vias 0 -> 15
- net LEDVDD: track 635.3 -> 797.9 mm, vias 28 -> 36
- net /row_driver/SEL1: track 0.00 -> 160.1 mm, vias 0 -> 6
- net /row_driver/SEL6: track 0.00 -> 146.5 mm, vias 0 -> 8
- net COLSEROUT: track 0.00 -> 142.6 mm, vias 0 -> 4
- net /row_driver/SEL2: track 0.00 -> 132.7 mm, vias 0 -> 6
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- added copper zone on B.Cu, net GND
- added copper zone on B.Cu, net Net-(C72-Pad1)
- added copper zone on F.Cu, net Net-(C72-Pad1)
Other:
- rule pad_to_mask_clearance: 0.2 -> 0.14
- board text removed: "A(5V)"
- board text removed: "DC5V"
- board text removed: "IR RECV"
- board text removed: "K(OC)"
- board text removed: "Ver 4.0 Proto 1"
- board text removed: "WiFi NTP dot-matrix clock"
- board text removed: "https://github.com/w-dee/dotmatrix_64x48"

Commit message: Too less PCB space.
Parts:
- removed CONN3: Push_Terminal_3P_2.54, components:Push_Terminal_3P_2.54
- removed D12: PESD12VL2BT, TO_SOT_Packages_SMD:SOT-23_Handsoldering
- removed LED50, LED51: IR, LEDs:LED_D5.0mm
- added C36: 1u, Capacitors_SMD:C_0603_HandSoldering, F.Cu at (112.0, 87.8)
- added C63: 0.1u 16V, Capacitors_SMD:C_0603_HandSoldering, F.Cu at (113.7, 78.1)
- added C78: 0.1u 16V, Capacitors_SMD:C_0603_HandSoldering, F.Cu at (113.6, 85.5)
- added C79: 1u 16V, Capacitors_SMD:C_0603_HandSoldering, F.Cu at (113.5, 86.7)
- added C80: 1u 16V, Capacitors_SMD:C_0603_HandSoldering, F.Cu at (113.7, 76.8)
- added C81: 10u 16V, Capacitors_SMD:C_1206_HandSoldering, B.Cu at (115.1, 90.5)
- added C82: 10u 16V, Capacitors_SMD:C_1206_HandSoldering, F.Cu at (113.5, 72.5)
- added C83: 0.1u 16V, Capacitors_SMD:C_0603_HandSoldering, F.Cu at (118.1, 85.0)
- added C84: 0.1u 16V, Capacitors_SMD:C_0603_HandSoldering, F.Cu at (118.1, 83.9)
- added C85: 0.1u 16V, Capacitors_SMD:C_0603_HandSoldering, F.Cu at (118.1, 88.0)
- added C86: 0.1u 16V, Capacitors_SMD:C_0603_HandSoldering, F.Cu at (118.1, 86.8)
- added C87: 1u, Capacitors_SMD:C_0603_HandSoldering, F.Cu at (61.9, 87.5)
- added CONN4: Pin_Header_Straight_1x05_Pitch2.54mm, Pin_Headers:Pin_Header_Straight_1x05_Pitch2.54mm, F.Cu at (112.5, 107.2)
- added D8: Led_Small, components:LED1608_Handsoldering, B.Cu at (100.5, 30.0)
- added J3: Micro_SD_Card, components:microSD_Push_Push_SMD, F.Cu at (93.6, 80.2)
- added J4: Conn_01x02, Wire_Connections_Bridges:WireConnection_1.50mmDrill, F.Cu at (112.0, 149.4)
- added L5: BLM21PG331SN 300R@100MHz, Capacitors_SMD:C_0805_HandSoldering, F.Cu at (67.7, 68.3)
- added Q31: Q_NPN_BEC, TO_SOT_Packages_SMD:SOT-23_Handsoldering, B.Cu at (303.4, 95.1)
- added R1: 4.7k, Resistors_SMD:R_0603_HandSoldering, B.Cu at (304.9, 92.3)
- added R137: 120R, Resistors_SMD:R_0603_HandSoldering, F.Cu at (107.0, 53.8)
- added R138: 4.7k, Resistors_SMD:R_0603_HandSoldering, F.Cu at (111.8, 28.4)
- added R139: 10R, Resistors_SMD:R_0603_HandSoldering, F.Cu at (294.9, 54.3)
- added R140: 10R, Resistors_SMD:R_0603_HandSoldering, F.Cu at (294.9, 56.8)
- added U18: CM1293A-04SO, TO_SOT_Packages_SMD:SOT-23-6_Handsoldering, F.Cu at (104.0, 21.0)
- added U26: CM1293A-04SO, TO_SOT_Packages_SMD:SOT-23-6_Handsoldering, B.Cu at (115.4, 108.8)
- added U27: CM1293A-04SO, TO_SOT_Packages_SMD:SOT-23-6_Handsoldering, F.Cu at (36.8, 86.3)
- C18: value 0.1u -> 1u
- C19, C34, C67, C70, C73, R3, R40, R53, U20, U21: moved to B.Cu
- C2: value 0.1u -> 10u; footprint Capacitors_SMD:C_0603_HandSoldering -> Capacitors_SMD:C_1206_HandSoldering
- C20: value 10u -> 1u; footprint Capacitors_SMD:C_1206_HandSoldering -> Capacitors_SMD:C_0603_HandSoldering; moved to B.Cu
- C62, C65, CONN2, R119, R120, R126, R128, R13, R131, R132, R2, R27, R41, R49, R51, R54, R55, R57, R74, R75, R76, R8, U16: moved to F.Cu
- J1: value Conn_02x04_Odd_Even -> Conn_01x03_Female; footprint Pin_Headers:Pin_Header_Angled_2x04_Pitch2.54mm -> Pin_Headers:Pin_Header_Angled_1x03_Pitch2.54mm
- J2: value Conn_02x04_Odd_Even -> Conn_01x03_Male; footprint Pin_Headers:Pin_Header_Angled_2x04_Pitch2.54mm -> Pin_Headers:Pin_Header_Angled_1x03_Pitch2.54mm
- LED49: footprint LEDs:LED_D5.0mm -> LEDs:LED_PLCC_2835_Handsoldering
- P1, P2: footprint Pin_Headers:Pin_Header_Straight_1x08_Pitch2.54mm -> Pin_Headers:Pin_Header_Straight_1x06_Pitch2.54mm
- Q1: value Q_NPN_BCE RN5006 -> AO3401; footprint TO_SOT_Packages_SMD:SOT-89-3_Handsoldering -> TO_SOT_Packages_SMD:SOT-23_Handsoldering
- R100: value 0 -> 10k; moved to F.Cu
- R12: value 1k -> 10k
- R125, R127: value 10k -> 120R; moved to F.Cu
- R130: value 120R -> 10k; moved to F.Cu
- R133, R134, R135, R136, R77, R78: footprint components:SolderJumper -> components:SolderJumper_S
- R42: value 10k DNI -> 10k
- R46: value 120R -> 0; footprint Resistors_SMD:R_0603_HandSoldering -> components:SolderJumper_S; moved to F.Cu
- R80, R81: footprint components:SolderJumper -> components:SolderJumper_S; moved to B.Cu
- R99: value 100k -> 10k
- U14: value MAX98357 -> TAS5720; footprint components:QFN-16-1EP_3x3mm_Pitch0.5mm-handsoldering -> components:QFN-32-1EP_4x4mm_Pitch0.4mm_Handsoldering
- moved L6 225.9 mm to (316.8, 93.2)
- moved R42 225.9 mm to (306.3, 98.3), turned to 180 degrees
- moved C3 225.5 mm to (305.6, 86.2), turned to 270 degrees
- moved Q1 225.0 mm to (308.8, 96.8), turned to 180 degrees
- moved C4 223.2 mm to (314.1, 89.9)
- moved D14 223.1 mm to (302.6, 86.0)
- moved R12 222.0 mm to (302.6, 89.5), turned to 270 degrees
- moved R125 94.3 mm to (52.1, 87.5), turned to 0 degrees
- moved R48 90.7 mm to (42.2, 85.3), turned to 0 degrees
- moved R56 83.7 mm to (47.1, 87.5), turned to 0 degrees
- moved R100 73.1 mm to (42.2, 87.7)
- moved R46 69.7 mm to (66.9, 81.3), turned to 0 degrees
- moved R126 69.3 mm to (67.4, 71.0)
- moved R127 68.9 mm to (67.4, 73.4)
- moved R131 60.7 mm to (57.1, 87.5), turned to 0 degrees
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Connections:
- net Net-(C22-Pad1) renamed /HC541VDD
- net Net-(C69-Pad1) renamed /USB_UART/VBUS
- C18 pad 1: LEDLOGICVDD -> Net-(C18-Pad1)
- C18 pad 2: GND -> Net-(C18-Pad2)
- C19 pad 1: LEDLOGICVDD -> Net-(C18-Pad1)
- C19 pad 2: GND -> Net-(C19-Pad2)
- C2 pad 1: Net-(C2-Pad1) -> ESPVDD
- C2 pad 2: IR_OUT -> GND
- C20 pad 1: LEDLOGICVDD -> GND
- C20 pad 2: GND -> Net-(C20-Pad2)
- C3 pad 1: Net-(C3-Pad1) -> IR_OUT
- C3 pad 2: Net-(C2-Pad1) -> Net-(C3-Pad2)
- C4 pad 1: LEDVDD -> Net-(C4-Pad1)
- C68 pad 1: ESPVDD -> LEDLOGICVDD
- J1 pad 2: GND -> E_TX2
- J1 pad 3: VSPI_SCK -> E_RX2
- J2 pad 1: VSPI_MOSI -> E_TX2
- J2 pad 2: VSPI_MISO -> E_RX2
- L6 pad 2: Net-(CONN3-Pad3) -> Net-(C4-Pad1)
- LED49 pad 1: /IR_Sensor/IRLED_K -> GND
- P2 pad 3: Net-(P2-Pad3) -> E_RX
- P2 pad 4: Net-(P2-Pad4) -> E_TX
- P2 pad 5: Net-(P2-Pad5) -> DTR
- P2 pad 6: Net-(P2-Pad6) -> RTS
- Q1 pad 1: Net-(C3-Pad1) -> Net-(Q1-Pad1)
- Q1 pad 2: /IR_Sensor/IRLED_K -> Net-(C4-Pad1)
- Q1 pad 3: GND -> IRLED_A
- R100 pad 1: Net-(R100-Pad1) -> Net-(J3-Pad8)
- R12 pad 1: Net-(C2-Pad1) -> IR_OUT
- R12 pad 2: Net-(C3-Pad1) -> Net-(C3-Pad2)
- R122 pad 1: VSPI_MISO -> E_RX2
- R122 pad 2: ESPVDD -> LEDLOGICVDD
- R123 pad 2: ESPVDD -> LEDLOGICVDD
- R124 pad 2: ESPVDD -> LEDLOGICVDD
- R125 pad 1: VSPI_MOSI -> E_HS2_CMD
- R125 pad 2: ESPVDD -> Net-(R125-Pad2)
- R126 pad 1: VSPI_SS -> Net-(J3-Pad2)
- R126 pad 2: ESPVDD -> LEDLOGICVDD
- R127 pad 1: VSPI_SCK -> E_HS2_DATA0
- R127 pad 2: ESPVDD -> Net-(R127-Pad2)
- R130 pad 1: VSPI_MISO -> Net-(J3-Pad1)
- R130 pad 2: Net-(R130-Pad2) -> LEDLOGICVDD
- R131 pad 1: VSPI_SCK -> Net-(R131-Pad1)
- R131 pad 2: Net-(R131-Pad2) -> D_COLCLK
- R132 pad 1: VSPI_SS -> Net-(R132-Pad1)
- R132 pad 2: Net-(R132-Pad2) -> D_COLSER
- R16 pad 2: LEDVDD -> IRLED_A
- R17 pad 1: Net-(LED50-Pad2) -> Net-(Q1-Pad1)
- R17 pad 2: LEDVDD -> Net-(Q31-Pad3)
- R26 pad 1: Net-(LED51-Pad2) -> Net-(LED49-Pad2)
- R26 pad 2: LEDVDD -> IRLED_A
- R3 pad 2: ESPVDD -> LEDLOGICVDD
- R34 pad 2: ESPVDD -> LEDLOGICVDD
- R40 pad 1: ESPVDD -> LEDLOGICVDD
- R42 pad 1: GND -> IRLED_A
- R42 pad 2: Net-(C3-Pad1) -> GND
- R46 pad 1: Net-(R46-Pad1) -> MS_SEL
- R46 pad 2: I2S_SPK_GAIN1 -> GND
- R48 pad 2: I2S_SPK_GAIN0 -> E_HS2_CLK
- R52 pad 1: D_LED1642_RST -> D_COLLATCH
- R53 pad 2: D_COLCLK -> E_TX2
- R54 pad 2: D_COLSER -> E_RX2
- R56 pad 1: D_COLLATCH -> D_LED1642_RST
- R99 pad 1: I2S_SPK_GAIN1 -> Net-(R99-Pad1)
- R99 pad 2: I2S_SPK_GAIN0 -> LEDLOGICVDD
- U14 pad 1: I2S_SPK_DATA -> Net-(C18-Pad1)
- U14 pad 10: /IR_Sensor/SPK_N -> GND
- U14 pad 11: GND -> LEDLOGICVDD
- U14 pad 12: (no net) -> GND
- U14 pad 13: (no net) -> GND
- U14 pad 14: I2S_SPK_LRCLK -> VCC
- U14 pad 15: GND -> VCC
- U14 pad 16: I2S_SPK_BCLK -> /IR_Sensor/SPK_N
- U14 pad 17: GND -> /IR_Sensor/SPK_N
- U14 pad 2: I2S_SPK_GAIN0 -> Net-(R99-Pad1)
- U14 pad 3: GND -> Net-(R99-Pad1)
- U14 pad 4: Net-(R100-Pad1) -> I2S_SPK_LRCLK
- U14 pad 5: (no net) -> I2S_SPK_LRCLK
- U14 pad 6: (no net) -> I2S_SPK_BCLK
- U14 pad 7: LEDLOGICVDD -> I2S_SPK_DATA
- U14 pad 8: LEDLOGICVDD -> SCL
- U14 pad 9: /IR_Sensor/SPK_P -> SDA
- U16 pad 13: Net-(R46-Pad1) -> Net-(R48-Pad1)
- U16 pad 16: Net-(R48-Pad1) -> Net-(R56-Pad2)
- U16 pad 23: Net-(R56-Pad2) -> Net-(R125-Pad2)
- U16 pad 24: Net-(R52-Pad2) -> Net-(R127-Pad2)
- U16 pad 26: Net-(R51-Pad2) -> Net-(R138-Pad1)
- U16 pad 29: Net-(R132-Pad2) -> Net-(R52-Pad2)
- U16 pad 30: Net-(R131-Pad2) -> Net-(R132-Pad1)
- U16 pad 31: Net-(R130-Pad2) -> Net-(R131-Pad1)
- U16 pad 4: Net-(U16-Pad4) -> Net-(R51-Pad2)
- U16 pad 5: Net-(U16-Pad5) -> Net-(R121-Pad2)
- U16 pad 9: Net-(R121-Pad2) -> Net-(R137-Pad1)
- U20 pad 24: Net-(P2-Pad6) -> RTS
- U20 pad 25: Net-(P2-Pad4) -> E_TX
- U20 pad 26: Net-(P2-Pad3) -> E_RX
- U20 pad 28: Net-(P2-Pad5) -> DTR
- U21 pad 1: VSPI_SS -> E_RX2
- U21 pad 3: VSPI_MISO -> E_TX2
- U21 pad 4: VSPI_MOSI -> Net-(U21-Pad4)
- U21 pad 6: VSPI_SCK -> Net-(U21-Pad6)
- U22 pad 1: GND -> IRLED_A
Routing:
- net GND: track 2184.6 -> 3086.4 mm, vias 117 -> 241
- net IRLED_A: track 0.00 -> 290.2 mm, vias 0 -> 7
- net /IR_Sensor/IRLED_K: track 286.9 -> 0.00 mm, vias 2 -> 0
- net LEDLOGICVDD: track 99.0 -> 296.0 mm, vias 5 -> 18
- net E_RX2: track 0.00 -> 128.2 mm, vias 0 -> 2
- net E_TX2: track 0.00 -> 127.1 mm, vias 0 -> 2
- net VSPI_MISO: track 122.3 -> 0.00 mm, vias 2 -> 0
- net VSPI_SS: track 118.2 -> 3.14 mm, vias 2 -> 1
- net LEDVDD: track 797.9 -> 698.8 mm, vias 36 -> 37
- net ESPVDD: track 91.0 -> 10.9 mm, vias 4 -> 1
- net I2S_SPK_MCLK: track 0.00 -> 73.6 mm, vias 0 -> 1
- net I2S_SPK_GAIN1: track 68.8 -> 0.00 mm, vias 3 -> 0
- net RTS: track 63.6 -> 130.0 mm, vias 2 -> 7
- net I2S_SPK_GAIN0: track 63.8 -> 0.00 mm, vias 2 -> 0
- net DTR: track 52.7 -> 110.6 mm, vias 2 -> 7
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- added copper zone on F.Cu, net /IR_Sensor/SPK_N
- added copper zone on F.Cu, net /IR_Sensor/SPK_P
- added copper zone on F.Cu, net GND
- removed copper zone on B.Cu, net Net-(C72-Pad1)
- removed copper zone on F.Cu, net Net-(C72-Pad1)
Other:
- outline, holes or cut-outs redrawn

Commit message: Added stereo power amplifier
Parts:
- removed C20: 1u, Capacitors_SMD:C_0603_HandSoldering
- removed LS1: Speaker, Wire_Connections_Bridges:WireConnection_1.50mmDrill
- removed Q31: Q_NPN_BEC, TO_SOT_Packages_SMD:SOT-23_Handsoldering
- removed R12, R42: 10k, Resistors_SMD:R_0603_HandSoldering
- added C88: 2200p 16V, Capacitors_SMD:C_0603_HandSoldering, F.Cu at (95.7, 102.2)
- added C89: 2200p 16V, Capacitors_SMD:C_0603_HandSoldering, F.Cu at (95.7, 104.9)
- added C90: 2200p 16V, Capacitors_SMD:C_0603_HandSoldering, F.Cu at (95.7, 107.5)
- added C91: 2200p 16V, Capacitors_SMD:C_0603_HandSoldering, F.Cu at (95.7, 110.2)
- added C92: 2200p 16V, Capacitors_SMD:C_0603_HandSoldering, F.Cu at (95.7, 103.5)
- added C93: 2200p 16V, Capacitors_SMD:C_0603_HandSoldering, F.Cu at (95.7, 106.0)
- added C94: 2200p 16V, Capacitors_SMD:C_0603_HandSoldering, F.Cu at (95.7, 108.8)
- added C95: 2200p 16V, Capacitors_SMD:C_0603_HandSoldering, F.Cu at (95.7, 111.3)
- added C96: 1u, Capacitors_SMD:C_0603_HandSoldering, F.Cu at (82.2, 92.2)
- added F2: FUSE 2A, Resistors_SMD:R_1812, B.Cu at (98.0, 116.0)
- added JP1: Jumper_NC_Small, components:J_2.3mm, F.Cu at (105.0, 117.4)
- added L10: 300R@100MHz 4A, Capacitors_SMD:C_0805_HandSoldering, B.Cu at (93.2, 107.5)
- added L11: 300R@100MHz 4A, Capacitors_SMD:C_0805_HandSoldering, B.Cu at (93.2, 110.0)
- added L7: 100R@100MHz 4A, Capacitors_SMD:C_0805_HandSoldering, F.Cu at (101.6, 114.4)
- added L8: 300R@100MHz 4A, Capacitors_SMD:C_0805_HandSoldering, B.Cu at (93.2, 102.2)
- added L9: 300R@100MHz 4A, Capacitors_SMD:C_0805_HandSoldering, B.Cu at (93.2, 104.8)
- added R141: 10k, Resistors_SMD:R_0603_HandSoldering, F.Cu at (110.6, 108.6)
- added R142: 68R, Resistors_SMD:R_0603_HandSoldering, F.Cu at (99.2, 103.4)
- added R143: 68R, Resistors_SMD:R_0603_HandSoldering, F.Cu at (99.3, 106.0)
- added R144: 68R, Resistors_SMD:R_0603_HandSoldering, F.Cu at (99.5, 108.6)
- added R145: 68R, Resistors_SMD:R_0603_HandSoldering, F.Cu at (99.5, 111.2)
- C18, C36: value 1u -> 1u 16V
- C19: value 1u -> 0.1u 16V; moved to F.Cu
- C29, C31, C57, C59, C60, C61, C63, C77, C78, C87, L5, Q2, Q4, R100, R125, R126, R127, R130, R139, R140, R16, R17, R26, R28, R46, R48, R50, R52, R56, T1, U27: moved to B.Cu
- C3: value 220p -> 1u 16V; moved to F.Cu
- C79: value 1u 16V -> 22u 16V; footprint Capacitors_SMD:C_0603_HandSoldering -> Capacitors_SMD:C_1206_HandSoldering
- C80: value 1u 16V -> 22u 16V; footprint Capacitors_SMD:C_0603_HandSoldering -> Capacitors_SMD:C_1206_HandSoldering; moved to B.Cu
- C81: value 10u 16V -> 0.22u 30V; footprint Capacitors_SMD:C_1206_HandSoldering -> Capacitors_SMD:C_0603_HandSoldering; moved to F.Cu
- C82: value 10u 16V -> 0.22u 30V; footprint Capacitors_SMD:C_1206_HandSoldering -> Capacitors_SMD:C_0603_HandSoldering
- C83, C84: value 0.1u 16V -> 0.22u 30V
- C85: value 0.1u 16V -> 22u 16V; footprint Capacitors_SMD:C_0603_HandSoldering -> Capacitors_SMD:C_1206_HandSoldering
- C86: value 0.1u 16V -> 22u 16V; footprint Capacitors_SMD:C_0603_HandSoldering -> Capacitors_SMD:C_1206_HandSoldering; moved to B.Cu
- CONN1: footprint Connect:BARREL_JACK -> components:BARREL_JACK_HIGH_CURRENT_PJ018
- F1: footprint Resistors_SMD:R_1812_HandSoldering -> Resistors_SMD:R_1812
- J4: value Conn_01x02 -> Conn_01x06; footprint Wire_Connections_Bridges:WireConnection_1.50mmDrill -> components:Push_Terminal_6P_2.54
- R40, R53: moved to F.Cu
- SW1, SW2: footprint Buttons_Switches_SMD:SW_SPST_FSMSM -> components:TACT_SW_SMD_Panasonic-EVPAWBD2A
- SW3, SW4, SW5, SW6, SW7, SW8: footprint components:SW_PUSH_6mm-2pin -> components:TACT_SW_SMD_Panasonic-EVPAWBD2A
- U14: value TAS5720 -> TAS5805M; footprint components:QFN-32-1EP_4x4mm_Pitch0.4mm_Handsoldering -> components:HTSSOP-28_4.4x9.7mm_Pitch0.65mm_PowerPad; moved to B.Cu
- moved R1 216.3 mm to (88.6, 94.8), turned to 0 degrees
- moved R140 211.4 mm to (84.1, 72.4)
- moved R139 211.0 mm to (85.1, 76.6)
- moved L6 209.9 mm to (108.1, 70.5), turned to 180 degrees
- moved C4 209.5 mm to (105.6, 69.0), turned to 180 degrees
- moved Q1 208.5 mm to (101.4, 75.9), turned to 270 degrees
- moved LED49 207.2 mm to (80.9, 75.0), turned to 90 degrees
- moved R26 204.5 mm to (86.3, 75.2)
- moved R16 199.5 mm to (85.0, 73.8), turned to 0 degrees
- moved D14 198.9 mm to (104.3, 71.1), turned to 180 degrees
- moved C3 195.2 mm to (111.2, 102.8), turned to 90 degrees
- moved R17 187.4 mm to (103.6, 73.9), turned to 90 degrees
- moved R56 82.6 mm to (116.6, 42.8), turned to 270 degrees
- moved R125 77.3 mm to (114.3, 41.6), turned to 90 degrees
- moved R48 76.5 mm to (112.0, 54.0), turned to 270 degrees
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Connections:
- net Net-(U24-Pad6) renamed IRLED_K
- C18 pad 1: Net-(C18-Pad1) -> LEDLOGICVDD
- C18 pad 2: Net-(C18-Pad2) -> /PowerAmplifier/PAGND
- C19 pad 1: Net-(C18-Pad1) -> LEDLOGICVDD
- C19 pad 2: Net-(C19-Pad2) -> /PowerAmplifier/PAGND
- C3 pad 1: IR_OUT -> Net-(C3-Pad1)
- C3 pad 2: Net-(C3-Pad2) -> /PowerAmplifier/PAGND
- C36 pad 1: GND -> Net-(C36-Pad1)
- C36 pad 2: LEDLOGICVDD -> /PowerAmplifier/PAGND
- C63 pad 1: VCC -> /PowerAmplifier/PAVDD
- C63 pad 2: GND -> /PowerAmplifier/PAGND
- C72 pad 1: Net-(C72-Pad1) -> DC_IN_P
- C78 pad 1: VCC -> /PowerAmplifier/PAVDD
- C78 pad 2: GND -> /PowerAmplifier/PAGND
- C79 pad 1: VCC -> /PowerAmplifier/PAVDD
- C79 pad 2: GND -> /PowerAmplifier/PAGND
- C80 pad 1: VCC -> /PowerAmplifier/PAVDD
- C80 pad 2: GND -> /PowerAmplifier/PAGND
- C81 pad 1: VCC -> Net-(C81-Pad1)
- C81 pad 2: GND -> Net-(C81-Pad2)
- C82 pad 1: VCC -> Net-(C82-Pad1)
- C82 pad 2: GND -> Net-(C82-Pad2)
- C83 pad 1: /IR_Sensor/SPK_P -> Net-(C83-Pad1)
- C84 pad 1: /IR_Sensor/SPK_P -> Net-(C84-Pad1)
- C84 pad 2: Net-(C83-Pad2) -> Net-(C84-Pad2)
- C85 pad 1: /IR_Sensor/SPK_N -> /PowerAmplifier/PAVDD
- C85 pad 2: Net-(C85-Pad2) -> /PowerAmplifier/PAGND
- C86 pad 1: /IR_Sensor/SPK_N -> /PowerAmplifier/PAVDD
- C86 pad 2: Net-(C85-Pad2) -> /PowerAmplifier/PAGND
- F1 pad 1: DC_IN_P -> V12_PREFUSE
- F1 pad 2: Net-(C72-Pad1) -> VCC
- R1 pad 1: Net-(Q31-Pad3) -> GND
- R1 pad 2: Net-(C4-Pad1) -> IRLED_A
- R17 pad 2: Net-(Q31-Pad3) -> IR_OUT
- R99 pad 1: Net-(R99-Pad1) -> LEDLOGICVDD
- R99 pad 2: LEDLOGICVDD -> Net-(R99-Pad2)
- T1 pad 1: Net-(C72-Pad1) -> DC_IN_P
- T1 pad 4: VCC -> V12_PREFUSE
- U14 pad 1: Net-(C18-Pad1) -> /PowerAmplifier/PAGND
- U14 pad 10: GND -> SDA
- U14 pad 11: LEDLOGICVDD -> SCL
- U14 pad 12: GND -> Net-(R141-Pad2)
- U14 pad 13: GND -> Net-(C36-Pad1)
- U14 pad 14: VCC -> /PowerAmplifier/PAGND
- U14 pad 15: VCC -> /PowerAmplifier/PAVDD
- U14 pad 16: /IR_Sensor/SPK_N -> /PowerAmplifier/PAVDD
- U14 pad 17: /IR_Sensor/SPK_N -> Net-(C84-Pad1)
- U14 pad 18: Net-(C85-Pad2) -> Net-(C84-Pad2)
- U14 pad 19: GND -> /PowerAmplifier/PAGND
- U14 pad 2: Net-(R99-Pad1) -> LEDLOGICVDD
- U14 pad 20: GND -> Net-(C83-Pad1)
- U14 pad 21: GND -> Net-(C83-Pad2)
- U14 pad 22: GND -> Net-(C82-Pad1)
- U14 pad 23: Net-(C83-Pad2) -> Net-(C82-Pad2)
- U14 pad 24: /IR_Sensor/SPK_P -> /PowerAmplifier/PAGND
- U14 pad 25: /IR_Sensor/SPK_P -> Net-(C81-Pad1)
- U14 pad 26: VCC -> Net-(C81-Pad2)
- U14 pad 27: VCC -> /PowerAmplifier/PAVDD
- U14 pad 28: VCC -> /PowerAmplifier/PAVDD
- U14 pad 29: GND -> /PowerAmplifier/PAGND
- U14 pad 3: Net-(R99-Pad1) -> Net-(R99-Pad2)
- U14 pad 4: I2S_SPK_LRCLK -> Net-(C3-Pad1)
- U14 pad 5: I2S_SPK_LRCLK -> /PowerAmplifier/PAGND
- U14 pad 6: I2S_SPK_BCLK -> I2S_SPK_LRCLK
- U14 pad 7: I2S_SPK_DATA -> I2S_SPK_BCLK
- U14 pad 8: SCL -> I2S_SPK_DATA
- U14 pad 9: SDA -> Net-(U14-Pad9)
- U22 pad 1: IRLED_A -> Net-(U22-Pad1)
Routing:
- net IRLED_A: track 290.2 -> 63.5 mm, vias 7 -> 3
- net VSPI_MOSI: track 138.9 -> 0.00 mm, vias 5 -> 0
- net VSPI_SCK: track 130.0 -> 0.00 mm, vias 5 -> 0
- net /PowerAmplifier/PAGND: track 0.00 -> 74.0 mm, vias 0 -> 3
- net DC_IN_P: track 0.00 -> 73.7 mm, vias 0 -> 8
- net VCC: track 95.2 -> 37.3 mm, vias 5 -> 2
- net E_HS2_CMD: track 0.00 -> 52.3 mm, vias 0 -> 3
- net E_HS2_DATA0: track 0.00 -> 52.0 mm, vias 0 -> 3
- net IR_OUT: track 75.6 -> 35.4 mm, vias 7 -> 5
- net V12_PREFUSE: track 0.00 -> 37.9 mm, vias 0 -> 19
- net LEDLOGICVDD: track 296.0 -> 332.9 mm, vias 18 -> 19
- net E_HS2_CLK: track 0.00 -> 35.5 mm, vias 0 -> 3
- net /power/DC_IN_N: track 0.00 -> 35.0 mm, vias 0 -> 1
- net Net-(C55-Pad2): track 43.9 -> 12.4 mm, vias 5 -> 2
- net /IR_Sensor/SPK_N: track 26.8 -> 0.00 mm, vias 2 -> 0
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- added copper zone on B.Cu, net /PowerAmplifier/PAGND
- added copper zone on F.Cu, net /PowerAmplifier/PAGND
- added copper zone on B.Cu, net /PowerAmplifier/PAVDD
- added copper zone on F.Cu, net /PowerAmplifier/PAVDD
- added copper zone on B.Cu, net DC_IN_P
- added copper zone on F.Cu, net DC_IN_P
- added copper zone on B.Cu, net Net-(F2-Pad2)
- added copper zone on F.Cu, net Net-(F2-Pad2)
- added copper zone on B.Cu, net V12_PREFUSE
- added copper zone on F.Cu, net V12_PREFUSE
- removed copper zone on F.Cu, net /IR_Sensor/SPK_N
- removed copper zone on F.Cu, net /IR_Sensor/SPK_P
- removed copper zone on F.Cu, net /power/LEDDC_SW
- removed copper zone on F.Cu, net VCC
