File: power_amp.sch (KiCad schematic (older format))
At the start: 37 parts, among them J4 Conn_01x06, U14 TAS5805M

Commit message: Switched to new kicad libraries
Parts:
- C18, C19, C3, C36, C63, C78, C79, C80, C81, C82, C83, C84, C85, C86, C88, C89, C90, C91, C92, C93, C94, C95: symbol device:C -> dotmatrix_64x48-rescue:C-device
- F2: symbol device:Polyfuse_Small -> dotmatrix_64x48-rescue:Polyfuse_Small-device
- J4: symbol Connector:Conn_01x06 -> dotmatrix_64x48-rescue:Conn_01x06-Connector
- JP1: symbol device:Jumper_NC_Small -> dotmatrix_64x48-rescue:Jumper_NC_Small-device
- L10, L11, L7, L8, L9: symbol device:Ferrite_Bead_Small -> dotmatrix_64x48-rescue:Ferrite_Bead_Small-device
- R141, R142, R143, R144, R145, R99: symbol device:R -> dotmatrix_64x48-rescue:R-device
Changed lines of the file:
@@
 $EndComp
 $Comp
-L device:Polyfuse_Small F?
+L dotmatrix_64x48-rescue:Polyfuse_Small-device F?
 U 1 1 5BEBDE63
 P 1600 900
@@
 PAVDD
 $Comp
-L device:C C?
+L dotmatrix_64x48-rescue:C-device C?
 U 1 1 5BF678A2
 P 5250 1500
@@
 $EndComp
 $Comp
-L device:C C?
+L dotmatrix_64x48-rescue:C-device C?
 U 1 1 5BF67BDF
 P 4850 1500
@@
 $EndComp
 $Comp
-L device:C C?
+L dotmatrix_64x48-rescue:C-device C?
 U 1 1 5BF68272
 P 5050 1500
@@
 PAVDD
 $Comp
-L device:C C?
+L dotmatrix_64x48-rescue:C-device C?
 U 1 1 5BF7F19F
 P 5250 3900
@@
 $EndComp
 $Comp
-L device:C C?
+L dotmatrix_64x48-rescue:C-device C?
 U 1 1 5BF7F1A9
 P 4850 3900
@@
 $EndComp
 $Comp
-L device:C C?
+L dotmatrix_64x48-rescue:C-device C?
 U 1 1 5BF7F1B3
 P 5050 3900
@@
 	4400 3250 4400 3150
 $Comp
-L device:C C?
+L dotmatrix_64x48-rescue:C-device C?
 U 1 1 5BF8D61C
 P 1850 1900
@@
 $EndComp
 $Comp
-L device:C C?
+L dotmatrix_64x48-rescue:C-device C?
 U 1 1 5BF8DAF9
 P 2050 1900
@@
 Connection ~ 2050 1750
 $Comp
-L device:C C?
+L dotmatrix_64x48-rescue:C-device C?
 U 1 1 5BFAD080
 P 2350 3150
@@
 	3000 3150 2500 3150
 $Comp
-L power:GND #PWR?
+L dotmatrix_64x48-rescue:GND-power #PWR?
 U 1 1 5BFBAC84
 P 1400 1200
@@
 SDA
 $Comp
-L device:R R?
+L dotmatrix_64x48-rescue:R-device R?
 U 1 1 5BFBCA36
 P 2700 2150
@@
 	2550 1750 2800 1750
 $Comp
-L device:R R?
+L dotmatrix_64x48-rescue:R-device R?
 U 1 1 5BFCF6F8
 P 2700 3050
@@
 NoConn ~ 3000 2750
 $Comp
-L device:Ferrite_Bead_Small L?
+L dotmatrix_64x48-rescue:Ferrite_Bead_Small-device L?
 U 1 1 5C0019D9
 P 2000 900
@@
 	2100 900  2350 900
 $Comp
-L device:C C?
+L dotmatrix_64x48-rescue:C-device C?
 U 1 1 5C010B8D
 P 5200 2250
@@
 $EndComp
 $Comp
-L device:C C?
+L dotmatrix_64x48-rescue:C-device C?
 U 1 1 5C01A66F
 P 5200 2550
@@
 $EndComp
 $Comp
-L device:C C?
+L dotmatrix_64x48-rescue:C-device C?
 U 1 1 5C01A8C6
 P 5200 2750
@@
 $EndComp
 $Comp
-L device:C C?
+L dotmatrix_64x48-rescue:C-device C?
 U 1 1 5C01AB01
 P 5200 3050
@@
 	5050 3050 4400 3050
 $Comp
-L device:Ferrite_Bead_Small L?
+L dotmatrix_64x48-rescue:Ferrite_Bead_Small-device L?
 U 1 1 5C0438A0
 P 5600 2150
@@
 $EndComp
 $Comp
-L device:Ferrite_Bead_Small L?
+L dotmatrix_64x48-rescue:Ferrite_Bead_Small-device L?
 U 1 1 5C0496AD
 P 5600 2450
@@
 $EndComp
 $Comp
-L device:Ferrite_Bead_Small L?
+L dotmatrix_64x48-rescue:Ferrite_Bead_Small-device L?
 U 1 1 5C04EC52
 P 5600 2650
@@
 $EndComp
 $Comp
-L device:Ferrite_Bead_Small L?
+L dotmatrix_64x48-rescue:Ferrite_Bead_Small-device L?
 U 1 1 5C054279
 P 5600 2950
@@
 $EndComp
 $Comp
-L device:C C?
+L dotmatrix_64x48-rescue:C-device C?
 U 1 1 5C0599C2
 P 6900 2250
@@
 $EndComp
 $Comp
-L device:C C?
+L dotmatrix_64x48-rescue:C-device C?
 U 1 1 5C06F54D
 P 6900 2550
@@
 $EndComp
 $Comp
-L device:C C?
+L dotmatrix_64x48-rescue:C-device C?
 U 1 1 5C074CA9
 P 6900 2750
@@
 $EndComp
 $Comp
-L device:C C?
+L dotmatrix_64x48-rescue:C-device C?
 U 1 1 5C07A2A6
 P 6900 3050
@@
 $EndComp
 $Comp
-L device:C C?
+L dotmatrix_64x48-rescue:C-device C?
 U 1 1 5C07FA1E
 P 7900 2150
@@
 $EndComp
 $Comp
-L device:C C?
+L dotmatrix_64x48-rescue:C-device C?
 U 1 1 5C07FA28
 P 7900 2450
@@
 $EndComp
 $Comp
-L device:C C?
+L dotmatrix_64x48-rescue:C-device C?
 U 1 1 5C07FA32
 P 7900 2650
@@
 $EndComp
 $Comp
-L device:C C?
+L dotmatrix_64x48-rescue:C-device C?
 U 1 1 5C07FA3C
 P 7900 2950
@@
 $EndComp
 $Comp
-L device:R R?
+L dotmatrix_64x48-rescue:R-device R?
 U 1 1 5C086352
 P 8750 2150
@@
 $EndComp
 $Comp
-L device:R R?
+L dotmatrix_64x48-rescue:R-device R?
 U 1 1 5C091602
 P 8750 2450
@@
 $EndComp
 $Comp
-L device:R R?
+L dotmatrix_64x48-rescue:R-device R?
 U 1 1 5C096BBA
 P 8750 2650
@@
 $EndComp
 $Comp
-L device:R R?
+L dotmatrix_64x48-rescue:R-device R?
 U 1 1 5C09C15E
 P 8750 2950
@@
 	7700 2950 7750 2950
 $Comp
-L Connector:Conn_01x06 J4
+L dotmatrix_64x48-rescue:Conn_01x06-Connector J4
 U 1 1 5BE19489
 P 10250 2400
@@
 V12_PREFUSE
 $Comp
-L power:GND #PWR?
+L dotmatrix_64x48-rescue:GND-power #PWR?
 U 1 1 5BE4E7B0
 P 10050 2300
@@
 $EndComp
 $Comp
-L device:Jumper_NC_Small JP1
+L dotmatrix_64x48-rescue:Jumper_NC_Small-device JP1
 U 1 1 5BE3A85D
 P 1750 1150
@@
 PAGND
 $Comp
-L device:C C?
+L dotmatrix_64x48-rescue:C-device C?
 U 1 1 5BE6763D
 P 2350 2250
