File: usb_uart.sch (KiCad schematic (older format))
At the start: 12 parts, among them U20 CP2102N-A01-GQFN28, U25 CM1293A-04SO

Commit message: Added power input filter circut; Adjust MLCC size/value to be able to use cheap components
Parts:
- C67: value 10u 10V -> 22u/6.3V
- C69: value 10u 10V -> 10u/35V
Changed lines of the file:
@@
 P 3800 2350
 F 0 "C69" H 3750 1950 50  0000 L CNN
-F 1 "10u 10V" V 3650 1850 50  0000 L CNN
+F 1 "10u/35V" V 3650 1850 50  0000 L CNN
 F 2 "Capacitor_SMD:C_0603_1608Metric_Pad1.05x0.95mm_HandSolder" H 3915 2259 50  0001 L CNN
 F 3 "" H 3800 2350 50  0000 C CNN
@@
 P 3800 1450
 F 0 "C67" H 3750 1050 50  0000 L CNN
-F 1 "10u 10V" V 3650 950 50  0000 L CNN
+F 1 "22u/6.3V" V 3650 950 50  0000 L CNN
 F 2 "Capacitor_SMD:C_0603_1608Metric_Pad1.05x0.95mm_HandSolder" H 3915 1359 50  0001 L CNN
 F 3 "" H 3800 1450 50  0000 C CNN

Commit message: Changed footprints from old 4.x's R/C to 5.x's
Parts:
- C70, C71: value 1u -> 1u/35V; footprint Capacitors_SMD:C_0603_HandSoldering -> Capacitor_SMD:C_0603_1608Metric_Pad1.05x0.95mm_HandSolder
- C73, C74: value 0.1u -> 0.1u/35V; footprint Capacitors_SMD:C_0603_HandSoldering -> Capacitor_SMD:C_0603_1608Metric_Pad1.05x0.95mm_HandSolder
- R116, R117: footprint Resistors_SMD:R_0603_HandSoldering -> Resistor_SMD:R_0603_1608Metric_Pad1.05x0.95mm_HandSolder
Changed lines of the file:
@@
 P 4000 2350
 F 0 "C71" H 3950 1950 50  0000 L CNN
-F 1 "1u" H 4000 1850 50  0000 L CNN
-F 2 "Capacitors_SMD:C_0603_HandSoldering" H 4115 2259 50  0001 L CNN
+F 1 "1u/35V" H 4000 1850 50  0000 L CNN
+F 2 "Capacitor_SMD:C_0603_1608Metric_Pad1.05x0.95mm_HandSolder" H 4115 2259 50  0001 L CNN
 F 3 "" H 4000 2350 50  0000 C CNN
 	1    4000 2350
@@
 P 4200 2350
 F 0 "C74" H 4150 1950 50  0000 L CNN
-F 1 "0.1u" H 4150 1850 50  0000 L CNN
-F 2 "Capacitors_SMD:C_0603_HandSoldering" H 4315 2259 50  0001 L CNN
+F 1 "0.1u/35V" H 4150 1850 50  0000 L CNN
+F 2 "Capacitor_SMD:C_0603_1608Metric_Pad1.05x0.95mm_HandSolder" H 4315 2259 50  0001 L CNN
 F 3 "" H 4200 2350 50  0000 C CNN
 	1    4200 2350
@@
 P 4000 1450
 F 0 "C70" H 3950 1050 50  0000 L CNN
-F 1 "1u" H 4000 950 50  0000 L CNN
-F 2 "Capacitors_SMD:C_0603_HandSoldering" H 4115 1359 50  0001 L CNN
+F 1 "1u/35V" H 4000 950 50  0000 L CNN
+F 2 "Capacitor_SMD:C_0603_1608Metric_Pad1.05x0.95mm_HandSolder" H 4115 1359 50  0001 L CNN
 F 3 "" H 4000 1450 50  0000 C CNN
 	1    4000 1450
@@
 P 4200 1450
 F 0 "C73" H 4150 1050 50  0000 L CNN
-F 1 "0.1u" H 4150 950 50  0000 L CNN
-F 2 "Capacitors_SMD:C_0603_HandSoldering" H 4315 1359 50  0001 L CNN
+F 1 "0.1u/35V" H 4150 950 50  0000 L CNN
+F 2 "Capacitor_SMD:C_0603_1608Metric_Pad1.05x0.95mm_HandSolder" H 4315 1359 50  0001 L CNN
 F 3 "" H 4200 1450 50  0000 C CNN
 	1    4200 1450
@@
 F 0 "R117" V 4550 1450 50  0000 L CNN
 F 1 "1k" V 4650 1600 50  0000 L CNN
-F 2 "Resistors_SMD:R_0603_HandSoldering" V 4480 1550 50  0001 C CNN
+F 2 "Resistor_SMD:R_0603_1608Metric_Pad1.05x0.95mm_HandSolder" V 4480 1550 50  0001 C CNN
 F 3 "" H 4550 1550 50  0000 C CNN
 	1    4550 1550
@@
 F 0 "R116" V 3250 1750 50  0000 L CNN
 F 1 "4.7k" V 3350 1900 50  0000 L CNN
-F 2 "Resistors_SMD:R_0603_HandSoldering" V 3180 1850 50  0001 C CNN
+F 2 "Resistor_SMD:R_0603_1608Metric_Pad1.05x0.95mm_HandSolder" V 3180 1850 50  0001 C CNN
 F 3 "" H 3250 1850 50  0000 C CNN
 	1    3250 1850
