File: column_driver.kicad_sch (KiCad schematic)
At the start: 24 parts, among them U10 LED1642GW, U3 LED1642GW, U4 LED1642GW, U5 LED1642GW, U6 LED1642GW, U7 LED1642GW, U8 LED1642GW, U9 LED1642GW

Commit message: To use WS2812-2020 as status LEDs; No critical DRC errors found
Parts:
- R18, R19, R20, R21, R22, R23, R24, R25: value 22k -> 10k
Changed lines of the file:
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@@
       (effects (font (size 1.27 1.27)) (justify left))
     )
-    (property "Value" "22k" (id 1) (at 53.848 72.263 0)
+    (property "Value" "10k" (id 1) (at 53.848 72.263 0)
       (effects (font (size 1.27 1.27)) (justify left))
     )
@@
       (effects (font (size 1.27 1.27)) (justify left))
     )
-    (property "Value" "22k" (id 1) (at 53.848 143.383 0)
+    (property "Value" "10k" (id 1) (at 53.848 143.383 0)
       (effects (font (size 1.27 1.27)) (justify left))
     )
@@
       (effects (font (size 1.27 1.27)) (justify left))
     )
-    (property "Value" "22k" (id 1) (at 107.188 72.263 0)
+    (property "Value" "10k" (id 1) (at 107.188 72.263 0)
       (effects (font (size 1.27 1.27)) (justify left))
     )
@@
       (effects (font (size 1.27 1.27)) (justify left))
     )
-    (property "Value" "22k" (id 1) (at 107.188 143.383 0)
+    (property "Value" "10k" (id 1) (at 107.188 143.383 0)
       (effects (font (size 1.27 1.27)) (justify left))
     )
@@
       (effects (font (size 1.27 1.27)) (justify left))
     )
-    (property "Value" "22k" (id 1) (at 160.528 72.263 0)
+    (property "Value" "10k" (id 1) (at 160.528 72.263 0)
       (effects (font (size 1.27 1.27)) (justify left))
     )
@@
       (effects (font (size 1.27 1.27)) (justify left))
     )
-    (property "Value" "22k" (id 1) (at 160.528 143.383 0)
+    (property "Value" "10k" (id 1) (at 160.528 143.383 0)
       (effects (font (size 1.27 1.27)) (justify left))
     )
@@
       (effects (font (size 1.27 1.27)) (justify left))
     )
-    (property "Value" "22k" (id 1) (at 213.868 72.263 0)
+    (property "Value" "10k" (id 1) (at 213.868 72.263 0)
       (effects (font (size 1.27 1.27)) (justify left))
     )
@@
       (effects (font (size 1.27 1.27)) (justify left))
     )
-    (property "Value" "22k" (id 1) (at 217.678 143.383 0)
+    (property "Value" "10k" (id 1) (at 217.678 143.383 0)
       (effects (font (size 1.27 1.27)) (justify left))
     )
