File: fet-driver.kicad_sch (KiCad schematic)
At the start: 32 parts, among them Q21 AO3401, Q22 AO3401, Q23 AO3401, Q24 AO3401, Q25 AO3401, Q26 AO3401, Q27 AO3401, Q28 AO3401

Commit message: Moved leftside sensors to rightside; Unified old footprints to new footprints; DRC clear
Parts:
- Q21, Q22, Q23, Q24, Q25, Q26, Q27, Q28: footprint TO_SOT_Packages_SMD:SOT-23_Handsoldering -> Package_TO_SOT_SMD:SOT-23_Handsoldering
Changed lines of the file:
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@@
       (effects (font (size 1.27 1.27)) (justify left))
     )
-    (property "Footprint" "TO_SOT_Packages_SMD:SOT-23_Handsoldering" (id 2) (at 114.3 35.56 0)
+    (property "Footprint" "Package_TO_SOT_SMD:SOT-23_Handsoldering" (id 2) (at 114.3 35.56 0)
       (effects (font (size 1.27 1.27)) hide)
     )
@@
       (effects (font (size 1.27 1.27)) (justify left))
     )
-    (property "Footprint" "TO_SOT_Packages_SMD:SOT-23_Handsoldering" (id 2) (at 114.3 54.61 0)
+    (property "Footprint" "Package_TO_SOT_SMD:SOT-23_Handsoldering" (id 2) (at 114.3 54.61 0)
       (effects (font (size 1.27 1.27)) hide)
     )
@@
       (effects (font (size 1.27 1.27)) (justify left))
     )
-    (property "Footprint" "TO_SOT_Packages_SMD:SOT-23_Handsoldering" (id 2) (at 114.3 73.66 0)
+    (property "Footprint" "Package_TO_SOT_SMD:SOT-23_Handsoldering" (id 2) (at 114.3 73.66 0)
       (effects (font (size 1.27 1.27)) hide)
     )
@@
       (effects (font (size 1.27 1.27)) (justify left))
     )
-    (property "Footprint" "TO_SOT_Packages_SMD:SOT-23_Handsoldering" (id 2) (at 114.3 92.71 0)
+    (property "Footprint" "Package_TO_SOT_SMD:SOT-23_Handsoldering" (id 2) (at 114.3 92.71 0)
       (effects (font (size 1.27 1.27)) hide)
     )
@@
       (effects (font (size 1.27 1.27)) (justify left))
     )
-    (property "Footprint" "TO_SOT_Packages_SMD:SOT-23_Handsoldering" (id 2) (at 114.3 113.03 0)
+    (property "Footprint" "Package_TO_SOT_SMD:SOT-23_Handsoldering" (id 2) (at 114.3 113.03 0)
       (effects (font (size 1.27 1.27)) hide)
     )
@@
       (effects (font (size 1.27 1.27)) (justify left))
     )
-    (property "Footprint" "TO_SOT_Packages_SMD:SOT-23_Handsoldering" (id 2) (at 114.3 132.08 0)
+    (property "Footprint" "Package_TO_SOT_SMD:SOT-23_Handsoldering" (id 2) (at 114.3 132.08 0)
       (effects (font (size 1.27 1.27)) hide)
     )
@@
       (effects (font (size 1.27 1.27)) (justify left))
     )
-    (property "Footprint" "TO_SOT_Packages_SMD:SOT-23_Handsoldering" (id 2) (at 114.3 151.13 0)
+    (property "Footprint" "Package_TO_SOT_SMD:SOT-23_Handsoldering" (id 2) (at 114.3 151.13 0)
       (effects (font (size 1.27 1.27)) hide)
     )
@@
       (effects (font (size 1.27 1.27)) (justify left))
     )
-    (property "Footprint" "TO_SOT_Packages_SMD:SOT-23_Handsoldering" (id 2) (at 114.3 170.18 0)
+    (property "Footprint" "Package_TO_SOT_SMD:SOT-23_Handsoldering" (id 2) (at 114.3 170.18 0)
       (effects (font (size 1.27 1.27)) hide)
     )
